Commit message: Modify physical parameters (inertia, mass, size)

File: rbsherpa_hl_description/urdf/bases/rbsherpa_hl_base.gazebo.xacro (robot description, xacro)
@@ -13,7 +13,7 @@
 				<!-- For V0 0.365 -->
 				<!-- wheelSeparation>0.365</wheelSeparation -->
-				<wheelSeparation>0.433</wheelSeparation>
-				<wheelDiameter>0.1524</wheelDiameter>
-				<commandTopic>rsherpa_hl/cmd_vel</commandTopic>
+				<wheelSeparation>0.720</wheelSeparation>
+				<wheelDiameter>0.3683</wheelDiameter>
+				<commandTopic>rbsherpa_hl/cmd_vel</commandTopic>
 				<odometryTopic>odom</odometryTopic>
 				<odometryFrame>$(prefix_frame)odom</odometryFrame>

File: rbsherpa_hl_description/urdf/bases/rbsherpa_hl_base.urdf.xacro (robot description, xacro)
@@ -24,7 +24,7 @@
   <link name="${prefix}base_link">
     <inertial>
-      <mass value="25.0" />
-      <origin xyz="0 0 0" />
-      <inertia  ixx="0.007" ixy="0.0"  ixz="0.0"  iyy="0.007"  iyz="0.0"  izz="0.78" />
+      <mass value="498.75915" />
+      <origin xyz="0.01399 0.00092 0.54575" />
+      <inertia  ixx="66.799101" ixy="-0.03168423"  ixz="12.670655"  iyy="151.592685"  iyz="0.0015868674"  izz="157.124924" />
     </inertial>
     <visual>

File: rbsherpa_hl_description/urdf/structures/structure.urdf.xacro (robot description, xacro)
@@ -2,13 +2,4 @@
 <robot name="rbsherpa_structure" xmlns:xacro="http://www.ros.org/wiki/xacro">
   <xacro:property name="M_PI" value="3.1415926535897931" />
-  <!-- TODO: Modify these values -->
-  <xacro:property name="wheel_radius" value="0.125" />
-  <xacro:property name="wheel_height" value="0.14" /> <!-- really is the wheel width -->
-  <xacro:property name="wheel_mass" value="6.5" /> <!-- in kg-->
-   <xacro:macro name="cylinder_inertia" params="m r h">
-    <inertia  ixx="${m*(3*r*r+h*h)/12}" ixy = "0" ixz = "0"
-              iyy="${m*r*r/2}" iyz = "0"
-              izz="${m*(3*r*r+h*h)/12}" />
-  </xacro:macro>
   <xacro:macro name="structure" params="prefix parent *origin">
 	<!--fixed joint -->
@@ -23,17 +14,19 @@
           <origin xyz="0 0 0" rpy="0 0 0" />
           <geometry>
-			 <mesh filename="package://rbsherpa_hl_description/meshes/structure/rbsherpa_hl_column.dae" />
+			      <mesh filename="package://rbsherpa_hl_description/meshes/structure/rbsherpa_hl_column.dae" />
           </geometry>
       </visual>
       <collision>
-		<origin xyz="0 0 0" rpy="0 0 0" />
+		    <origin xyz="0 0 0" rpy="0 0 0" />
         <geometry>
-			<mesh filename="package://rbsherpa_hl_description/meshes/structure/rbsherpa_hl_column.stl" />
+			    <mesh filename="package://rbsherpa_hl_description/meshes/structure/rbsherpa_hl_column.stl" />
         </geometry>
       </collision>
       <inertial>
-        <mass value="${wheel_mass}" />
-        <origin xyz="0 0 0" />
-        <cylinder_inertia  m="${wheel_mass}" r="${wheel_radius}" h="${wheel_height}" />
+        <mass value="14.92765" />
+        <origin xyz="-0.0195 -0.01 -0.750" />
+        <inertia  ixx="2.807543" ixy = "0" ixz = "0"
+                  iyy="2.804071" iyz = "0"
+                  izz="0.0137441" />
       </inertial>
     </link>
@@ -49,17 +42,19 @@
           <origin xyz="0 0 0" rpy="0 0 0" />
           <geometry>
-			 <mesh filename="package://rbsherpa_hl_description/meshes/structure/rbsherpa_hl_tt_giro.dae" />
+			      <mesh filename="package://rbsherpa_hl_description/meshes/structure/rbsherpa_hl_tt_giro.dae" />
           </geometry>
       </visual>
       <collision>
-		<origin xyz="0 0 0" rpy="0 0 0" />
+		    <origin xyz="0 0 0" rpy="0 0 0" />
         <geometry>
-			<mesh filename="package://rbsherpa_hl_description/meshes/structure/rbsherpa_hl_tt_giro.stl" />
+			    <mesh filename="package://rbsherpa_hl_description/meshes/structure/rbsherpa_hl_tt_giro.stl" />
         </geometry>
       </collision>
       <inertial>
-        <mass value="${wheel_mass}" />
-        <origin xyz="0 0 0" />
-        <cylinder_inertia  m="${wheel_mass}" r="${wheel_radius}" h="${wheel_height}" />
+        <mass value="4.64491" />
+        <origin xyz="0 0 0.004" />
+        <inertia  ixx="0.134515" ixy = "0" ixz = "0"
+                  iyy="0.0086520177" iyz = "0"
+                  izz="0.143118" />
       </inertial>
     </link>

File: rbsherpa_hl_description/urdf/wheels/motor_rubber_wheel.urdf.xacro (robot description, xacro)
@@ -4,15 +4,5 @@
   <xacro:include filename="$(find rbsherpa_hl_description)/urdf/wheels/motor_rubber_wheel.gazebo.xacro"/>
   <xacro:property name="M_PI" value="3.1415926535897931" />
-  <!-- Wheels -->
-  <xacro:property name="wheel_radius" value="0.125" />
-  <xacro:property name="wheel_height" value="0.14" /> <!-- really is the wheel width -->
-  <xacro:property name="wheel_mass" value="6.5" /> <!-- in kg-->
-  <xacro:macro name="cylinder_inertia" params="m r h">
-    <inertia  ixx="${m*(3*r*r+h*h)/12}" ixy = "0" ixz = "0"
-              iyy="${m*r*r/2}" iyz = "0"
-              izz="${m*(3*r*r+h*h)/12}" />
-  </xacro:macro>
   <xacro:macro name="motor_rubber_wheel" params="prefix parent *origin reflect hq">
-	<!--WHEEL TIRE -->
     <joint name="${prefix}_wheel_joint" type="continuous">
       <parent link="${parent}"/>
@@ -52,7 +42,9 @@
       </collision>
       <inertial>
-        <mass value="${wheel_mass}" />
-        <origin xyz="0 0 0" />
-        <cylinder_inertia  m="${wheel_mass}" r="${wheel_radius}" h="${wheel_height}" />
+        <mass value="37.29668" />
+        <origin xyz="0.00122 -0.00633 0.07032" />
+        <inertia  ixx="0.656095" ixy = "0.0002884484" ixz = "0.0037546231"
+                  iyy="0.645381" iyz = "0.06221658"
+                  izz="0.160381" />
       </inertial>
     </link>

File: rbsherpa_hl_description/urdf/wheels/rubber_wheel.urdf.xacro (robot description, xacro)
@@ -5,12 +5,7 @@
   <xacro:property name="M_PI" value="3.1415926535897931" />
   <!-- Wheels -->
-  <xacro:property name="wheel_radius" value="0.125" />
-  <xacro:property name="wheel_height" value="0.14" /> <!-- really is the wheel width -->
-  <xacro:property name="wheel_mass" value="6.5" /> <!-- in kg-->
-  <xacro:macro name="cylinder_inertia" params="m r h">
-    <inertia  ixx="${m*(3*r*r+h*h)/12}" ixy = "0" ixz = "0"
-              iyy="${m*r*r/2}" iyz = "0"
-              izz="${m*(3*r*r+h*h)/12}" />
-  </xacro:macro>
+  <xacro:property name="wheel_radius" value="0.3683" />
+  <xacro:property name="wheel_height" value="0.14" /> <!--TODO: Unknown --> <!-- really is the wheel width -->
+  <xacro:property name="wheel_mass" value="5.7745" /> <!-- in kg-->
   <xacro:macro name="rubber_wheel" params="prefix parent *origin reflect hq">
 	<!--WHEEL TIRE -->
@@ -53,6 +48,8 @@
       <inertial>
         <mass value="${wheel_mass}" />
-        <origin xyz="0 0 0" />
-        <cylinder_inertia  m="${wheel_mass}" r="${wheel_radius}" h="${wheel_height}" />
+        <origin xyz="0.01608 0.01055 0" />
+        <inertia  ixx="0.09185239" ixy = "0" ixz = "0"
+                  iyy="0.05298241" iyz = "0"
+                  izz="0.05298241" />
       </inertial>
     </link>
