Commit message: rbsherpa_hl_description:: Changed inertial values

File: rbsherpa_hl_description/urdf/bases/rbsherpa_hl_base_tank.urdf.xacro (robot description, xacro)
@@ -5,8 +5,8 @@
     <xacro:property name="PI" value="3.1415926535897931"/>
     <xacro:property name="wheel_width" value="0.14" />
-    <xacro:macro name="cuboid_inertia" params="m h w d">
-      <inertia  ixx="${m*(h*h+d*d)/12}" ixy = "0" ixz = "0"
-                iyy="${m*(w*w+d*d)/12}" iyz = "0"
-                izz="${m*(w*w+h*h)/12}" />
+  <xacro:macro name="box_inertia" params="m x y z">
+    <inertia  ixx="${m*(y*y+z*z)/12}" ixy = "0" ixz = "0"
+              iyy="${m*(x*x+z*z)/12}" iyz = "0"
+              izz="${m*(x*x+y*y)/12}" />
     </xacro:macro>
     <!-- BASE FOOTPRINT -->
@@ -29,13 +29,7 @@
     <link name="${prefix}base_link">
       <inertial>
-        <mass value="381.91147" />
-        <xacro:if value="${hq}">
-          <origin xyz="0.01210 0.00057 0.41465" />
-          <inertia  ixx="66.029446" ixy="-0.05457547"  ixz="9.08271"  iyy="97.833795"  iyz="0.0012187052"  izz="79.714477" />
-        </xacro:if>
-        <xacro:unless value="${hq}">
-          <origin xyz="0 0 0.5" />
-          <cuboid_inertia  m="381.91147" h="0.925" w="1.55" d="0.5" />
-        </xacro:unless>
+        <mass value="400" />
+        <origin xyz="0 0 0.5" />
+        <box_inertia m="400" x="0.9" y="1.5" z="0.5"/>
       </inertial>
       <visual>

File: rbsherpa_hl_description/urdf/pantilt/pan_tilt.urdf.xacro (robot description, xacro)
@@ -67,7 +67,7 @@
       </collision>
       <inertial>
-        <mass value="0.005" />
+        <mass value="0.5" />
         <origin xyz="0 0 0" />
-        <solid_cuboid_inertia m="0.005" h="0.05" d="0.05" w="0.05"/>
+        <solid_cuboid_inertia m="0.5" h="0.05" d="0.05" w="0.05"/>
       </inertial>
     </link>
@@ -88,5 +88,5 @@
       <actuator name="${prefix}torso_pantilt_tilt_motor">
         <mechanicalReduction>1</mechanicalReduction>
-        <hardwareInterface>PositionJointInterface</hardwareInterface>
+        <hardwareInterface>hardware_interface/PositionJointInterface</hardwareInterface>
       </actuator>
     </transmission>
@@ -108,7 +108,7 @@
       </collision>
       <inertial>
-        <mass value="0.005" />
+        <mass value="0.5" />
         <origin xyz="0 0 0" />
-        <solid_cuboid_inertia m="0.005" h="0.05" d="0.05" w="0.05"/>
+        <solid_cuboid_inertia m="0.5" h="0.05" d="0.05" w="0.05"/>
       </inertial>
     </link>

File: rbsherpa_hl_description/urdf/wheels/wheel_steer.urdf.xacro (robot description, xacro)
@@ -42,6 +42,6 @@
       </collision>
       <inertial>
-        <mass value="32.81532" />
-        <xacro:if value="${hq}">
+        <mass value="5" />
+        <!--xacro:if value="${hq}">
           <origin xyz="0.00002 -0.06358 -0.18084" />
           <inertia  ixx="0.469495" ixy = "0.0001387555" ixz = "0.00006456469"
@@ -49,8 +49,8 @@
                     izz="0.263583" />
         </xacro:if>
-        <xacro:unless value="${hq}">
+        <xacro:unless value="${hq}"-->
           <origin xyz="0 0 -0.18084" />
           <cylinder_inertia  m="5" r="0.1" h="0.2" />
-        </xacro:unless>
+        <!--/xacro:unless-->
       </inertial>
     </link>

File: rbsherpa_hl_description/urdf/wheels/wheel_traction.urdf.xacro (robot description, xacro)
@@ -44,5 +44,5 @@
 	    <inertial>
 	      <mass value="6.91837" />
-				<xacro:if value="${hq}">
+				<!--xacro:if value="${hq}">
 		      <origin xyz="0 0.00036 0" />
 		      <inertia  ixx="0.06952851" ixy = "0" ixz = "0"
@@ -50,8 +50,8 @@
 		                izz="0.0695285" />
 				</xacro:if>
-				<xacro:unless value="${hq}">
+				<xacro:unless value="${hq}"-->
 					<origin xyz="0 0 0" />
 	        <cylinder_inertia  m="6.91837" r="${wheel_radius}" h="${wheel_height}" />
-				</xacro:unless>
+				<!--/xacro:unless-->
 	    </inertial>
 	  </link>
