Commit message: [rbsherpa_hl_description]:height of footprint corrected

File: rbsherpa_hl_description/urdf/bases/rbsherpa_hl_base.urdf.xacro (robot description, xacro)
@@ -16,5 +16,5 @@
     </link>
     <joint name="${prefix}base_footprint_joint" type="fixed">
-       <origin xyz="0 0 ${wheel_radius - wheel_offset_z}" rpy="0 0 0" />
+       <origin xyz="0 0 ${wheel_radius - wheel_offset_z - motor_wheel_offset_z}" rpy="0 0 0" />
       <parent link="${prefix}base_footprint"/>
       <child link="${prefix}base_link" />

Commit message: Update physical properties and refactor xacro files

File: rbsherpa_hl_description/urdf/bases/rbsherpa_hl_base.urdf.xacro (robot description, xacro)
@@ -2,57 +2,60 @@
 <robot name="rbsherpa_hl_base" xmlns:xacro="http://www.ros.org/wiki/xacro">
   <xacro:macro name="rbsherpa_hl_base" params="prefix publish_bf hq">
-  <!-- Robot mechanical and motor parameters -->
-  <xacro:property name="PI" value="3.1415926535897931"/>
-  <xacro:property name="wheel_width" value="0.14" />
-  <!-- BASE FOOTPRINT -->
-  <xacro:if value="${publish_bf}">
-    <link name="${prefix}base_footprint">
+    <!-- Robot mechanical and motor parameters -->
+    <xacro:property name="PI" value="3.1415926535897931"/>
+    <xacro:property name="wheel_width" value="0.14" />
+    <!-- BASE FOOTPRINT -->
+    <xacro:if value="${publish_bf}">
+      <link name="${prefix}base_footprint">
+        <visual>
+            <origin xyz="0 0 0" rpy="0 0 0" />
+            <geometry>
+               <box size="0.001 0.001 0.001" />
+            </geometry>
+        </visual>
+      </link>
+      <joint name="${prefix}base_footprint_joint" type="fixed">
+        <!--origin xyz="0 0 ${wheel_radius - wheel_offset_z - motor_wheel_offset_z}" rpy="0 0 0" /-->
+        <origin xyz="0 0 0" rpy="0 0 0" />
+        <parent link="${prefix}base_footprint"/>
+        <child link="${prefix}base_link" />
+      </joint>
+    </xacro:if>
+    <!-- BASE_LINK -->
+    <link name="${prefix}base_link">
+      <inertial>
+        <mass value="381.91147" />
+        <origin xyz="0.01210 0.00057 0.41465" />
+        <inertia  ixx="66.029446" ixy="-0.05457547"  ixz="9.08271"  iyy="97.833795"  iyz="0.0012187052"  izz="79.714477" />
+      </inertial>
       <visual>
-          <origin xyz="0 0 0" rpy="0 0 0" />
+        <origin xyz="0 0 0" rpy="0 0 0" />
+        <xacro:if value="${hq}">
           <geometry>
-             <box size="0.001 0.001 0.001" />
+            <mesh filename="package://rbsherpa_hl_description/meshes/bases/rbsherpa_hl_base.dae"/>
           </geometry>
+        </xacro:if>
+        <xacro:unless value="${hq}">
+          <geometry>
+            <mesh filename="package://rbsherpa_hl_description/meshes/bases/rbsherpa_hl_base.stl"/>
+          </geometry>
+        </xacro:unless>
+        <!--
+        <geometry>
+          <box size="1.4 0.7 0.5" />
+        </geometry>
+        <material name="darkgrey">
+          <color rgba="0.1 0.1 0.1 1"/>
+        </material>
+        -->
       </visual>
+      <collision>
+        <origin xyz="0 0 0.6" rpy="0 0 0 " />
+        <geometry>
+          <!--mesh filename="package://rbsherpa_hl_description/meshes/bases/rbsherpa_hl_base.dae"/-->
+          <box size="1.4 0.6 0.5" />
+        </geometry>
+      </collision>
     </link>
-    <joint name="${prefix}base_footprint_joint" type="fixed">
-       <!--origin xyz="0 0 ${wheel_radius - wheel_offset_z - motor_wheel_offset_z}" rpy="0 0 0" /-->
-       <origin xyz="0 0 0" rpy="0 0 0" />
-      <parent link="${prefix}base_footprint"/>
-      <child link="${prefix}base_link" />
-    </joint>
-  </xacro:if>
-  <!-- BASE_LINK -->
-  <link name="${prefix}base_link">
-    <inertial>
-      <mass value="498.75915" />
-      <origin xyz="0.01399 0.00092 0.54575" />
-      <inertia  ixx="66.799101" ixy="-0.03168423"  ixz="12.670655"  iyy="151.592685"  iyz="0.0015868674"  izz="157.124924" />
-    </inertial>
-    <visual>
-       <origin xyz="0 0 0" rpy="0 0 0" />
-       <xacro:if value="${hq}">
-       <geometry>
-         <mesh filename="package://rbsherpa_hl_description/meshes/bases/rbsherpa_hl_base.dae"/>
-       </geometry>
-       </xacro:if>
-       <xacro:unless value="${hq}">
-       <geometry>
-       <mesh filename="package://rbsherpa_hl_description/meshes/bases/rbsherpa_hl_base.stl"/>
-       </geometry>
-       </xacro:unless>
- <geometry>
-<box size="1.4 0.7 0.5" /></geometry>
-       <material name="darkgrey">
-         <color rgba="0.1 0.1 0.1 1"/>
-       </material>
-    </visual>
-    <collision>
-       <origin xyz="0 0 0.6" rpy="0 0 0 " />
-       <geometry>
-         <!--mesh filename="package://rbsherpa_hl_description/meshes/bases/rbsherpa_hl_base.dae"/-->
-			<box size="1.4 0.6 0.5" />
-       </geometry>
-    </collision>
-  </link>
   </xacro:macro>
 </robot>

File: rbsherpa_hl_description/urdf/structures/structure.urdf.xacro (robot description, xacro)
@@ -11,9 +11,8 @@
     <link name="${prefix}structure_link">
       <visual>
-        <!-- COLUMN -->
-          <origin xyz="0 0 0" rpy="0 0 0" />
-          <geometry>
-			      <mesh filename="package://rbsherpa_hl_description/meshes/structure/rbsherpa_hl_column.dae" />
-          </geometry>
+        <origin xyz="0 0 0" rpy="0 0 0" />
+        <geometry>
+		      <mesh filename="package://rbsherpa_hl_description/meshes/structure/rbsherpa_hl_column.dae" />
+        </geometry>
       </visual>
       <collision>
@@ -26,7 +25,7 @@
         <mass value="14.92765" />
         <origin xyz="-0.0195 -0.01 -0.750" />
-        <inertia  ixx="2.807543" ixy = "0" ixz = "0"
-                  iyy="2.804071" iyz = "0"
-                  izz="0.0137441" />
+        <inertia  ixx="2.80754349924" ixy = "0" ixz = "0"
+                  iyy="2.80407121984" iyz = "0"
+                  izz="0.01374410335" />
       </inertial>
     </link>
@@ -40,8 +39,8 @@
     <link name="${prefix}platform_link">
       <visual>
-          <origin xyz="0 0 0" rpy="0 0 0" />
-          <geometry>
-			      <mesh filename="package://rbsherpa_hl_description/meshes/structure/rbsherpa_hl_tt_giro.dae" />
-          </geometry>
+        <origin xyz="0 0 0" rpy="0 0 0" />
+        <geometry>
+		      <mesh filename="package://rbsherpa_hl_description/meshes/structure/rbsherpa_hl_tt_giro.dae" />
+        </geometry>
       </visual>
       <collision>
@@ -54,7 +53,7 @@
         <mass value="4.64491" />
         <origin xyz="0 0 0.004" />
-        <inertia  ixx="0.134515" ixy = "0" ixz = "0"
-                  iyy="0.0086520177" iyz = "0"
-                  izz="0.143118" />
+        <inertia  ixx="0.13451516929" ixy = "0" ixz = "0"
+                  iyy="0.00865201773" iyz = "0"
+                  izz="0.14311764130" />
       </inertial>
     </link>

File: rbsherpa_hl_description/urdf/wheels/motor_wheel.urdf.xacro (robot description, xacro)
@@ -5,56 +5,37 @@
   <xacro:property name="wheel_joint_damping" value="2.0" />
   <xacro:property name="wheel_joint_friction" value="1.0" />
-  <xacro:property name="wheel_mass" value="5.7745" /> <!-- in kg-->
-  <xacro:macro name="cylinder_inertia" params="m r h">
-    <inertia  ixx="${m*(3*r*r+h*h)/12}" ixy = "0" ixz = "0"
-              iyy="${m*(3*r*r+h*h)/12}" iyz = "0"
-              izz="${m*r*r/2}" />
-  </xacro:macro>
-  <xacro:macro name="motor_wheel" params="prefix parent *origin reflect hq">
-    <joint name="${prefix}_wheel_joint" type="continuous">
-      <parent link="${parent}"/>
-      <child link="${prefix}_wheel_link"/>
-      <xacro:insert_block name="origin" />
-      <axis xyz="0 1 0" rpy="0 0 0" />
-      <limit effort="100" velocity="100"/>
-      <joint_properties damping="${wheel_joint_damping}" friction="${wheel_joint_friction}"/>
-    </joint>
-    <link name="${prefix}_wheel_link">
-      <visual>
-        <!-- HIGH RESOLUTION WHEELS -->
-        <xacro:if value="${hq}">
-          <origin xyz="0 0 0" rpy="0 0 0" />
-          <geometry>
-			<xacro:if value="${reflect}">
-			 <mesh filename="package://rbsherpa_hl_description/meshes/wheels/rbsherpa_hl_motorwheel.dae" />
-			</xacro:if>
-			<xacro:unless value="${reflect}">
-			 <mesh filename="package://rbsherpa_hl_description/meshes/wheels/rbsherpa_hl_motorwheel.dae" />
-			</xacro:unless>
-          </geometry>
-        </xacro:if>
-       <!-- LOW RESOLUTION WHEELS -->
-        <xacro:unless value="${hq}">
-          <origin xyz="0 0 0" rpy="${M_PI/2} 0 0" />
-          <geometry>
-            <cylinder length="${wheel_height}" radius="${wheel_radius}" />
-          </geometry>
-        </xacro:unless>
-      </visual>
-      <collision>
-		<origin xyz="0 0 0" rpy="${M_PI/2} 0 0" />
-        <geometry>
-          <cylinder length="${wheel_height}" radius="${wheel_radius}" />
-        </geometry>
-      </collision>
-      <inertial>
-        <mass value="${wheel_mass}" />
-        <origin xyz="0.01608 0.01055 0" />
-        <inertia  ixx="0.09185239" ixy = "0" ixz = "0"
-                  iyy="0.05298241" iyz = "0"
-                  izz="0.05298241" />
-      </inertial>
-    </link>
-    <xacro:motor_wheel_transmission prefix="${prefix}" />
+	<xacro:property name="wheel_radius" value="0.18415" />
+	<xacro:property name="wheel_height" value="0.14" />
+  <xacro:macro name="motor_wheel" params="prefix parent *origin">
+	  <joint name="${prefix}_wheel_joint" type="continuous">
+	    <parent link="${parent}"/>
+	    <child link="${prefix}_wheel_link"/>
+	    <xacro:insert_block name="origin" />
+	    <axis xyz="0 1 0" rpy="0 0 0" />
+	    <limit effort="100" velocity="100"/>
+	    <joint_properties damping="${wheel_joint_damping}" friction="${wheel_joint_friction}"/>
+	  </joint>
+	  <link name="${prefix}_wheel_link">
+	    <visual>
+	      <origin xyz="0 0 0" rpy="0 0 0" />
+	      <geometry>
+					<mesh filename="package://rbsherpa_hl_description/meshes/wheels/rbsherpa_hl_motorwheel.dae" />
+	      </geometry>
+	    </visual>
+	    <collision>
+				<origin xyz="0 0 0" rpy="${M_PI/2} 0 0" />
+	      <geometry>
+	        <cylinder length="${wheel_height}" radius="${wheel_radius}" />
+	      </geometry>
+	    </collision>
+	    <inertial>
+	      <mass value="6.91837" />
+	      <origin xyz="0 0.00036 0" />
+	      <inertia  ixx="0.06952851" ixy = "0" ixz = "0"
+	                iyy="0.12393" iyz = "0"
+	                izz="0.0695285" />
+	    </inertial>
+	  </link>
+	  <xacro:motor_wheel_transmission prefix="${prefix}" />
   </xacro:macro>
 </robot>

File: rbsherpa_hl_description/urdf/wheels/steer_wheel.urdf.xacro (robot description, xacro)
@@ -3,12 +3,8 @@
   <xacro:include filename="$(find rbsherpa_hl_description)/urdf/wheels/steer_wheel.transmission.xacro"/>
   <xacro:property name="M_PI" value="3.1415926535897931" />
-  <!-- Wheels -->
-  <xacro:property name="wheel_radius" value="0.18415" />
-  <xacro:property name="wheel_height" value="0.14" /> <!--TODO: Unknown --> <!-- really is the wheel width -->
   <xacro:property name="steer_joint_damping" value="0.01" />
   <xacro:property name="steer_joint_friction" value="0.01" />
   <xacro:property name="steer_joint_position_limit" value="2.9" />
-  <xacro:macro name="steer_wheel" params="prefix parent *origin reflect hq">
-	<!--WHEEL TIRE -->
+  <xacro:macro name="steer_wheel" params="prefix parent *origin">
     <joint name="${prefix}_wheel_joint" type="revolute">
       <parent link="${parent}"/>
@@ -21,38 +17,21 @@
     <link name="${prefix}_wheel_link">
       <visual>
-        <!-- HIGH RESOLUTION WHEELS -->
-        <xacro:if value="${hq}">
-          <origin xyz="0 0 0" rpy="0 0 0" />
-          <geometry>
-			<xacro:if value="${reflect}">
-			 <mesh filename="package://rbsherpa_hl_description/meshes/wheels/rbsherpa_hl_wheel.dae" />
-			 <!--cylinder length="${wheel_height}" radius="${wheel_radius}" /-->
-			</xacro:if>
-			<xacro:unless value="${reflect}">
-			 <mesh filename="package://rbsherpa_hl_description/meshes/wheels/rbsherpa_hl_wheel.dae" />
-			 <!--cylinder length="${wheel_height}" radius="${wheel_radius}" /-->
-			</xacro:unless>
-          </geometry>
-        </xacro:if>
-       <!-- LOW RESOLUTION WHEELS -->
-        <xacro:unless value="${hq}">
-          <origin xyz="0 0 0" rpy="${M_PI/2} 0 0" />
-          <geometry>
-            <cylinder length="${wheel_height}" radius="${wheel_radius}" />
-          </geometry>
-        </xacro:unless>
+        <origin xyz="0 0 0" rpy="0 0 0" />
+        <geometry>
+  			  <mesh filename="package://rbsherpa_hl_description/meshes/wheels/rbsherpa_hl_wheel.dae" />
+        </geometry>
       </visual>
       <collision>
-		<origin xyz="0 0 0" rpy="0 0 0" />
+		    <origin xyz="0 0 0" rpy="0 0 0" />
         <geometry>
-			<cylinder length="0.1" radius="0.1" />
+			    <cylinder length="0.1" radius="0.1" />
         </geometry>
       </collision>
       <inertial>
-      <mass value="37.29668" />
-        <origin xyz="0.00122 -0.00633 0.07032" />
-        <inertia  ixx="0.656095" ixy = "0.0002884484" ixz = "0.0037546231"
-                  iyy="0.645381" iyz = "0.06221658"
-                  izz="0.160381" />
+        <mass value="32.81532" />
+        <origin xyz="0.00002 -0.06358 -0.18084" />
+        <inertia  ixx="0.469495" ixy = "0.0001387555" ixz = "0.00006456469"
+                  iyy="0.496194" iyz = "0.01288985"
+                  izz="0.263583" />
       </inertial>
     </link>

Commit message: Set inertias for low quality model

File: rbsherpa_hl_description/urdf/bases/rbsherpa_hl_base.urdf.xacro (robot description, xacro)
@@ -5,4 +5,9 @@
     <xacro:property name="PI" value="3.1415926535897931"/>
     <xacro:property name="wheel_width" value="0.14" />
+    <xacro:macro name="cuboid_inertia" params="m h w d">
+      <inertia  ixx="${m*(h*h+d*d)/12}" ixy = "0" ixz = "0"
+                iyy="${m*(w*w+d*d)/12}" iyz = "0"
+                izz="${m*(w*w+h*h)/12}" />
+    </xacro:macro>
     <!-- BASE FOOTPRINT -->
     <xacro:if value="${publish_bf}">
@@ -16,5 +21,4 @@
       </link>
       <joint name="${prefix}base_footprint_joint" type="fixed">
-        <!--origin xyz="0 0 ${wheel_radius - wheel_offset_z - motor_wheel_offset_z}" rpy="0 0 0" /-->
         <origin xyz="0 0 0" rpy="0 0 0" />
         <parent link="${prefix}base_footprint"/>
@@ -26,6 +30,12 @@
       <inertial>
         <mass value="381.91147" />
-        <origin xyz="0.01210 0.00057 0.41465" />
-        <inertia  ixx="66.029446" ixy="-0.05457547"  ixz="9.08271"  iyy="97.833795"  iyz="0.0012187052"  izz="79.714477" />
+        <xacro:if value="${hq}">
+          <origin xyz="0.01210 0.00057 0.41465" />
+          <inertia  ixx="66.029446" ixy="-0.05457547"  ixz="9.08271"  iyy="97.833795"  iyz="0.0012187052"  izz="79.714477" />
+        </xacro:if>
+        <xacro:unless value="${hq}">
+          <origin xyz="0 0 0.5" />
+          <cuboid_inertia  m="381.91147" h="0.925" w="1.55" d="0.5" />
+        </xacro:unless>
       </inertial>
       <visual>
@@ -42,12 +52,4 @@
           </geometry>
         </xacro:unless>
-        <!--
-        <geometry>
-          <box size="1.4 0.7 0.5" />
-        </geometry>
-        <material name="darkgrey">
-          <color rgba="0.1 0.1 0.1 1"/>
-        </material>
-        -->
       </visual>
       <collision>

File: rbsherpa_hl_description/urdf/wheels/motor_wheel.urdf.xacro (robot description, xacro)
@@ -7,4 +7,9 @@
 	<xacro:property name="wheel_radius" value="0.18415" />
 	<xacro:property name="wheel_height" value="0.14" />
+	<xacro:macro name="cylinder_inertia" params="m r h">
+		<inertia 	ixx="${m*(3*r*r+h*h)/12}" ixy = "0" ixz = "0"
+							iyy="${m*r*r/2}" iyz = "0"
+							izz="${m*(3*r*r+h*h)/12}" />
+	</xacro:macro>
   <xacro:macro name="motor_wheel" params="prefix parent *origin hq">
 	  <joint name="${prefix}_wheel_joint" type="continuous">
@@ -39,8 +44,14 @@
 	    <inertial>
 	      <mass value="6.91837" />
-	      <origin xyz="0 0.00036 0" />
-	      <inertia  ixx="0.06952851" ixy = "0" ixz = "0"
-	                iyy="0.12393" iyz = "0"
-	                izz="0.0695285" />
+				<xacro:if value="${hq}">
+		      <origin xyz="0 0.00036 0" />
+		      <inertia  ixx="0.06952851" ixy = "0" ixz = "0"
+		                iyy="0.12393" iyz = "0"
+		                izz="0.0695285" />
+				</xacro:if>
+				<xacro:unless value="${hq}">
+					<origin xyz="0 0 0" />
+	        <cylinder_inertia  m="6.91837" r="${wheel_radius}" h="${wheel_height}" />
+				</xacro:unless>
 	    </inertial>
 	  </link>

File: rbsherpa_hl_description/urdf/wheels/steer_wheel.urdf.xacro (robot description, xacro)
@@ -6,4 +6,9 @@
   <xacro:property name="steer_joint_friction" value="0.01" />
   <xacro:property name="steer_joint_position_limit" value="2.9" />
+  <xacro:macro name="cylinder_inertia" params="m r h">
+    <inertia  ixx="${m*(3*r*r+h*h)/12}" ixy = "0" ixz = "0"
+              iyy="${m*r*r/2}" iyz = "0"
+              izz="${m*(3*r*r+h*h)/12}" />
+  </xacro:macro>
   <xacro:macro name="steer_wheel" params="prefix parent *origin hq">
     <joint name="${prefix}_wheel_joint" type="revolute">
@@ -38,8 +43,14 @@
       <inertial>
         <mass value="32.81532" />
-        <origin xyz="0.00002 -0.06358 -0.18084" />
-        <inertia  ixx="0.469495" ixy = "0.0001387555" ixz = "0.00006456469"
-                  iyy="0.496194" iyz = "0.01288985"
-                  izz="0.263583" />
+        <xacro:if value="${hq}">
+          <origin xyz="0.00002 -0.06358 -0.18084" />
+          <inertia  ixx="0.469495" ixy = "0.0001387555" ixz = "0.00006456469"
+                    iyy="0.496194" iyz = "0.01288985"
+                    izz="0.263583" />
+        </xacro:if>
+        <xacro:unless value="${hq}">
+          <origin xyz="0 0 -0.18084" />
+          <cylinder_inertia  m="5" r="0.1" h="0.2" />
+        </xacro:unless>
       </inertial>
     </link>
