Commit message: Updated names of mesh files

File: rbsherpa_hl_description/urdf/bases/rbsherpa_hl_base.urdf.xacro (robot description, xacro)
@@ -21,5 +21,5 @@
       </link>
       <joint name="${prefix}base_footprint_joint" type="fixed">
-        <origin xyz="0 0 0" rpy="0 0 0" />
+        <origin xyz="0 0 ${wheel_radius}" rpy="0 0 0" />
         <parent link="${prefix}base_footprint"/>
         <child link="${prefix}base_link" />
@@ -41,7 +41,7 @@
       <visual>
         <xacro:if value="${hq}">
-          <origin xyz="0 0 0" rpy="0 0 0" />
+          <origin xyz="0 0 0" rpy="0 0 3.1415" />
           <geometry>
-            <mesh filename="package://rbsherpa_hl_description/meshes/bases/rbsherpa_hl_base.dae"/>
+            <mesh filename="package://rbsherpa_hl_description/meshes/bases/rbsherpa_hl_base_v2.dae"/>
           </geometry>
         </xacro:if>

File: rbsherpa_hl_description/urdf/structures/structure.urdf.xacro (robot description, xacro)
@@ -71,14 +71,14 @@
         <origin xyz="0 0 0" rpy="0 0 0"/>
         <geometry>
-          <mesh filename="package://vulcano_torso_description/meshes/pantilt/base.stl"/>
-        </geometry>
-       <material name="lightgrey">
-         <color rgba="0.3 0.3 0.3 1"/>
-       </material>
-      </visual>
-      <collision>
-        <origin xyz="0 0 0" rpy="0 0 0"/>
-        <geometry>
-          <mesh filename="package://vulcano_torso_description/meshes/pantilt/base.stl"/>
+          <mesh filename="package://rbsherpa_hl_description/meshes/pantilt/base.stl"/>
+        </geometry>
+       <material name="lightgrey">
+         <color rgba="0.3 0.3 0.3 1"/>
+       </material>
+      </visual>
+      <collision>
+        <origin xyz="0 0 0" rpy="0 0 0"/>
+        <geometry>
+          <mesh filename="package://rbsherpa_hl_description/meshes/pantilt/base.stl"/>
         </geometry>
       </collision>
@@ -100,14 +100,14 @@
         <origin xyz="0 0 0" rpy="0 0 0"/>
         <geometry>
-          <mesh filename="package://vulcano_torso_description/meshes/pantilt/dynamixel_l42.stl"/>
-        </geometry>
-       <material name="lightgrey">
-         <color rgba="0.3 0.3 0.3 1"/>
-       </material>
-      </visual>
-      <collision>
-        <origin xyz="0 0 0" rpy="0 0 0"/>
-        <geometry>
-          <mesh filename="package://vulcano_torso_description/meshes/pantilt/dynamixel_l42.stl"/>
+          <mesh filename="package://rbsherpa_hl_description/meshes/pantilt/dynamixel_l42.stl"/>
+        </geometry>
+       <material name="lightgrey">
+         <color rgba="0.3 0.3 0.3 1"/>
+       </material>
+      </visual>
+      <collision>
+        <origin xyz="0 0 0" rpy="0 0 0"/>
+        <geometry>
+          <mesh filename="package://rbsherpa_hl_description/meshes/pantilt/dynamixel_l42.stl"/>
         </geometry>
       </collision>
@@ -130,14 +130,14 @@
         <origin xyz="0 0 0" rpy="0 0 0"/>
         <geometry>
-          <mesh filename="package://vulcano_torso_description/meshes/pantilt/pan.stl"/>
-        </geometry>
-       <material name="lightgrey">
-         <color rgba="0.3 0.3 0.3 1"/>
-       </material>
-      </visual>
-      <collision>
-        <origin xyz="0 0 0" rpy="0 0 0"/>
-        <geometry>
-          <mesh filename="package://vulcano_torso_description/meshes/pantilt/pan.stl"/>
+          <mesh filename="package://rbsherpa_hl_description/meshes/pantilt/pan.stl"/>
+        </geometry>
+       <material name="lightgrey">
+         <color rgba="0.3 0.3 0.3 1"/>
+       </material>
+      </visual>
+      <collision>
+        <origin xyz="0 0 0" rpy="0 0 0"/>
+        <geometry>
+          <mesh filename="package://rbsherpa_hl_description/meshes/pantilt/pan.stl"/>
         </geometry>
       </collision>
@@ -161,14 +161,14 @@
         <origin xyz="0 0 0" rpy="0 0 0"/>
         <geometry>
-          <mesh filename="package://vulcano_torso_description/meshes/pantilt/dynamixel_l42.stl"/>
-        </geometry>
-       <material name="lightgrey">
-         <color rgba="0.3 0.3 0.3 1"/>
-       </material>
-      </visual>
-      <collision>
-        <origin xyz="0 0 0" rpy="0 0 0"/>
-        <geometry>
-          <mesh filename="package://vulcano_torso_description/meshes/pantilt/dynamixel_l42.stl"/>
+          <mesh filename="package://rbsherpa_hl_description/meshes/pantilt/dynamixel_l42.stl"/>
+        </geometry>
+       <material name="lightgrey">
+         <color rgba="0.3 0.3 0.3 1"/>
+       </material>
+      </visual>
+      <collision>
+        <origin xyz="0 0 0" rpy="0 0 0"/>
+        <geometry>
+          <mesh filename="package://rbsherpa_hl_description/meshes/pantilt/dynamixel_l42.stl"/>
         </geometry>
       </collision>
@@ -189,14 +189,14 @@
         <origin xyz="0 0 0" rpy="0 0 0"/>
         <geometry>
-          <mesh filename="package://vulcano_torso_description/meshes/pantilt/tilt_support.stl"/>
-        </geometry>
-       <material name="lightgrey">
-         <color rgba="0.3 0.3 0.3 1"/>
-       </material>
-      </visual>
-      <collision>
-        <origin xyz="0 0 0" rpy="0 0 0"/>
-        <geometry>
-          <mesh filename="package://vulcano_torso_description/meshes/pantilt/tilt_support.stl"/>
+          <mesh filename="package://rbsherpa_hl_description/meshes/pantilt/tilt_support.stl"/>
+        </geometry>
+       <material name="lightgrey">
+         <color rgba="0.3 0.3 0.3 1"/>
+       </material>
+      </visual>
+      <collision>
+        <origin xyz="0 0 0" rpy="0 0 0"/>
+        <geometry>
+          <mesh filename="package://rbsherpa_hl_description/meshes/pantilt/tilt_support.stl"/>
         </geometry>
       </collision>
@@ -217,14 +217,14 @@
         <origin xyz="0 0 0" rpy="0 0 0"/>
         <geometry>
-          <mesh filename="package://vulcano_torso_description/meshes/pantilt/tilt.stl"/>
-        </geometry>
-       <material name="lightgrey">
-         <color rgba="0.3 0.3 0.3 1"/>
-       </material>
-      </visual>
-      <collision>
-        <origin xyz="0 0 0" rpy="0 0 0"/>
-        <geometry>
-          <mesh filename="package://vulcano_torso_description/meshes/pantilt/tilt.stl"/>
+          <mesh filename="package://rbsherpa_hl_description/meshes/pantilt/tilt.stl"/>
+        </geometry>
+       <material name="lightgrey">
+         <color rgba="0.3 0.3 0.3 1"/>
+       </material>
+      </visual>
+      <collision>
+        <origin xyz="0 0 0" rpy="0 0 0"/>
+        <geometry>
+          <mesh filename="package://rbsherpa_hl_description/meshes/pantilt/tilt.stl"/>
         </geometry>
       </collision>
@@ -244,14 +244,14 @@
         <origin xyz="0 0 0" rpy="0 0 0"/>
         <geometry>
-          <mesh filename="package://vulcano_torso_description/meshes/pantilt/pantilt.stl"/>
-        </geometry>
-       <material name="lightgrey">
-         <color rgba="0.3 0.3 0.3 1"/>
-       </material>
-      </visual>
-      <collision>
-        <origin xyz="0 0 0" rpy="0 0 0"/>
-        <geometry>
-          <mesh filename="package://vulcano_torso_description/meshes/pantilt/pantilt.stl"/>
+          <mesh filename="package://rbsherpa_hl_description/meshes/pantilt/pantilt.stl"/>
+        </geometry>
+       <material name="lightgrey">
+         <color rgba="0.3 0.3 0.3 1"/>
+       </material>
+      </visual>
+      <collision>
+        <origin xyz="0 0 0" rpy="0 0 0"/>
+        <geometry>
+          <mesh filename="package://rbsherpa_hl_description/meshes/pantilt/pantilt.stl"/>
         </geometry>
       </collision>

File: rbsherpa_hl_description/urdf/wheels/wheel_steer.urdf.xacro (robot description, xacro)
@@ -11,6 +11,6 @@
               izz="${m*(3*r*r+h*h)/12}" />
   </xacro:macro>
-  <xacro:macro name="wheel_steer" params="prefix parent *origin hq">
-    <joint name="${prefix}_joint" type="revolute">
+  <xacro:macro name="wheel_steer" params="prefix parent *origin type hq">
+    <joint name="${prefix}_joint" type="${type}">
       <parent link="${parent}"/>
       <child link="${prefix}_link"/>
@@ -25,5 +25,5 @@
           <origin xyz="0 0 0" rpy="0 0 0" />
           <geometry>
-    			  <mesh filename="package://rbsherpa_hl_description/meshes/wheels/rbsherpa_hl_wheel_steer.dae" />
+    			  <mesh filename="package://rbsherpa_hl_description/meshes/wheels/rbsherpa_hl_steer_wheel.dae" />
           </geometry>
         </xacro:if>

File: rbsherpa_hl_description/urdf/wheels/wheel_traction.urdf.xacro (robot description, xacro)
@@ -26,5 +26,5 @@
 		      <origin xyz="0 0 0" rpy="0 0 0" />
 		      <geometry>
-						<mesh filename="package://rbsherpa_hl_description/meshes/wheels/rbsherpa_hl_wheel_traction.dae" />
+						<mesh filename="package://rbsherpa_hl_description/meshes/wheels/rbsherpa_hl_traction_wheel.dae" />
 		      </geometry>
 				</xacro:if>

Commit message: rbsherpa_hl_description:: invertial values and joint limits changed

File: rbsherpa_hl_description/urdf/bases/rbsherpa_hl_base.urdf.xacro (robot description, xacro)
@@ -5,8 +5,8 @@
     <xacro:property name="PI" value="3.1415926535897931"/>
     <xacro:property name="wheel_width" value="0.14" />
-    <xacro:macro name="cuboid_inertia" params="m h w d">
-      <inertia  ixx="${m*(h*h+d*d)/12}" ixy = "0" ixz = "0"
-                iyy="${m*(w*w+d*d)/12}" iyz = "0"
-                izz="${m*(w*w+h*h)/12}" />
+  <xacro:macro name="box_inertia" params="m x y z">
+    <inertia  ixx="${m*(y*y+z*z)/12}" ixy = "0" ixz = "0"
+              iyy="${m*(x*x+z*z)/12}" iyz = "0"
+              izz="${m*(x*x+y*y)/12}" />
     </xacro:macro>
     <!-- BASE FOOTPRINT -->
@@ -29,13 +29,7 @@
     <link name="${prefix}base_link">
       <inertial>
-        <mass value="381.91147" />
-        <xacro:if value="${hq}">
-          <origin xyz="0.01210 0.00057 0.41465" />
-          <inertia  ixx="66.029446" ixy="-0.05457547"  ixz="9.08271"  iyy="97.833795"  iyz="0.0012187052"  izz="79.714477" />
-        </xacro:if>
-        <xacro:unless value="${hq}">
-          <origin xyz="0 0 0.5" />
-          <cuboid_inertia  m="381.91147" h="0.925" w="1.55" d="0.5" />
-        </xacro:unless>
+        <mass value="600" />
+        <origin xyz="0 0 0.5" />
+        <box_inertia m="600" x="0.9" y="1.5" z="0.5"/>
       </inertial>
       <visual>

File: rbsherpa_hl_description/urdf/structures/elevator_structure.urdf.xacro (robot description, xacro)
@@ -30,7 +30,7 @@
       </collision>
       <inertial>
-        <mass value="0.005" />
-        <origin xyz="0 0 -0.27" />
-        <solid_cuboid_inertia m="0.005" h="0.05" d="0.05" w="0.05"/>
+        <mass value="1" />
+        <origin xyz="0 0 0" />
+        <solid_cuboid_inertia m="1" h="0.1" d="0.1" w="0.1"/>
       </inertial>
     </link>
@@ -41,5 +41,5 @@
       <child link="${prefix}torso_elevator_link"/>
       <axis xyz="0 0 1"/>
-      <limit lower="0.0" upper="0.5" effort="1.0" velocity="0.07"/>
+      <limit lower="0.0" upper="0.5" effort="100.0" velocity="0.07"/>
       <xacro:insert_block name="origin" />
     </joint>
@@ -58,7 +58,7 @@
       </collision>
       <inertial>
-        <mass value="0.005" />
+        <mass value="0.1" />
         <origin xyz="0 0 -0.27" />
-        <solid_cuboid_inertia m="0.005" h="0.05" d="0.05" w="0.05"/>
+        <solid_cuboid_inertia m="0.1" h="0.1" d="0.1" w="0.1"/>
       </inertial>
     </link>
@@ -78,5 +78,5 @@
       <child link="${prefix}torso_pantilt_pan_link"/>
       <axis xyz="0 0 1"/>
-      <limit lower="-3.14" upper="3.14" effort="1.0" velocity="0.1"/>
+      <limit lower="-3.14" upper="3.14" effort="10.0" velocity="0.5"/>
       <xacro:insert_block name="origin" />
     </joint>
@@ -95,7 +95,7 @@
       </collision>
       <inertial>
-        <mass value="0.005" />
-        <origin xyz="0 0 -0.27" />
-        <solid_cuboid_inertia m="0.005" h="0.05" d="0.05" w="0.05"/>
+        <mass value="0.05" />
+        <origin xyz="0 0 0" />
+        <solid_cuboid_inertia m="0.05" h="0.1" d="0.1" w="0.1"/>
       </inertial>
     </link>
@@ -123,5 +123,5 @@
       <child link="${prefix}gun_tilt_link"/>
       <axis xyz="0 1 0"/>
-      <limit lower="-0.57" upper="0.1" effort="1.0" velocity="0.5"/>
+      <limit lower="-0.57" upper="0.1" effort="10.0" velocity="0.5"/>
       <xacro:insert_block name="origin" />
     </joint>
@@ -143,7 +143,7 @@
       </collision>
       <inertial>
-        <mass value="0.005" />
-        <origin xyz="0 0 -0.27" />
-        <solid_cuboid_inertia m="0.005" h="0.05" d="0.05" w="0.05"/>
+        <mass value="0.05" />
+        <origin xyz="0 0 0" />
+        <solid_cuboid_inertia m="0.05" h="0.1" d="0.1" w="0.1"/>
       </inertial>
     </link>

File: rbsherpa_hl_description/urdf/structures/gimbal.urdf.xacro (robot description, xacro)
@@ -30,7 +30,7 @@
       </collision>
       <inertial>
-        <mass value="0.005" />
-        <origin xyz="0 0 -0.27" />
-        <solid_cuboid_inertia m="0.005" h="0.05" d="0.05" w="0.05"/>
+        <mass value="0.05" />
+        <origin xyz="0 0 0" />
+        <solid_cuboid_inertia m="0.05" h="0.1" d="0.1" w="0.1"/>
       </inertial>
     </link>
@@ -56,7 +56,7 @@
       </collision>
       <inertial>
-        <mass value="0.005" />
-        <origin xyz="0 0 -0.27" />
-        <solid_cuboid_inertia m="0.005" h="0.05" d="0.05" w="0.05"/>
+        <mass value="0.05" />
+        <origin xyz="0 0 0" />
+        <solid_cuboid_inertia m="0.05" h="0.1" d="0.1" w="0.1"/>
       </inertial>
     </link>
@@ -80,7 +80,7 @@
     <link name="${prefix}gimbal_roll_link">
       <inertial>
-        <mass value="0.005" />
-        <origin xyz="0 0 -0.27" />
-        <solid_cuboid_inertia m="0.005" h="0.05" d="0.05" w="0.05"/>
+        <mass value="0.05" />
+        <origin xyz="0 0 0" />
+        <solid_cuboid_inertia m="0.05" h="0.1" d="0.1" w="0.1"/>
       </inertial>
     </link>
@@ -104,7 +104,7 @@
     <link name="${prefix}gimbal_pitch_link">
       <inertial>
-        <mass value="0.005" />
-        <origin xyz="0 0 -0.27" />
-        <solid_cuboid_inertia m="0.005" h="0.05" d="0.05" w="0.05"/>
+        <mass value="0.05" />
+        <origin xyz="0 0 0" />
+        <solid_cuboid_inertia m="0.05" h="0.1" d="0.1" w="0.1"/>
       </inertial>
     </link>

File: rbsherpa_hl_description/urdf/wheels/wheel_steer.urdf.xacro (robot description, xacro)
@@ -17,5 +17,5 @@
       <xacro:insert_block name="origin" />
       <axis xyz="0 0 1" rpy="0 0 0" />
-      <limit effort="100" velocity="50" lower="-${steer_joint_position_limit}" upper="${steer_joint_position_limit}"/>
+      <limit effort="30.0" velocity="50.0" lower="-${steer_joint_position_limit}" upper="${steer_joint_position_limit}"/>
       <joint_properties damping="${steer_joint_damping}" friction="${steer_joint_friction}"/>
     </joint>

File: rbsherpa_hl_description/urdf/wheels/wheel_traction.urdf.xacro (robot description, xacro)
@@ -18,5 +18,5 @@
 	    <xacro:insert_block name="origin" />
 	    <axis xyz="0 1 0" rpy="0 0 0" />
-	    <limit effort="100" velocity="100"/>
+	    <limit effort="10.0" velocity="10.0"/>
 	    <joint_properties damping="${wheel_joint_damping}" friction="${wheel_joint_friction}"/>
 	  </joint>
