Commit message: URDF added to the model

File: rbsherpa_hl_description/robots/rbsherpa_hl_std.urdf.xacro (robot description, xacro)
@@ -9,5 +9,9 @@
 	<!-- Import RBSHERPA wheels -->
 	<xacro:include filename="$(find rbsherpa_hl_description)/urdf/wheels/rubber_wheel.urdf.xacro" />
-    <xacro:arg name="prefix" default="rbsherpa_hl_"/>
+	<!-- Import RBSHERPA motor wheels -->
+	<xacro:include filename="$(find rbsherpa_hl_description)/urdf/wheels/motor_rubber_wheel.urdf.xacro" />
+	<!-- Import RBSHERPA structure-->
+	<xacro:include filename="$(find rbsherpa_hl_description)/urdf/structures/structure.urdf.xacro" />
+    <xacro:arg name="prefix" default="rbsherpa_hl"/>
 	<!-- Import all available sensors -->
 	<!--xacro:include filename="$(find robotnik_sensors)/urdf/all_sensors.urdf.xacro" /-->
@@ -22,4 +26,8 @@
 	<xacro:property name="wheel_offset_y" value="0.36" />
 	<xacro:property name="wheel_offset_z" value="0.48265" />
+	<!-- Motor wheel parameters -->
+	<xacro:property name="motor_wheel_offset_x" value="0.0" />    <!-- x,y,z in translation from base_link to the center of the wheel -->
+	<xacro:property name="motor_wheel_offset_y" value="0.029" />
+	<xacro:property name="motor_wheel_offset_z" value="-0.28265" />
 	<!-- Flag to select the high or low quality model -->
 	<xacro:property name="hq" value="true" />
@@ -30,4 +38,8 @@
 	<!-- RBSherpa base -->
 	<xacro:rbsherpa_hl_base prefix="$(arg prefix)" publish_bf="true" hq="${hq}" />
+	<!-- Structure -->
+	<xacro:structure prefix="$(arg prefix)" parent="$(arg prefix)base_link">
+		<origin xyz="0.4785 0.01 2.05265" rpy="0 0 0"/>
+	</xacro:structure>
 	<!-- Gazebo ros control pluggins -->
 	<!--xacro:ros_control/-->
@@ -46,4 +58,17 @@
 		<origin xyz="-${wheel_offset_x} ${wheel_offset_y} ${wheel_offset_z}" rpy="0 0 0"/>
 	</xacro:rubber_wheel>
+	<!-- MOTOR WHEELS -->
+	<xacro:motor_rubber_wheel prefix="$(arg prefix)motor_front_right" parent="$(arg prefix)front_right_wheel_link" reflect="false" hq="${hq}">
+		<origin xyz="${motor_wheel_offset_x} -${motor_wheel_offset_y} ${motor_wheel_offset_z}" rpy="0 0 ${PI}"/>
+	</xacro:motor_rubber_wheel>
+	<xacro:motor_rubber_wheel prefix="$(arg prefix)motor_front_left" parent="$(arg prefix)front_left_wheel_link" reflect="true" hq="${hq}">
+		<origin xyz="${motor_wheel_offset_x} ${motor_wheel_offset_y} ${motor_wheel_offset_z}" rpy="0 0 0"/>
+	</xacro:motor_rubber_wheel>
+	<xacro:motor_rubber_wheel prefix="$(arg prefix)motor_back_right" parent="$(arg prefix)back_right_wheel_link" reflect="false" hq="${hq}">
+		<origin xyz="-${motor_wheel_offset_x} -${motor_wheel_offset_y} ${motor_wheel_offset_z}" rpy="0 0 ${PI}"/>
+	</xacro:motor_rubber_wheel>
+	<xacro:motor_rubber_wheel prefix="$(arg prefix)motor_back_left" parent="$(arg prefix)back_left_wheel_link" reflect="true" hq="${hq}">
+		<origin xyz="-${motor_wheel_offset_x} ${motor_wheel_offset_y} ${motor_wheel_offset_z}" rpy="0 0 0"/>
+	</xacro:motor_rubber_wheel>
 	<!-- SENSORS -->
 	<!--xacro:sensor_hokuyo_ust10lx prefix="$(arg prefix)front_laser" parent="$(arg prefix)base_link" prefix_topic="front_laser">

File: rbsherpa_hl_description/urdf/structures/structure.urdf.xacro (robot description, xacro)
@@ -0,0 +1,67 @@
+<?xml version="1.0"?>
+<robot name="rbsherpa_structure" xmlns:xacro="http://www.ros.org/wiki/xacro">
+  <xacro:property name="M_PI" value="3.1415926535897931" />
+  <!-- TODO: Modify these values -->
+  <xacro:property name="wheel_radius" value="0.125" />
+  <xacro:property name="wheel_height" value="0.14" /> <!-- really is the wheel width -->
+  <xacro:property name="wheel_mass" value="6.5" /> <!-- in kg-->
+   <xacro:macro name="cylinder_inertia" params="m r h">
+    <inertia  ixx="${m*(3*r*r+h*h)/12}" ixy = "0" ixz = "0"
+              iyy="${m*r*r/2}" iyz = "0"
+              izz="${m*(3*r*r+h*h)/12}" />
+  </xacro:macro>
+  <xacro:macro name="structure" params="prefix parent *origin">
+	<!--fixed joint -->
+    <joint name="${prefix}structure_joint" type="fixed">
+      <parent link="${parent}"/>
+      <child link="${prefix}structure_link"/>
+      <xacro:insert_block name="origin" />
+    </joint>
+    <link name="${prefix}structure_link">
+      <visual>
+        <!-- COLUMN -->
+          <origin xyz="0 0 0" rpy="0 0 0" />
+          <geometry>
+			 <mesh filename="package://rbsherpa_hl_description/meshes/structure/rbsherpa_hl_column.dae" />
+          </geometry>
+      </visual>
+      <collision>
+		<origin xyz="0 0 0" rpy="0 0 0" />
+        <geometry>
+			<mesh filename="package://rbsherpa_hl_description/meshes/structure/rbsherpa_hl_column.stl" />
+        </geometry>
+      </collision>
+      <inertial>
+        <mass value="${wheel_mass}" />
+        <origin xyz="0 0 0" />
+        <cylinder_inertia  m="${wheel_mass}" r="${wheel_radius}" h="${wheel_height}" />
+      </inertial>
+    </link>
+    <!--GIRO: fixed joint -->
+    <joint name="${prefix}platform_joint" type="fixed">
+      <parent link="${prefix}structure_link"/>
+      <origin xyz="-0.01 -0.01 0" rpy="0 0 0" />
+      <child link="${prefix}platform_link"/>
+      <xacro:insert_block name="origin" />
+    </joint>
+    <link name="${prefix}platform_link">
+      <visual>
+          <origin xyz="0 0 0" rpy="0 0 0" />
+          <geometry>
+			 <mesh filename="package://rbsherpa_hl_description/meshes/structure/rbsherpa_hl_tt_giro.dae" />
+          </geometry>
+      </visual>
+      <collision>
+		<origin xyz="0 0 0" rpy="0 0 0" />
+        <geometry>
+			<mesh filename="package://rbsherpa_hl_description/meshes/structure/rbsherpa_hl_tt_giro.stl" />
+        </geometry>
+      </collision>
+      <inertial>
+        <mass value="${wheel_mass}" />
+        <origin xyz="0 0 0" />
+        <cylinder_inertia  m="${wheel_mass}" r="${wheel_radius}" h="${wheel_height}" />
+      </inertial>
+    </link>
+  </xacro:macro>
+</robot>

File: rbsherpa_hl_description/urdf/wheels/rubber_wheel.urdf.xacro (robot description, xacro)
@@ -17,5 +17,5 @@
       <child link="${prefix}_wheel_link"/>
       <xacro:insert_block name="origin" />
-      <axis xyz="0 1 0" rpy="0 0 0" />
+      <axis xyz="0 0 1" rpy="0 0 0" />
       <limit effort="100" velocity="100"/>
       <joint_properties damping="0.0" friction="0.0"/>
@@ -28,8 +28,8 @@
           <geometry>
 			<xacro:if value="${reflect}">
-			 <mesh filename="package://rbsherpa_hl_description/meshes/wheels/rbsherpa_hl_motorwheel.dae" />
+			 <mesh filename="package://rbsherpa_hl_description/meshes/wheels/rbsherpa_hl_wheel.dae" />
 			</xacro:if>
 			<xacro:unless value="${reflect}">
-			 <mesh filename="package://rbsherpa_hl_description/meshes/wheels/rbsherpa_hl_motorwheel.dae" />
+			 <mesh filename="package://rbsherpa_hl_description/meshes/wheels/rbsherpa_hl_wheel.dae" />
 			</xacro:unless>
           </geometry>
@@ -46,5 +46,5 @@
 		<origin xyz="0 0 0" rpy="${M_PI/2} 0 0" />
         <geometry>
-          <cylinder length="${wheel_height}" radius="${wheel_radius}" />
+			<mesh filename="package://rbsherpa_hl_description/meshes/wheels/rbsherpa_hl_motorwheel.stl" />
         </geometry>
       </collision>

Commit message: Add front and rear lidar sensors

File: rbsherpa_hl_description/robots/rbsherpa_hl_std.urdf.xacro (robot description, xacro)
@@ -6,5 +6,5 @@
 	<!-- First we import all posible elements defined in the urdf.xacro files. All these elements are defined as macro:xacros -->
 	<!-- Import RBSHERPA base elements -->
-    <xacro:include filename="$(find rbsherpa_hl_description)/urdf/bases/rbsherpa_hl_base.urdf.xacro" /> <!-- v3 name from engineering department -->
+  <xacro:include filename="$(find rbsherpa_hl_description)/urdf/bases/rbsherpa_hl_base.urdf.xacro" />
 	<!-- Import RBSHERPA wheels -->
 	<xacro:include filename="$(find rbsherpa_hl_description)/urdf/wheels/rubber_wheel.urdf.xacro" />
@@ -13,7 +13,7 @@
 	<!-- Import RBSHERPA structure-->
 	<xacro:include filename="$(find rbsherpa_hl_description)/urdf/structures/structure.urdf.xacro" />
-    <xacro:arg name="prefix" default="rbsherpa_hl"/>
-	<!-- Import all available sensors -->
-	<!--xacro:include filename="$(find robotnik_sensors)/urdf/all_sensors.urdf.xacro" /-->
+  <!-- Import all available sensors -->
+  <xacro:include filename="$(find robotnik_sensors)/urdf/all_sensors.urdf.xacro" />
+  <xacro:arg name="prefix" default="rbsherpa_hl"/>
     <!-- Import Gazebo Stuff -->
     <!--xacro:include filename="$(find rbsherpa_xl_description)/urdf/common.gazebo.xacro" /-->
@@ -72,12 +72,9 @@
 	</xacro:motor_rubber_wheel>
 	<!-- SENSORS -->
-	<!--xacro:sensor_hokuyo_ust10lx prefix="$(arg prefix)front_laser" parent="$(arg prefix)base_link" prefix_topic="front_laser">
-		<origin xyz="0.223 0.0 0.159" rpy="0 3.1416 3.1416"/>
-	</xacro:sensor_hokuyo_ust10lx>
-	<xacro:sensor_imu_hector prefix="$(arg prefix)imu" parent="$(arg prefix)base_link">
-		<origin xyz="0.002 0.053 0.1485" rpy="0 0 0"/>
-	</xacro:sensor_imu_hector>
-    <xacro:sensor_orbbec_astra prefix="$(arg prefix)front_rgbd_camera" parent="$(arg prefix)base_link" prefix_topic="front_rgbd_camera">
-        <origin xyz="0.234 0.0125 0.107" rpy="0 0 0"/>
-    </xacro:sensor_orbbec_astra-->
+  <xacro:sensor_sick_s300 prefix="$(arg prefix)front_laser" parent="$(arg prefix)base_link" prefix_scan="front_laser">
+		<origin xyz="0.9285 -0.51 0.45891" rpy="0 0 ${-PI/4.0}"/>
+	</xacro:sensor_sick_s300>
+	<xacro:sensor_sick_s300 prefix="$(arg prefix)rear_laser" parent="$(arg prefix)base_link" prefix_scan="rear_laser">
+		<origin xyz="-0.9285 0.51 0.45891" rpy="0 0 ${3.0*PI/4.0}"/>
+	</xacro:sensor_sick_s300>
 </robot>

Commit message: [rbsherpa_hl_description]:added ros_control controllers

File: rbsherpa_hl_description/robots/rbsherpa_hl_std.urdf.xacro (robot description, xacro)
@@ -17,5 +17,5 @@
   <xacro:arg name="prefix" default="rbsherpa_hl"/>
     <!-- Import Gazebo Stuff -->
-    <!--xacro:include filename="$(find rbsherpa_xl_description)/urdf/common.gazebo.xacro" /-->
+    <xacro:include filename="$(find rbsherpa_hl_description)/urdf/common.gazebo.xacro" />
 	<!-- ***************** -->
 	<!-- Global parameters -->
@@ -43,5 +43,5 @@
 	</xacro:structure>
 	<!-- Gazebo ros control pluggins -->
-	<!--xacro:ros_control/-->
+	<xacro:ros_control/>
 	<!--xacro:gazebo_colors prefix="$(arg prefix)"/-->
 	<!-- WHEELS -->

File: rbsherpa_hl_description/urdf/wheels/motor_rubber_wheel.gazebo.xacro (robot description, xacro)
@@ -1,5 +1,5 @@
 <?xml version="1.0"?>
 <robot xmlns:xacro="http://www.ros.org/wiki/xacro">
-	<xacro:macro name="rubber_wheel_gazebo" params="prefix">
+	<xacro:macro name="motor_rubber_wheel_gazebo" params="prefix">
 		<gazebo reference="${prefix}_wheel_link">
 				<mu1 value="1.0"/>

File: rbsherpa_hl_description/urdf/wheels/motor_rubber_wheel.transmission.xacro (robot description, xacro)
@@ -1,6 +1,6 @@
 <?xml version="1.0"?>
 <robot xmlns:xacro="http://www.ros.org/wiki/xacro">
-<xacro:macro name="rubber_wheel_transmission" params="prefix">
-	<transmission name="${prefix}_wheel_joint_trans">
+<xacro:macro name="motor_rubber_wheel_transmission" params="prefix">
+	<transmission name="${prefix}_motor_wheel_joint_trans">
 	  <type>transmission_interface/SimpleTransmission</type>
 	  <joint name="${prefix}_wheel_joint">

File: rbsherpa_hl_description/urdf/wheels/motor_rubber_wheel.urdf.xacro (robot description, xacro)
@@ -1,4 +1,6 @@
 <?xml version="1.0"?>
 <robot name="motor_wheel" xmlns:xacro="http://www.ros.org/wiki/xacro">
+  <xacro:include filename="$(find rbsherpa_hl_description)/urdf/wheels/motor_rubber_wheel.transmission.xacro"/>
+  <xacro:include filename="$(find rbsherpa_hl_description)/urdf/wheels/motor_rubber_wheel.gazebo.xacro"/>
   <xacro:property name="M_PI" value="3.1415926535897931" />
   <!-- Wheels -->
@@ -55,4 +57,6 @@
       </inertial>
     </link>
+    <xacro:motor_rubber_wheel_transmission prefix="${prefix}" />
+	<xacro:motor_rubber_wheel_gazebo prefix="${prefix}" />
   </xacro:macro>
 </robot>

File: rbsherpa_hl_description/urdf/wheels/rubber_wheel.urdf.xacro (robot description, xacro)
@@ -1,4 +1,6 @@
 <?xml version="1.0"?>
 <robot name="wheel" xmlns:xacro="http://www.ros.org/wiki/xacro">
+  <xacro:include filename="$(find rbsherpa_hl_description)/urdf/wheels/rubber_wheel.transmission.xacro"/>
+  <xacro:include filename="$(find rbsherpa_hl_description)/urdf/wheels/rubber_wheel.gazebo.xacro"/>
   <xacro:property name="M_PI" value="3.1415926535897931" />
   <!-- Wheels -->
@@ -55,4 +57,6 @@
       </inertial>
     </link>
+    <xacro:rubber_wheel_transmission prefix="${prefix}" />
+	<xacro:rubber_wheel_gazebo prefix="${prefix}" />
   </xacro:macro>
 </robot>

Commit message: [rbsherpa_hl_description]: xacro files modified to work with ros_control

File: rbsherpa_hl_description/robots/rbsherpa_hl_std.urdf.xacro (robot description, xacro)
@@ -29,5 +29,5 @@
 	<xacro:property name="motor_wheel_offset_x" value="0.0" />    <!-- x,y,z in translation from base_link to the center of the wheel -->
 	<xacro:property name="motor_wheel_offset_y" value="0.029" />
-	<xacro:property name="motor_wheel_offset_z" value="-0.28265" />
+	<xacro:property name="motor_wheel_offset_z" value="-0.28265" /> <!-- -0.28265 -->
 	<!-- Flag to select the high or low quality model -->
 	<xacro:property name="hq" value="true" />
@@ -59,17 +59,20 @@
 	</xacro:rubber_wheel>
 	<!-- MOTOR WHEELS -->
-	<xacro:motor_rubber_wheel prefix="$(arg prefix)motor_front_right" parent="$(arg prefix)front_right_wheel_link" reflect="false" hq="${hq}">
+	<xacro:motor_rubber_wheel prefix="$(arg prefix)front_right_motor" parent="$(arg prefix)front_right_wheel_link" reflect="false" hq="${hq}">
 		<origin xyz="${motor_wheel_offset_x} -${motor_wheel_offset_y} ${motor_wheel_offset_z}" rpy="0 0 ${PI}"/>
 	</xacro:motor_rubber_wheel>
-	<xacro:motor_rubber_wheel prefix="$(arg prefix)motor_front_left" parent="$(arg prefix)front_left_wheel_link" reflect="true" hq="${hq}">
+	<xacro:motor_rubber_wheel prefix="$(arg prefix)front_left_motor" parent="$(arg prefix)front_left_wheel_link" reflect="true" hq="${hq}">
 		<origin xyz="${motor_wheel_offset_x} ${motor_wheel_offset_y} ${motor_wheel_offset_z}" rpy="0 0 0"/>
 	</xacro:motor_rubber_wheel>
-	<xacro:motor_rubber_wheel prefix="$(arg prefix)motor_back_right" parent="$(arg prefix)back_right_wheel_link" reflect="false" hq="${hq}">
+	<xacro:motor_rubber_wheel prefix="$(arg prefix)back_right_motor" parent="$(arg prefix)back_right_wheel_link" reflect="false" hq="${hq}">
 		<origin xyz="-${motor_wheel_offset_x} -${motor_wheel_offset_y} ${motor_wheel_offset_z}" rpy="0 0 ${PI}"/>
 	</xacro:motor_rubber_wheel>
-	<xacro:motor_rubber_wheel prefix="$(arg prefix)motor_back_left" parent="$(arg prefix)back_left_wheel_link" reflect="true" hq="${hq}">
+	<xacro:motor_rubber_wheel prefix="$(arg prefix)back_left_motor" parent="$(arg prefix)back_left_wheel_link" reflect="true" hq="${hq}">
 		<origin xyz="-${motor_wheel_offset_x} ${motor_wheel_offset_y} ${motor_wheel_offset_z}" rpy="0 0 0"/>
 	</xacro:motor_rubber_wheel>
 	<!-- SENSORS -->
+    <!--xacro:sensor_imu prefix="imu" parent="${prefix}base_link">
+          <origin xyz="-0.40 0.06 0.75" rpy="0 0 0"/>
+	</xacro:sensor_imu-->
     <xacro:sensor_sick_s300 prefix="$(arg prefix)front_laser" parent="$(arg prefix)base_link" prefix_topic="front_laser">
 		<origin xyz="0.9285 -0.51 0.45891" rpy="0 0 ${-PI/4.0}"/>

File: rbsherpa_hl_description/urdf/bases/rbsherpa_hl_base.urdf.xacro (robot description, xacro)
@@ -4,5 +4,5 @@
   <!-- Robot mechanical and motor parameters -->
   <xacro:property name="PI" value="3.1415926535897931"/>
-  <xacro:property name="wheel_width" value="0.175" />
+  <xacro:property name="wheel_width" value="0.14" />
   <!-- BASE FOOTPRINT -->
   <xacro:if value="${publish_bf}">

File: rbsherpa_hl_description/urdf/wheels/motor_rubber_wheel.transmission.xacro (robot description, xacro)
@@ -1,13 +1,14 @@
 <?xml version="1.0"?>
 <robot xmlns:xacro="http://www.ros.org/wiki/xacro">
+ <xacro:property name="motor_wheel_mechanical_reduction" value="1.0" />
 <xacro:macro name="motor_rubber_wheel_transmission" params="prefix">
 	<transmission name="${prefix}_motor_wheel_joint_trans">
 	  <type>transmission_interface/SimpleTransmission</type>
 	  <joint name="${prefix}_wheel_joint">
-		<hardwareInterface>hardware_interface/VelocityJointInterface</hardwareInterface>
+		<hardwareInterface>hardware_interface/PositionJointInterface</hardwareInterface>
 	  </joint>
-	  <actuator name="${prefix}_wheel_joint_motor">
-		<mechanicalReduction>1</mechanicalReduction>
-		<motorTorqueConstant>20</motorTorqueConstant>
+	  <actuator name="${prefix}_motor_wheel_joint_motor">
+		<hardwareInterface>hardware_interface/PositionActuatorInterface</hardwareInterface>
+		<mechanicalReduction>${motor_wheel_mechanical_reduction}</mechanicalReduction>
 	  </actuator>
 	 </transmission>

File: rbsherpa_hl_description/urdf/wheels/rubber_wheel.transmission.xacro (robot description, xacro)
@@ -1,4 +1,5 @@
 <?xml version="1.0"?>
 <robot xmlns:xacro="http://www.ros.org/wiki/xacro">
+<xacro:property name="wheel_mechanical_reduction" value="1.0" />
 <xacro:macro name="rubber_wheel_transmission" params="prefix">
 	<transmission name="${prefix}_wheel_joint_trans">
@@ -8,6 +9,6 @@
 	  </joint>
 	  <actuator name="${prefix}_wheel_joint_motor">
-		<mechanicalReduction>1</mechanicalReduction>
-		<motorTorqueConstant>20</motorTorqueConstant>
+		<hardwareInterface>hardware_interface/VelocityActuatorInterface</hardwareInterface>
+		<mechanicalReduction>${wheel_mechanical_reduction}</mechanicalReduction>
 	  </actuator>
 	 </transmission>

File: rbsherpa_hl_description/urdf/wheels/rubber_wheel.urdf.xacro (robot description, xacro)
@@ -5,5 +5,5 @@
   <xacro:property name="M_PI" value="3.1415926535897931" />
   <!-- Wheels -->
-  <xacro:property name="wheel_radius" value="0.3683" />
+  <xacro:property name="wheel_radius" value="0.18415" />
   <xacro:property name="wheel_height" value="0.14" /> <!--TODO: Unknown --> <!-- really is the wheel width -->
   <xacro:property name="wheel_mass" value="5.7745" /> <!-- in kg-->
@@ -41,7 +41,7 @@
       </visual>
       <collision>
-		<origin xyz="0 0 0" rpy="${M_PI/2} 0 0" />
+		<origin xyz="0 0 0" rpy="0 0 0" />
         <geometry>
-			<mesh filename="package://rbsherpa_hl_description/meshes/wheels/rbsherpa_hl_motorwheel.stl" />
+			<mesh filename="package://rbsherpa_hl_description/meshes/wheels/rbsherpa_hl_wheel.stl" />
         </geometry>
       </collision>

Commit message: [rbsherpa_hl_description]:ros_controllers corrected

File: rbsherpa_hl_description/robots/rbsherpa_hl_std.urdf.xacro (robot description, xacro)
@@ -29,5 +29,5 @@
 	<xacro:property name="motor_wheel_offset_x" value="0.0" />    <!-- x,y,z in translation from base_link to the center of the wheel -->
 	<xacro:property name="motor_wheel_offset_y" value="0.029" />
-	<xacro:property name="motor_wheel_offset_z" value="-0.28265" /> <!-- -0.28265 -->
+	<xacro:property name="motor_wheel_offset_z" value="-0.2985" />
 	<!-- Flag to select the high or low quality model -->
 	<xacro:property name="hq" value="true" />

File: rbsherpa_hl_description/urdf/bases/rbsherpa_hl_base.urdf.xacro (robot description, xacro)
@@ -16,5 +16,6 @@
     </link>
     <joint name="${prefix}base_footprint_joint" type="fixed">
-       <origin xyz="0 0 ${wheel_radius - wheel_offset_z - motor_wheel_offset_z}" rpy="0 0 0" />
+       <!--origin xyz="0 0 ${wheel_radius - wheel_offset_z - motor_wheel_offset_z}" rpy="0 0 0" /-->
+       <origin xyz="0 0 0" rpy="0 0 0" />
       <parent link="${prefix}base_footprint"/>
       <child link="${prefix}base_link" />

File: rbsherpa_hl_description/urdf/wheels/motor_rubber_wheel.transmission.xacro (robot description, xacro)
@@ -6,8 +6,8 @@
 	  <type>transmission_interface/SimpleTransmission</type>
 	  <joint name="${prefix}_wheel_joint">
-		<hardwareInterface>hardware_interface/PositionJointInterface</hardwareInterface>
+		<hardwareInterface>hardware_interface/VelocityJointInterface</hardwareInterface>
 	  </joint>
 	  <actuator name="${prefix}_motor_wheel_joint_motor">
-		<hardwareInterface>hardware_interface/PositionActuatorInterface</hardwareInterface>
+		<hardwareInterface>hardware_interface/VelocityActuatorInterface</hardwareInterface>
 		<mechanicalReduction>${motor_wheel_mechanical_reduction}</mechanicalReduction>
 	  </actuator>

File: rbsherpa_hl_description/urdf/wheels/rubber_wheel.transmission.xacro (robot description, xacro)
@@ -6,8 +6,8 @@
 	  <type>transmission_interface/SimpleTransmission</type>
 	  <joint name="${prefix}_wheel_joint">
-		<hardwareInterface>hardware_interface/VelocityJointInterface</hardwareInterface>
+		<hardwareInterface>hardware_interface/PositionJointInterface</hardwareInterface>
 	  </joint>
 	  <actuator name="${prefix}_wheel_joint_motor">
-		<hardwareInterface>hardware_interface/VelocityActuatorInterface</hardwareInterface>
+		<hardwareInterface>hardware_interface/PositionActuatorInterface</hardwareInterface>
 		<mechanicalReduction>${wheel_mechanical_reduction}</mechanicalReduction>
 	  </actuator>
