Commit message: joint names modified

File: rbsherpa_hl_description/robots/rbsherpa_hl_std.urdf.xacro (robot description, xacro)
@@ -8,7 +8,7 @@
   <xacro:include filename="$(find rbsherpa_hl_description)/urdf/bases/rbsherpa_hl_base.urdf.xacro" />
 	<!-- Import RBSHERPA wheels -->
-	<xacro:include filename="$(find rbsherpa_hl_description)/urdf/wheels/rubber_wheel.urdf.xacro" />
+	<xacro:include filename="$(find rbsherpa_hl_description)/urdf/wheels/steer_wheel.urdf.xacro" />
 	<!-- Import RBSHERPA motor wheels -->
-	<xacro:include filename="$(find rbsherpa_hl_description)/urdf/wheels/motor_rubber_wheel.urdf.xacro" />
+	<xacro:include filename="$(find rbsherpa_hl_description)/urdf/wheels/motor_wheel.urdf.xacro" />
 	<!-- Import RBSHERPA structure-->
 	<xacro:include filename="$(find rbsherpa_hl_description)/urdf/structures/structure.urdf.xacro" />
@@ -39,36 +39,50 @@
 	<xacro:rbsherpa_hl_base prefix="$(arg prefix)" publish_bf="true" hq="${hq}" />
 	<!-- Structure -->
-	<xacro:structure prefix="$(arg prefix)" parent="$(arg prefix)base_link">
+	<!--xacro:structure prefix="$(arg prefix)" parent="$(arg prefix)base_link">
 		<origin xyz="0.4785 0.01 2.05265" rpy="0 0 0"/>
-	</xacro:structure>
+	</xacro:structure-->
 	<!-- Gazebo ros control pluggins -->
 	<xacro:ros_control/>
 	<!--xacro:gazebo_colors prefix="$(arg prefix)"/-->
 	<!-- WHEELS -->
-	<xacro:rubber_wheel prefix="$(arg prefix)front_right" parent="$(arg prefix)base_link" reflect="false" hq="${hq}">
+	<xacro:steer_wheel prefix="$(arg prefix)front_right_steer" parent="$(arg prefix)base_link" reflect="false" hq="${hq}">
 		<origin xyz="${wheel_offset_x} -${wheel_offset_y} ${wheel_offset_z}" rpy="0 0 0"/>
-	</xacro:rubber_wheel>
-	<xacro:rubber_wheel prefix="$(arg prefix)front_left" parent="$(arg prefix)base_link" reflect="true" hq="${hq}">
+	</xacro:steer_wheel>
+	<xacro:steer_wheel prefix="$(arg prefix)front_left_steer" parent="$(arg prefix)base_link" reflect="true" hq="${hq}">
 		<origin xyz="${wheel_offset_x} ${wheel_offset_y} ${wheel_offset_z}" rpy="0 0 0"/>
-	</xacro:rubber_wheel>
-	<xacro:rubber_wheel prefix="$(arg prefix)back_right" parent="$(arg prefix)base_link" reflect="false" hq="${hq}">
+	</xacro:steer_wheel>
+	<xacro:steer_wheel prefix="$(arg prefix)back_right_steer" parent="$(arg prefix)base_link" reflect="false" hq="${hq}">
 		<origin xyz="-${wheel_offset_x} -${wheel_offset_y} ${wheel_offset_z}" rpy="0 0 0"/>
-	</xacro:rubber_wheel>
-	<xacro:rubber_wheel prefix="$(arg prefix)back_left" parent="$(arg prefix)base_link" reflect="true" hq="${hq}">
+	</xacro:steer_wheel>
+	<xacro:steer_wheel prefix="$(arg prefix)back_left_steer" parent="$(arg prefix)base_link" reflect="true" hq="${hq}">
 		<origin xyz="-${wheel_offset_x} ${wheel_offset_y} ${wheel_offset_z}" rpy="0 0 0"/>
-	</xacro:rubber_wheel>
+	</xacro:steer_wheel>
 	<!-- MOTOR WHEELS -->
-	<xacro:motor_rubber_wheel prefix="$(arg prefix)front_right_motor" parent="$(arg prefix)front_right_wheel_link" reflect="false" hq="${hq}">
+	<xacro:motor_wheel prefix="$(arg prefix)front_right_motor" parent="$(arg prefix)front_right_steer_wheel_link" reflect="false" hq="${hq}">
 		<origin xyz="${motor_wheel_offset_x} -${motor_wheel_offset_y} ${motor_wheel_offset_z}" rpy="0 0 ${PI}"/>
-	</xacro:motor_rubber_wheel>
-	<xacro:motor_rubber_wheel prefix="$(arg prefix)front_left_motor" parent="$(arg prefix)front_left_wheel_link" reflect="true" hq="${hq}">
+	</xacro:motor_wheel>
+	<xacro:motor_wheel prefix="$(arg prefix)front_left_motor" parent="$(arg prefix)front_left_steer_wheel_link" reflect="true" hq="${hq}">
 		<origin xyz="${motor_wheel_offset_x} ${motor_wheel_offset_y} ${motor_wheel_offset_z}" rpy="0 0 0"/>
-	</xacro:motor_rubber_wheel>
-	<xacro:motor_rubber_wheel prefix="$(arg prefix)back_right_motor" parent="$(arg prefix)back_right_wheel_link" reflect="false" hq="${hq}">
+	</xacro:motor_wheel>
+	<xacro:motor_wheel prefix="$(arg prefix)back_right_motor" parent="$(arg prefix)back_right_steer_wheel_link" reflect="false" hq="${hq}">
 		<origin xyz="-${motor_wheel_offset_x} -${motor_wheel_offset_y} ${motor_wheel_offset_z}" rpy="0 0 ${PI}"/>
-	</xacro:motor_rubber_wheel>
-	<xacro:motor_rubber_wheel prefix="$(arg prefix)back_left_motor" parent="$(arg prefix)back_left_wheel_link" reflect="true" hq="${hq}">
+	</xacro:motor_wheel>
+	<xacro:motor_wheel prefix="$(arg prefix)back_left_motor" parent="$(arg prefix)back_left_steer_wheel_link" reflect="true" hq="${hq}">
 		<origin xyz="-${motor_wheel_offset_x} ${motor_wheel_offset_y} ${motor_wheel_offset_z}" rpy="0 0 0"/>
-	</xacro:motor_rubber_wheel>
+	</xacro:motor_wheel>
+<!--
+	<xacro:motor_wheel prefix="$(arg prefix)front_right_motor" parent="$(arg prefix)base_link" reflect="false" hq="${hq}">
+		<origin xyz="${motor_wheel_offset_x} -${motor_wheel_offset_y} ${motor_wheel_offset_z}" rpy="0 0 ${PI}"/>
+	</xacro:motor_wheel>
+	<xacro:motor_wheel prefix="$(arg prefix)front_left_motor" parent="$(arg prefix)base_link" reflect="true" hq="${hq}">
+		<origin xyz="${motor_wheel_offset_x} ${motor_wheel_offset_y} ${motor_wheel_offset_z}" rpy="0 0 0"/>
+	</xacro:motor_wheel>
+	<xacro:motor_wheel prefix="$(arg prefix)back_right_motor" parent="$(arg prefix)base_link" reflect="false" hq="${hq}">
+		<origin xyz="-${motor_wheel_offset_x} -${motor_wheel_offset_y} ${motor_wheel_offset_z}" rpy="0 0 ${PI}"/>
+	</xacro:motor_wheel>
+	<xacro:motor_wheel prefix="$(arg prefix)back_left_motor" parent="$(arg prefix)base_link" reflect="true" hq="${hq}">
+		<origin xyz="-${motor_wheel_offset_x} ${motor_wheel_offset_y} ${motor_wheel_offset_z}" rpy="0 0 0"/>
+	</xacro:motor_wheel>
+-->
 	<!-- SENSORS -->
     <!--xacro:sensor_imu prefix="imu" parent="${prefix}base_link">

File: rbsherpa_hl_description/urdf/bases/rbsherpa_hl_base.urdf.xacro (robot description, xacro)
@@ -41,4 +41,6 @@
        </geometry>
        </xacro:unless>
+ <geometry>
+<box size="1.4 0.7 0.5" /></geometry>
        <material name="darkgrey">
          <color rgba="0.1 0.1 0.1 1"/>
@@ -46,7 +48,8 @@
     </visual>
     <collision>
-       <origin xyz="0 0 0" rpy="0 0 0 " />
+       <origin xyz="0 0 0.6" rpy="0 0 0 " />
        <geometry>
-         <mesh filename="package://rbsherpa_hl_description/meshes/bases/rbsherpa_hl_base.dae"/>
+         <!--mesh filename="package://rbsherpa_hl_description/meshes/bases/rbsherpa_hl_base.dae"/-->
+			<box size="1.4 0.6 0.5" />
        </geometry>
     </collision>

File: rbsherpa_hl_description/urdf/wheels/motor_wheel.transmission.xacro (robot description, xacro)
@@ -2,5 +2,5 @@
 <robot xmlns:xacro="http://www.ros.org/wiki/xacro">
  <xacro:property name="motor_wheel_mechanical_reduction" value="1.0" />
-<xacro:macro name="motor_rubber_wheel_transmission" params="prefix">
+<xacro:macro name="motor_wheel_transmission" params="prefix">
 	<transmission name="${prefix}_motor_wheel_joint_trans">
 	  <type>transmission_interface/SimpleTransmission</type>

File: rbsherpa_hl_description/urdf/wheels/motor_wheel.urdf.xacro (robot description, xacro)
@@ -1,8 +1,15 @@
 <?xml version="1.0"?>
 <robot name="motor_wheel" xmlns:xacro="http://www.ros.org/wiki/xacro">
-  <xacro:include filename="$(find rbsherpa_hl_description)/urdf/wheels/motor_rubber_wheel.transmission.xacro"/>
-  <xacro:include filename="$(find rbsherpa_hl_description)/urdf/wheels/motor_rubber_wheel.gazebo.xacro"/>
+  <xacro:include filename="$(find rbsherpa_hl_description)/urdf/wheels/motor_wheel.transmission.xacro"/>
   <xacro:property name="M_PI" value="3.1415926535897931" />
-  <xacro:macro name="motor_rubber_wheel" params="prefix parent *origin reflect hq">
+  <xacro:property name="wheel_joint_damping" value="2.0" />
+  <xacro:property name="wheel_joint_friction" value="1.0" />
+  <xacro:property name="wheel_mass" value="5.7745" /> <!-- in kg-->
+  <xacro:macro name="cylinder_inertia" params="m r h">
+    <inertia  ixx="${m*(3*r*r+h*h)/12}" ixy = "0" ixz = "0"
+              iyy="${m*(3*r*r+h*h)/12}" iyz = "0"
+              izz="${m*r*r/2}" />
+  </xacro:macro>
+  <xacro:macro name="motor_wheel" params="prefix parent *origin reflect hq">
     <joint name="${prefix}_wheel_joint" type="continuous">
       <parent link="${parent}"/>
@@ -11,5 +18,5 @@
       <axis xyz="0 1 0" rpy="0 0 0" />
       <limit effort="100" velocity="100"/>
-      <joint_properties damping="0.0" friction="0.0"/>
+      <joint_properties damping="${wheel_joint_damping}" friction="${wheel_joint_friction}"/>
     </joint>
     <link name="${prefix}_wheel_link">
@@ -42,13 +49,12 @@
       </collision>
       <inertial>
-        <mass value="37.29668" />
-        <origin xyz="0.00122 -0.00633 0.07032" />
-        <inertia  ixx="0.656095" ixy = "0.0002884484" ixz = "0.0037546231"
-                  iyy="0.645381" iyz = "0.06221658"
-                  izz="0.160381" />
+        <mass value="${wheel_mass}" />
+        <origin xyz="0.01608 0.01055 0" />
+        <inertia  ixx="0.09185239" ixy = "0" ixz = "0"
+                  iyy="0.05298241" iyz = "0"
+                  izz="0.05298241" />
       </inertial>
     </link>
-    <xacro:motor_rubber_wheel_transmission prefix="${prefix}" />
-	<xacro:motor_rubber_wheel_gazebo prefix="${prefix}" />
+    <xacro:motor_wheel_transmission prefix="${prefix}" />
   </xacro:macro>
 </robot>

File: rbsherpa_hl_description/urdf/wheels/steer_wheel.urdf.xacro (robot description, xacro)
@@ -1,14 +1,13 @@
 <?xml version="1.0"?>
-<robot name="wheel" xmlns:xacro="http://www.ros.org/wiki/xacro">
-  <xacro:include filename="$(find rbsherpa_hl_description)/urdf/wheels/rubber_wheel.transmission.xacro"/>
-  <xacro:include filename="$(find rbsherpa_hl_description)/urdf/wheels/rubber_wheel.gazebo.xacro"/>
+<robot name="steer_wheel" xmlns:xacro="http://www.ros.org/wiki/xacro">
+  <xacro:include filename="$(find rbsherpa_hl_description)/urdf/wheels/steer_wheel.transmission.xacro"/>
   <xacro:property name="M_PI" value="3.1415926535897931" />
   <!-- Wheels -->
   <xacro:property name="wheel_radius" value="0.18415" />
   <xacro:property name="wheel_height" value="0.14" /> <!--TODO: Unknown --> <!-- really is the wheel width -->
-  <xacro:property name="wheel_mass" value="5.7745" /> <!-- in kg-->
-  <xacro:property name="steer_joint_damping" value="2.0" />
-  <xacro:property name="steer_joint_friction" value="1.0" />
-  <xacro:macro name="rubber_wheel" params="prefix parent *origin reflect hq">
+  <xacro:property name="steer_joint_damping" value="0.01" />
+  <xacro:property name="steer_joint_friction" value="0.01" />
+  <xacro:property name="steer_joint_position_limit" value="2.9" />
+  <xacro:macro name="steer_wheel" params="prefix parent *origin reflect hq">
 	<!--WHEEL TIRE -->
     <joint name="${prefix}_wheel_joint" type="revolute">
@@ -17,5 +16,5 @@
       <xacro:insert_block name="origin" />
       <axis xyz="0 0 1" rpy="0 0 0" />
-      <limit effort="100" velocity="100"/>
+      <limit effort="100" velocity="50" lower="-${steer_joint_position_limit}" upper="${steer_joint_position_limit}"/>
       <joint_properties damping="${steer_joint_damping}" friction="${steer_joint_friction}"/>
     </joint>
@@ -27,10 +26,10 @@
           <geometry>
 			<xacro:if value="${reflect}">
-			 <!--mesh filename="package://rbsherpa_hl_description/meshes/wheels/rbsherpa_hl_wheel.dae" /-->
-			 <cylinder length="${wheel_height}" radius="${wheel_radius}" />
+			 <mesh filename="package://rbsherpa_hl_description/meshes/wheels/rbsherpa_hl_wheel.dae" />
+			 <!--cylinder length="${wheel_height}" radius="${wheel_radius}" /-->
 			</xacro:if>
 			<xacro:unless value="${reflect}">
-			 <!--mesh filename="package://rbsherpa_hl_description/meshes/wheels/rbsherpa_hl_wheel.dae" /-->
-			 <cylinder length="${wheel_height}" radius="${wheel_radius}" />
+			 <mesh filename="package://rbsherpa_hl_description/meshes/wheels/rbsherpa_hl_wheel.dae" />
+			 <!--cylinder length="${wheel_height}" radius="${wheel_radius}" /-->
 			</xacro:unless>
           </geometry>
@@ -51,13 +50,12 @@
       </collision>
       <inertial>
-        <mass value="${wheel_mass}" />
-        <origin xyz="0.01608 0.01055 0" />
-        <inertia  ixx="0.09185239" ixy = "0" ixz = "0"
-                  iyy="0.05298241" iyz = "0"
-                  izz="0.05298241" />
+      <mass value="37.29668" />
+        <origin xyz="0.00122 -0.00633 0.07032" />
+        <inertia  ixx="0.656095" ixy = "0.0002884484" ixz = "0.0037546231"
+                  iyy="0.645381" iyz = "0.06221658"
+                  izz="0.160381" />
       </inertial>
     </link>
-    <xacro:rubber_wheel_transmission prefix="${prefix}" />
-	<!--xacro:rubber_wheel_gazebo prefix="${prefix}" /-->
+    <xacro:steer_wheel_transmission prefix="${prefix}" />
   </xacro:macro>
 </robot>

Commit message: Update robot model

File: rbsherpa_hl_description/robots/rbsherpa_hl_std.urdf.xacro (robot description, xacro)
@@ -16,6 +16,6 @@
   <xacro:include filename="$(find robotnik_sensors)/urdf/all_sensors.urdf.xacro" />
   <xacro:arg name="prefix" default="rbsherpa_hl"/>
-    <!-- Import Gazebo Stuff -->
-    <xacro:include filename="$(find rbsherpa_hl_description)/urdf/common.gazebo.xacro" />
+  <!-- Import Gazebo Stuff -->
+  <xacro:include filename="$(find rbsherpa_hl_description)/urdf/common.gazebo.xacro" />
 	<!-- ***************** -->
 	<!-- Global parameters -->
@@ -23,11 +23,11 @@
 	<xacro:property name="PI" value="3.1415926535897931"/>
 	<!-- Wheel parameters -->
-	<xacro:property name="wheel_offset_x" value="0.7115" />    <!-- x,y,z in translation from base_link to the center of the wheel -->
-	<xacro:property name="wheel_offset_y" value="0.36" />
-	<xacro:property name="wheel_offset_z" value="0.48265" />
+	<xacro:property name="steer_wheel_offset_x" value="0.6236" />    <!-- x,y,z in translation from base_link to the center of the wheel -->
+	<xacro:property name="steer_wheel_offset_y" value="0.36063" />
+	<xacro:property name="steer_wheel_offset_z" value="0.28762" />
 	<!-- Motor wheel parameters -->
 	<xacro:property name="motor_wheel_offset_x" value="0.0" />    <!-- x,y,z in translation from base_link to the center of the wheel -->
 	<xacro:property name="motor_wheel_offset_y" value="0.029" />
-	<xacro:property name="motor_wheel_offset_z" value="-0.2985" />
+	<xacro:property name="motor_wheel_offset_z" value="-0.28762" />
 	<!-- Flag to select the high or low quality model -->
 	<xacro:property name="hq" value="true" />
@@ -45,28 +45,28 @@
 	<xacro:ros_control/>
 	<!--xacro:gazebo_colors prefix="$(arg prefix)"/-->
-	<!-- WHEELS -->
-	<xacro:steer_wheel prefix="$(arg prefix)front_right_steer" parent="$(arg prefix)base_link" reflect="false" hq="${hq}">
-		<origin xyz="${wheel_offset_x} -${wheel_offset_y} ${wheel_offset_z}" rpy="0 0 0"/>
+	<!-- STEER WHEELS -->
+	<xacro:steer_wheel prefix="$(arg prefix)front_right_steer" parent="$(arg prefix)base_link">
+		<origin xyz="${steer_wheel_offset_x} -${steer_wheel_offset_y} ${steer_wheel_offset_z}" rpy="0 0 0"/>
 	</xacro:steer_wheel>
-	<xacro:steer_wheel prefix="$(arg prefix)front_left_steer" parent="$(arg prefix)base_link" reflect="true" hq="${hq}">
-		<origin xyz="${wheel_offset_x} ${wheel_offset_y} ${wheel_offset_z}" rpy="0 0 0"/>
+	<xacro:steer_wheel prefix="$(arg prefix)front_left_steer" parent="$(arg prefix)base_link">
+		<origin xyz="${steer_wheel_offset_x} ${steer_wheel_offset_y} ${steer_wheel_offset_z}" rpy="0 0 0"/>
 	</xacro:steer_wheel>
-	<xacro:steer_wheel prefix="$(arg prefix)back_right_steer" parent="$(arg prefix)base_link" reflect="false" hq="${hq}">
-		<origin xyz="-${wheel_offset_x} -${wheel_offset_y} ${wheel_offset_z}" rpy="0 0 0"/>
+	<xacro:steer_wheel prefix="$(arg prefix)back_right_steer" parent="$(arg prefix)base_link">
+		<origin xyz="-${steer_wheel_offset_x} -${steer_wheel_offset_y} ${steer_wheel_offset_z}" rpy="0 0 0"/>
 	</xacro:steer_wheel>
-	<xacro:steer_wheel prefix="$(arg prefix)back_left_steer" parent="$(arg prefix)base_link" reflect="true" hq="${hq}">
-		<origin xyz="-${wheel_offset_x} ${wheel_offset_y} ${wheel_offset_z}" rpy="0 0 0"/>
+	<xacro:steer_wheel prefix="$(arg prefix)back_left_steer" parent="$(arg prefix)base_link">
+		<origin xyz="-${steer_wheel_offset_x} ${steer_wheel_offset_y} ${steer_wheel_offset_z}" rpy="0 0 0"/>
 	</xacro:steer_wheel>
 	<!-- MOTOR WHEELS -->
-	<xacro:motor_wheel prefix="$(arg prefix)front_right_motor" parent="$(arg prefix)front_right_steer_wheel_link" reflect="false" hq="${hq}">
+	<xacro:motor_wheel prefix="$(arg prefix)front_right_motor" parent="$(arg prefix)front_right_steer_wheel_link">
 		<origin xyz="${motor_wheel_offset_x} -${motor_wheel_offset_y} ${motor_wheel_offset_z}" rpy="0 0 ${PI}"/>
 	</xacro:motor_wheel>
-	<xacro:motor_wheel prefix="$(arg prefix)front_left_motor" parent="$(arg prefix)front_left_steer_wheel_link" reflect="true" hq="${hq}">
+	<xacro:motor_wheel prefix="$(arg prefix)front_left_motor" parent="$(arg prefix)front_left_steer_wheel_link">
 		<origin xyz="${motor_wheel_offset_x} ${motor_wheel_offset_y} ${motor_wheel_offset_z}" rpy="0 0 0"/>
 	</xacro:motor_wheel>
-	<xacro:motor_wheel prefix="$(arg prefix)back_right_motor" parent="$(arg prefix)back_right_steer_wheel_link" reflect="false" hq="${hq}">
+	<xacro:motor_wheel prefix="$(arg prefix)back_right_motor" parent="$(arg prefix)back_right_steer_wheel_link">
 		<origin xyz="-${motor_wheel_offset_x} -${motor_wheel_offset_y} ${motor_wheel_offset_z}" rpy="0 0 ${PI}"/>
 	</xacro:motor_wheel>
-	<xacro:motor_wheel prefix="$(arg prefix)back_left_motor" parent="$(arg prefix)back_left_steer_wheel_link" reflect="true" hq="${hq}">
+	<xacro:motor_wheel prefix="$(arg prefix)back_left_motor" parent="$(arg prefix)back_left_steer_wheel_link">
 		<origin xyz="-${motor_wheel_offset_x} ${motor_wheel_offset_y} ${motor_wheel_offset_z}" rpy="0 0 0"/>
 	</xacro:motor_wheel>
@@ -90,8 +90,8 @@
 	</xacro:sensor_imu-->
     <xacro:sensor_sick_s300 prefix="$(arg prefix)front_laser" parent="$(arg prefix)base_link" prefix_topic="front_laser">
-		<origin xyz="0.9285 -0.51 0.45891" rpy="0 0 ${-PI/4.0}"/>
+		<origin xyz="0.81495 -0.53572 0.28772" rpy="0 0 ${-PI/4.0}"/>
 	</xacro:sensor_sick_s300>
 	<xacro:sensor_sick_s300 prefix="$(arg prefix)rear_laser" parent="$(arg prefix)base_link" prefix_topic="rear_laser">
-		<origin xyz="-0.9285 0.51 0.45891" rpy="0 0 ${3.0*PI/4.0}"/>
+		<origin xyz="-0.81495 0.53572 0.28772" rpy="0 0 ${3.0*PI/4.0}"/>
 	</xacro:sensor_sick_s300>
 </robot>
