Commit message: Define both hq and lq models

File: rbsherpa_hl_description/robots/rbsherpa_hl_std.urdf.xacro (robot description, xacro)
@@ -16,4 +16,5 @@
   <xacro:include filename="$(find robotnik_sensors)/urdf/all_sensors.urdf.xacro" />
   <xacro:arg name="prefix" default="rbsherpa_hl"/>
+	<xacro:arg name="hq" default="false"/>
   <!-- Import Gazebo Stuff -->
   <xacro:include filename="$(find rbsherpa_hl_description)/urdf/common.gazebo.xacro" />
@@ -30,6 +31,4 @@
 	<xacro:property name="motor_wheel_offset_y" value="0.029" />
 	<xacro:property name="motor_wheel_offset_z" value="-0.28762" />
-	<!-- Flag to select the high or low quality model -->
-	<xacro:property name="hq" value="true" />
 	<!-- *************** -->
 	<!-- Robots Elements -->
@@ -37,5 +36,5 @@
 	<!-- Here we create the robot elements using the xacro:macros imported at the beggining of this file -->
 	<!-- RBSherpa base -->
-	<xacro:rbsherpa_hl_base prefix="$(arg prefix)" publish_bf="true" hq="${hq}" />
+	<xacro:rbsherpa_hl_base prefix="$(arg prefix)" publish_bf="true" hq="$(arg hq)" />
 	<!-- Structure -->
 	<!--xacro:structure prefix="$(arg prefix)" parent="$(arg prefix)base_link">
@@ -46,43 +45,29 @@
 	<!--xacro:gazebo_colors prefix="$(arg prefix)"/-->
 	<!-- STEER WHEELS -->
-	<xacro:steer_wheel prefix="$(arg prefix)front_right_steer" parent="$(arg prefix)base_link">
+	<xacro:steer_wheel prefix="$(arg prefix)front_right_steer" parent="$(arg prefix)base_link" hq="$(arg hq)">
 		<origin xyz="${steer_wheel_offset_x} -${steer_wheel_offset_y} ${steer_wheel_offset_z}" rpy="0 0 0"/>
 	</xacro:steer_wheel>
-	<xacro:steer_wheel prefix="$(arg prefix)front_left_steer" parent="$(arg prefix)base_link">
+	<xacro:steer_wheel prefix="$(arg prefix)front_left_steer" parent="$(arg prefix)base_link" hq="$(arg hq)">
 		<origin xyz="${steer_wheel_offset_x} ${steer_wheel_offset_y} ${steer_wheel_offset_z}" rpy="0 0 0"/>
 	</xacro:steer_wheel>
-	<xacro:steer_wheel prefix="$(arg prefix)back_right_steer" parent="$(arg prefix)base_link">
+	<xacro:steer_wheel prefix="$(arg prefix)back_right_steer" parent="$(arg prefix)base_link" hq="$(arg hq)">
 		<origin xyz="-${steer_wheel_offset_x} -${steer_wheel_offset_y} ${steer_wheel_offset_z}" rpy="0 0 0"/>
 	</xacro:steer_wheel>
-	<xacro:steer_wheel prefix="$(arg prefix)back_left_steer" parent="$(arg prefix)base_link">
+	<xacro:steer_wheel prefix="$(arg prefix)back_left_steer" parent="$(arg prefix)base_link" hq="$(arg hq)">
 		<origin xyz="-${steer_wheel_offset_x} ${steer_wheel_offset_y} ${steer_wheel_offset_z}" rpy="0 0 0"/>
 	</xacro:steer_wheel>
 	<!-- MOTOR WHEELS -->
-	<xacro:motor_wheel prefix="$(arg prefix)front_right_motor" parent="$(arg prefix)front_right_steer_wheel_link">
+	<xacro:motor_wheel prefix="$(arg prefix)front_right_motor" parent="$(arg prefix)front_right_steer_wheel_link" hq="$(arg hq)">
 		<origin xyz="${motor_wheel_offset_x} -${motor_wheel_offset_y} ${motor_wheel_offset_z}" rpy="0 0 ${PI}"/>
 	</xacro:motor_wheel>
-	<xacro:motor_wheel prefix="$(arg prefix)front_left_motor" parent="$(arg prefix)front_left_steer_wheel_link">
+	<xacro:motor_wheel prefix="$(arg prefix)front_left_motor" parent="$(arg prefix)front_left_steer_wheel_link" hq="$(arg hq)">
 		<origin xyz="${motor_wheel_offset_x} ${motor_wheel_offset_y} ${motor_wheel_offset_z}" rpy="0 0 0"/>
 	</xacro:motor_wheel>
-	<xacro:motor_wheel prefix="$(arg prefix)back_right_motor" parent="$(arg prefix)back_right_steer_wheel_link">
+	<xacro:motor_wheel prefix="$(arg prefix)back_right_motor" parent="$(arg prefix)back_right_steer_wheel_link" hq="$(arg hq)">
 		<origin xyz="-${motor_wheel_offset_x} -${motor_wheel_offset_y} ${motor_wheel_offset_z}" rpy="0 0 ${PI}"/>
 	</xacro:motor_wheel>
-	<xacro:motor_wheel prefix="$(arg prefix)back_left_motor" parent="$(arg prefix)back_left_steer_wheel_link">
+	<xacro:motor_wheel prefix="$(arg prefix)back_left_motor" parent="$(arg prefix)back_left_steer_wheel_link" hq="$(arg hq)">
 		<origin xyz="-${motor_wheel_offset_x} ${motor_wheel_offset_y} ${motor_wheel_offset_z}" rpy="0 0 0"/>
 	</xacro:motor_wheel>
-<!--
-	<xacro:motor_wheel prefix="$(arg prefix)front_right_motor" parent="$(arg prefix)base_link" reflect="false" hq="${hq}">
-		<origin xyz="${motor_wheel_offset_x} -${motor_wheel_offset_y} ${motor_wheel_offset_z}" rpy="0 0 ${PI}"/>
-	</xacro:motor_wheel>
-	<xacro:motor_wheel prefix="$(arg prefix)front_left_motor" parent="$(arg prefix)base_link" reflect="true" hq="${hq}">
-		<origin xyz="${motor_wheel_offset_x} ${motor_wheel_offset_y} ${motor_wheel_offset_z}" rpy="0 0 0"/>
-	</xacro:motor_wheel>
-	<xacro:motor_wheel prefix="$(arg prefix)back_right_motor" parent="$(arg prefix)base_link" reflect="false" hq="${hq}">
-		<origin xyz="-${motor_wheel_offset_x} -${motor_wheel_offset_y} ${motor_wheel_offset_z}" rpy="0 0 ${PI}"/>
-	</xacro:motor_wheel>
-	<xacro:motor_wheel prefix="$(arg prefix)back_left_motor" parent="$(arg prefix)base_link" reflect="true" hq="${hq}">
-		<origin xyz="-${motor_wheel_offset_x} ${motor_wheel_offset_y} ${motor_wheel_offset_z}" rpy="0 0 0"/>
-	</xacro:motor_wheel>
--->
 	<!-- SENSORS -->
     <!--xacro:sensor_imu prefix="imu" parent="${prefix}base_link">

File: rbsherpa_hl_description/urdf/bases/rbsherpa_hl_base.urdf.xacro (robot description, xacro)
@@ -30,6 +30,6 @@
       </inertial>
       <visual>
-        <origin xyz="0 0 0" rpy="0 0 0" />
         <xacro:if value="${hq}">
+          <origin xyz="0 0 0" rpy="0 0 0" />
           <geometry>
             <mesh filename="package://rbsherpa_hl_description/meshes/bases/rbsherpa_hl_base.dae"/>
@@ -37,6 +37,7 @@
         </xacro:if>
         <xacro:unless value="${hq}">
+          <origin xyz="0 0 0.5" rpy="0 0 0" />
           <geometry>
-            <mesh filename="package://rbsherpa_hl_description/meshes/bases/rbsherpa_hl_base.stl"/>
+            <box size="1.55 0.925 0.5" />
           </geometry>
         </xacro:unless>
@@ -51,8 +52,8 @@
       </visual>
       <collision>
-        <origin xyz="0 0 0.6" rpy="0 0 0 " />
+        <origin xyz="0 0 0.5" rpy="0 0 0 " />
         <geometry>
           <!--mesh filename="package://rbsherpa_hl_description/meshes/bases/rbsherpa_hl_base.dae"/-->
-          <box size="1.4 0.6 0.5" />
+          <box size="1.55 0.925 0.5" />
         </geometry>
       </collision>

File: rbsherpa_hl_description/urdf/wheels/motor_wheel.urdf.xacro (robot description, xacro)
@@ -7,5 +7,5 @@
 	<xacro:property name="wheel_radius" value="0.18415" />
 	<xacro:property name="wheel_height" value="0.14" />
-  <xacro:macro name="motor_wheel" params="prefix parent *origin">
+  <xacro:macro name="motor_wheel" params="prefix parent *origin hq">
 	  <joint name="${prefix}_wheel_joint" type="continuous">
 	    <parent link="${parent}"/>
@@ -18,8 +18,16 @@
 	  <link name="${prefix}_wheel_link">
 	    <visual>
-	      <origin xyz="0 0 0" rpy="0 0 0" />
-	      <geometry>
-					<mesh filename="package://rbsherpa_hl_description/meshes/wheels/rbsherpa_hl_motorwheel.dae" />
-	      </geometry>
+				<xacro:if value="${hq}">
+		      <origin xyz="0 0 0" rpy="0 0 0" />
+		      <geometry>
+						<mesh filename="package://rbsherpa_hl_description/meshes/wheels/rbsherpa_hl_motorwheel.dae" />
+		      </geometry>
+				</xacro:if>
+				<xacro:unless value="${hq}">
+					<origin xyz="0 0 0" rpy="${M_PI/2} 0 0" />
+					<geometry>
+						<cylinder length="${wheel_height}" radius="${wheel_radius}" />
+					</geometry>
+				</xacro:unless>
 	    </visual>
 	    <collision>

File: rbsherpa_hl_description/urdf/wheels/steer_wheel.urdf.xacro (robot description, xacro)
@@ -6,5 +6,5 @@
   <xacro:property name="steer_joint_friction" value="0.01" />
   <xacro:property name="steer_joint_position_limit" value="2.9" />
-  <xacro:macro name="steer_wheel" params="prefix parent *origin">
+  <xacro:macro name="steer_wheel" params="prefix parent *origin hq">
     <joint name="${prefix}_wheel_joint" type="revolute">
       <parent link="${parent}"/>
@@ -17,13 +17,21 @@
     <link name="${prefix}_wheel_link">
       <visual>
-        <origin xyz="0 0 0" rpy="0 0 0" />
-        <geometry>
-  			  <mesh filename="package://rbsherpa_hl_description/meshes/wheels/rbsherpa_hl_wheel.dae" />
-        </geometry>
+        <xacro:if value="${hq}">
+          <origin xyz="0 0 0" rpy="0 0 0" />
+          <geometry>
+    			  <mesh filename="package://rbsherpa_hl_description/meshes/wheels/rbsherpa_hl_wheel.dae" />
+          </geometry>
+        </xacro:if>
+        <xacro:unless value="${hq}">
+          <origin xyz="0 0 0" rpy="0 0 0" />
+          <geometry>
+    			  <cylinder length="0.2" radius="0.1" />
+          </geometry>
+        </xacro:unless>
       </visual>
       <collision>
 		    <origin xyz="0 0 0" rpy="0 0 0" />
         <geometry>
-			    <cylinder length="0.1" radius="0.1" />
+			    <cylinder length="0.2" radius="0.1" />
         </geometry>
       </collision>

Commit message: Use planar_move plugin

File: rbsherpa_hl_description/robots/rbsherpa_hl_std.urdf.xacro (robot description, xacro)
@@ -17,6 +17,8 @@
   <xacro:arg name="prefix" default="rbsherpa_hl"/>
 	<xacro:arg name="hq" default="false"/>
+  <xacro:arg name="ros_planar_move_plugin" default="true"/>
   <!-- Import Gazebo Stuff -->
   <xacro:include filename="$(find rbsherpa_hl_description)/urdf/common.gazebo.xacro" />
+  <xacro:include filename="$(find rbsherpa_hl_description)/urdf/bases/rbsherpa_hl_base.gazebo.xacro" />
 	<!-- ***************** -->
 	<!-- Global parameters -->
@@ -41,42 +43,48 @@
 		<origin xyz="0.4785 0.01 2.05265" rpy="0 0 0"/>
 	</xacro:structure-->
-	<!-- Gazebo ros control pluggins -->
+	<!--xacro:gazebo_colors prefix="$(arg prefix)"/-->
+  <xacro:macro name="rbsherpa_hl" params="prefix hq">
+		<!-- STEER WHEELS -->
+		<xacro:steer_wheel prefix="$(arg prefix)front_right_steer" parent="$(arg prefix)base_link" hq="$(arg hq)">
+			<origin xyz="${steer_wheel_offset_x} -${steer_wheel_offset_y} ${steer_wheel_offset_z}" rpy="0 0 0"/>
+		</xacro:steer_wheel>
+		<xacro:steer_wheel prefix="$(arg prefix)front_left_steer" parent="$(arg prefix)base_link" hq="$(arg hq)">
+			<origin xyz="${steer_wheel_offset_x} ${steer_wheel_offset_y} ${steer_wheel_offset_z}" rpy="0 0 0"/>
+		</xacro:steer_wheel>
+		<xacro:steer_wheel prefix="$(arg prefix)back_right_steer" parent="$(arg prefix)base_link" hq="$(arg hq)">
+			<origin xyz="-${steer_wheel_offset_x} -${steer_wheel_offset_y} ${steer_wheel_offset_z}" rpy="0 0 0"/>
+		</xacro:steer_wheel>
+		<xacro:steer_wheel prefix="$(arg prefix)back_left_steer" parent="$(arg prefix)base_link" hq="$(arg hq)">
+			<origin xyz="-${steer_wheel_offset_x} ${steer_wheel_offset_y} ${steer_wheel_offset_z}" rpy="0 0 0"/>
+		</xacro:steer_wheel>
+		<!-- MOTOR WHEELS -->
+		<xacro:motor_wheel prefix="$(arg prefix)front_right_motor" parent="$(arg prefix)front_right_steer_wheel_link" hq="$(arg hq)">
+			<origin xyz="${motor_wheel_offset_x} -${motor_wheel_offset_y} ${motor_wheel_offset_z}" rpy="0 0 ${PI}"/>
+		</xacro:motor_wheel>
+		<xacro:motor_wheel prefix="$(arg prefix)front_left_motor" parent="$(arg prefix)front_left_steer_wheel_link" hq="$(arg hq)">
+			<origin xyz="${motor_wheel_offset_x} ${motor_wheel_offset_y} ${motor_wheel_offset_z}" rpy="0 0 0"/>
+		</xacro:motor_wheel>
+		<xacro:motor_wheel prefix="$(arg prefix)back_right_motor" parent="$(arg prefix)back_right_steer_wheel_link" hq="$(arg hq)">
+			<origin xyz="-${motor_wheel_offset_x} -${motor_wheel_offset_y} ${motor_wheel_offset_z}" rpy="0 0 ${PI}"/>
+		</xacro:motor_wheel>
+		<xacro:motor_wheel prefix="$(arg prefix)back_left_motor" parent="$(arg prefix)back_left_steer_wheel_link" hq="$(arg hq)">
+			<origin xyz="-${motor_wheel_offset_x} ${motor_wheel_offset_y} ${motor_wheel_offset_z}" rpy="0 0 0"/>
+		</xacro:motor_wheel>
+		<!-- SENSORS -->
+	    <!--xacro:sensor_imu prefix="imu" parent="${prefix}base_link">
+	          <origin xyz="-0.40 0.06 0.75" rpy="0 0 0"/>
+		</xacro:sensor_imu-->
+		<xacro:sensor_sick_s300 prefix="$(arg prefix)front_laser" parent="$(arg prefix)base_link" prefix_topic="front_laser">
+			<origin xyz="0.81495 -0.53572 0.28772" rpy="0 0 ${-PI/4.0}"/>
+		</xacro:sensor_sick_s300>
+		<xacro:sensor_sick_s300 prefix="$(arg prefix)rear_laser" parent="$(arg prefix)base_link" prefix_topic="rear_laser">
+			<origin xyz="-0.81495 0.53572 0.28772" rpy="0 0 ${3.0*PI/4.0}"/>
+		</xacro:sensor_sick_s300>
+	</xacro:macro>
+	<!-- Gazebo ros control plugins -->
 	<xacro:ros_control/>
-	<!--xacro:gazebo_colors prefix="$(arg prefix)"/-->
-	<!-- STEER WHEELS -->
-	<xacro:steer_wheel prefix="$(arg prefix)front_right_steer" parent="$(arg prefix)base_link" hq="$(arg hq)">
-		<origin xyz="${steer_wheel_offset_x} -${steer_wheel_offset_y} ${steer_wheel_offset_z}" rpy="0 0 0"/>
-	</xacro:steer_wheel>
-	<xacro:steer_wheel prefix="$(arg prefix)front_left_steer" parent="$(arg prefix)base_link" hq="$(arg hq)">
-		<origin xyz="${steer_wheel_offset_x} ${steer_wheel_offset_y} ${steer_wheel_offset_z}" rpy="0 0 0"/>
-	</xacro:steer_wheel>
-	<xacro:steer_wheel prefix="$(arg prefix)back_right_steer" parent="$(arg prefix)base_link" hq="$(arg hq)">
-		<origin xyz="-${steer_wheel_offset_x} -${steer_wheel_offset_y} ${steer_wheel_offset_z}" rpy="0 0 0"/>
-	</xacro:steer_wheel>
-	<xacro:steer_wheel prefix="$(arg prefix)back_left_steer" parent="$(arg prefix)base_link" hq="$(arg hq)">
-		<origin xyz="-${steer_wheel_offset_x} ${steer_wheel_offset_y} ${steer_wheel_offset_z}" rpy="0 0 0"/>
-	</xacro:steer_wheel>
-	<!-- MOTOR WHEELS -->
-	<xacro:motor_wheel prefix="$(arg prefix)front_right_motor" parent="$(arg prefix)front_right_steer_wheel_link" hq="$(arg hq)">
-		<origin xyz="${motor_wheel_offset_x} -${motor_wheel_offset_y} ${motor_wheel_offset_z}" rpy="0 0 ${PI}"/>
-	</xacro:motor_wheel>
-	<xacro:motor_wheel prefix="$(arg prefix)front_left_motor" parent="$(arg prefix)front_left_steer_wheel_link" hq="$(arg hq)">
-		<origin xyz="${motor_wheel_offset_x} ${motor_wheel_offset_y} ${motor_wheel_offset_z}" rpy="0 0 0"/>
-	</xacro:motor_wheel>
-	<xacro:motor_wheel prefix="$(arg prefix)back_right_motor" parent="$(arg prefix)back_right_steer_wheel_link" hq="$(arg hq)">
-		<origin xyz="-${motor_wheel_offset_x} -${motor_wheel_offset_y} ${motor_wheel_offset_z}" rpy="0 0 ${PI}"/>
-	</xacro:motor_wheel>
-	<xacro:motor_wheel prefix="$(arg prefix)back_left_motor" parent="$(arg prefix)back_left_steer_wheel_link" hq="$(arg hq)">
-		<origin xyz="-${motor_wheel_offset_x} ${motor_wheel_offset_y} ${motor_wheel_offset_z}" rpy="0 0 0"/>
-	</xacro:motor_wheel>
-	<!-- SENSORS -->
-    <!--xacro:sensor_imu prefix="imu" parent="${prefix}base_link">
-          <origin xyz="-0.40 0.06 0.75" rpy="0 0 0"/>
-	</xacro:sensor_imu-->
-    <xacro:sensor_sick_s300 prefix="$(arg prefix)front_laser" parent="$(arg prefix)base_link" prefix_topic="front_laser">
-		<origin xyz="0.81495 -0.53572 0.28772" rpy="0 0 ${-PI/4.0}"/>
-	</xacro:sensor_sick_s300>
-	<xacro:sensor_sick_s300 prefix="$(arg prefix)rear_laser" parent="$(arg prefix)base_link" prefix_topic="rear_laser">
-		<origin xyz="-0.81495 0.53572 0.28772" rpy="0 0 ${3.0*PI/4.0}"/>
-	</xacro:sensor_sick_s300>
+	<xacro:if value="$(arg ros_planar_move_plugin)">
+		<xacro:omni_steering prefix="$(arg prefix)" publish_tf="false"/>
+	</xacro:if>
+	<xacro:rbsherpa_hl prefix="$(arg prefix)" hq="false"/>
 </robot>

File: rbsherpa_hl_description/urdf/bases/rbsherpa_hl_base.gazebo.xacro (robot description, xacro)
@@ -32,5 +32,5 @@
 		</gazebo>
 	</xacro:macro>
-	<xacro:macro name="ros_control" params="prefix_frame prefix_topic">
+	<xacro:macro name="ros_control">
 	   <gazebo>
       <plugin name="ros_control" filename="libgazebo_ros_control.so">
@@ -42,4 +42,16 @@
    </gazebo>
    </xacro:macro>
+	 <xacro:macro name="omni_steering" params="prefix publish_tf">
+		<gazebo>
+			<plugin name="omni_steering" filename="libgazebo_ros_planar_move.so">
+				<commandTopic>rbsherpa_hl_control/cmd_vel</commandTopic>
+				<odometryTopic>rbsherpa_hl_control/odom</odometryTopic>
+				<odometryFrame>${prefix}odom</odometryFrame>
+				<odometryRate>50.0</odometryRate>
+				<robotBaseFrame>${prefix}base_footprint</robotBaseFrame>
+				<publishTF>${publish_tf}</publishTF>
+			</plugin>
+		</gazebo>
+	 </xacro:macro>
 	<gazebo reference="base_footprint">
 		<material>Gazebo/Green</material>
