Commit message: renamed motor_wheels to traction_wheels

File: rbsherpa_hl_description/robots/rbsherpa_hl_std.urdf.xacro (robot description, xacro)
@@ -7,8 +7,8 @@
 	<!-- Import RBSHERPA base elements -->
   <xacro:include filename="$(find rbsherpa_hl_description)/urdf/bases/rbsherpa_hl_base.urdf.xacro" />
-	<!-- Import RBSHERPA wheels -->
+	<!-- Import RBSHERPA steer wheels -->
 	<xacro:include filename="$(find rbsherpa_hl_description)/urdf/wheels/steer_wheel.urdf.xacro" />
-	<!-- Import RBSHERPA motor wheels -->
-	<xacro:include filename="$(find rbsherpa_hl_description)/urdf/wheels/motor_wheel.urdf.xacro" />
+	<!-- Import RBSHERPA traction wheels -->
+	<xacro:include filename="$(find rbsherpa_hl_description)/urdf/wheels/traction_wheel.urdf.xacro" />
 	<!-- Import RBSHERPA structure-->
 	<xacro:include filename="$(find rbsherpa_hl_description)/urdf/structures/structure.urdf.xacro" />
@@ -25,12 +25,12 @@
 	<!-- ***************** -->
 	<xacro:property name="PI" value="3.1415926535897931"/>
-	<!-- Wheel parameters -->
+	<!-- Steer wheel parameters -->
 	<xacro:property name="steer_wheel_offset_x" value="0.6236" />    <!-- x,y,z in translation from base_link to the center of the wheel -->
 	<xacro:property name="steer_wheel_offset_y" value="0.36063" />
 	<xacro:property name="steer_wheel_offset_z" value="0.28762" />
-	<!-- Motor wheel parameters -->
-	<xacro:property name="motor_wheel_offset_x" value="0.0" />    <!-- x,y,z in translation from base_link to the center of the wheel -->
-	<xacro:property name="motor_wheel_offset_y" value="0.029" />
-	<xacro:property name="motor_wheel_offset_z" value="-0.28762" />
+	<!-- Traction wheel parameters -->
+	<xacro:property name="traction_wheel_offset_x" value="0.0" />    <!-- x,y,z in translation from base_link to the center of the wheel -->
+	<xacro:property name="traction_wheel_offset_y" value="0.029" />
+	<xacro:property name="traction_wheel_offset_z" value="-0.28762" />
 	<!-- *************** -->
 	<!-- Robots Elements -->
@@ -58,17 +58,17 @@
 			<origin xyz="-${steer_wheel_offset_x} ${steer_wheel_offset_y} ${steer_wheel_offset_z}" rpy="0 0 0"/>
 		</xacro:steer_wheel>
-		<!-- MOTOR WHEELS -->
-		<xacro:motor_wheel prefix="$(arg prefix)front_right_motor" parent="$(arg prefix)front_right_steer_wheel_link" hq="$(arg hq)">
-			<origin xyz="${motor_wheel_offset_x} -${motor_wheel_offset_y} ${motor_wheel_offset_z}" rpy="0 0 ${PI}"/>
-		</xacro:motor_wheel>
-		<xacro:motor_wheel prefix="$(arg prefix)front_left_motor" parent="$(arg prefix)front_left_steer_wheel_link" hq="$(arg hq)">
-			<origin xyz="${motor_wheel_offset_x} ${motor_wheel_offset_y} ${motor_wheel_offset_z}" rpy="0 0 0"/>
-		</xacro:motor_wheel>
-		<xacro:motor_wheel prefix="$(arg prefix)back_right_motor" parent="$(arg prefix)back_right_steer_wheel_link" hq="$(arg hq)">
-			<origin xyz="-${motor_wheel_offset_x} -${motor_wheel_offset_y} ${motor_wheel_offset_z}" rpy="0 0 ${PI}"/>
-		</xacro:motor_wheel>
-		<xacro:motor_wheel prefix="$(arg prefix)back_left_motor" parent="$(arg prefix)back_left_steer_wheel_link" hq="$(arg hq)">
-			<origin xyz="-${motor_wheel_offset_x} ${motor_wheel_offset_y} ${motor_wheel_offset_z}" rpy="0 0 0"/>
-		</xacro:motor_wheel>
+		<!-- traction WHEELS -->
+		<xacro:traction_wheel prefix="$(arg prefix)front_right_traction" parent="$(arg prefix)front_right_steer_wheel_link" hq="$(arg hq)">
+			<origin xyz="${traction_wheel_offset_x} -${traction_wheel_offset_y} ${traction_wheel_offset_z}" rpy="0 0 ${PI}"/>
+		</xacro:traction_wheel>
+		<xacro:traction_wheel prefix="$(arg prefix)front_left_traction" parent="$(arg prefix)front_left_steer_wheel_link" hq="$(arg hq)">
+			<origin xyz="${traction_wheel_offset_x} ${traction_wheel_offset_y} ${traction_wheel_offset_z}" rpy="0 0 0"/>
+		</xacro:traction_wheel>
+		<xacro:traction_wheel prefix="$(arg prefix)back_right_traction" parent="$(arg prefix)back_right_steer_wheel_link" hq="$(arg hq)">
+			<origin xyz="-${traction_wheel_offset_x} -${traction_wheel_offset_y} ${traction_wheel_offset_z}" rpy="0 0 ${PI}"/>
+		</xacro:traction_wheel>
+		<xacro:traction_wheel prefix="$(arg prefix)back_left_traction" parent="$(arg prefix)back_left_steer_wheel_link" hq="$(arg hq)">
+			<origin xyz="-${traction_wheel_offset_x} ${traction_wheel_offset_y} ${traction_wheel_offset_z}" rpy="0 0 0"/>
+		</xacro:traction_wheel>
 		<!-- SENSORS -->
 	    <!--xacro:sensor_imu prefix="imu" parent="${prefix}base_link">

File: rbsherpa_hl_description/urdf/wheels/steer_wheel.urdf.xacro (robot description, xacro)
@@ -25,5 +25,5 @@
           <origin xyz="0 0 0" rpy="0 0 0" />
           <geometry>
-    			  <mesh filename="package://rbsherpa_hl_description/meshes/wheels/rbsherpa_hl_wheel.dae" />
+    			  <mesh filename="package://rbsherpa_hl_description/meshes/wheels/rbsherpa_hl_steer_wheel.dae" />
           </geometry>
         </xacro:if>

File: rbsherpa_hl_description/urdf/wheels/traction_wheel.transmission.xacro (robot description, xacro)
@@ -1,14 +1,14 @@
 <?xml version="1.0"?>
 <robot xmlns:xacro="http://www.ros.org/wiki/xacro">
- <xacro:property name="motor_wheel_mechanical_reduction" value="1.0" />
-<xacro:macro name="motor_wheel_transmission" params="prefix">
-	<transmission name="${prefix}_motor_wheel_joint_trans">
+ <xacro:property name="traction_wheel_mechanical_reduction" value="1.0" />
+<xacro:macro name="traction_wheel_transmission" params="prefix">
+	<transmission name="${prefix}_traction_wheel_joint_trans">
 	  <type>transmission_interface/SimpleTransmission</type>
 	  <joint name="${prefix}_wheel_joint">
 		<hardwareInterface>hardware_interface/VelocityJointInterface</hardwareInterface>
 	  </joint>
-	  <actuator name="${prefix}_motor_wheel_joint_motor">
+	  <actuator name="${prefix}_traction_wheel_joint_motor">
 		<hardwareInterface>hardware_interface/VelocityActuatorInterface</hardwareInterface>
-		<mechanicalReduction>${motor_wheel_mechanical_reduction}</mechanicalReduction>
+		<mechanicalReduction>${traction_wheel_mechanical_reduction}</mechanicalReduction>
 	  </actuator>
 	 </transmission>

File: rbsherpa_hl_description/urdf/wheels/traction_wheel.urdf.xacro (robot description, xacro)
@@ -1,5 +1,5 @@
 <?xml version="1.0"?>
-<robot name="motor_wheel" xmlns:xacro="http://www.ros.org/wiki/xacro">
-  <xacro:include filename="$(find rbsherpa_hl_description)/urdf/wheels/motor_wheel.transmission.xacro"/>
+<robot name="traction_wheel" xmlns:xacro="http://www.ros.org/wiki/xacro">
+  <xacro:include filename="$(find rbsherpa_hl_description)/urdf/wheels/traction_wheel.transmission.xacro"/>
   <xacro:property name="M_PI" value="3.1415926535897931" />
   <xacro:property name="wheel_joint_damping" value="2.0" />
@@ -12,5 +12,5 @@
 							izz="${m*(3*r*r+h*h)/12}" />
 	</xacro:macro>
-  <xacro:macro name="motor_wheel" params="prefix parent *origin hq">
+  <xacro:macro name="traction_wheel" params="prefix parent *origin hq">
 	  <joint name="${prefix}_wheel_joint" type="continuous">
 	    <parent link="${parent}"/>
@@ -26,5 +26,5 @@
 		      <origin xyz="0 0 0" rpy="0 0 0" />
 		      <geometry>
-						<mesh filename="package://rbsherpa_hl_description/meshes/wheels/rbsherpa_hl_motorwheel.dae" />
+						<mesh filename="package://rbsherpa_hl_description/meshes/wheels/rbsherpa_hl_traction_wheel.dae" />
 		      </geometry>
 				</xacro:if>
@@ -56,5 +56,5 @@
 	    </inertial>
 	  </link>
-	  <xacro:motor_wheel_transmission prefix="${prefix}" />
+	  <xacro:traction_wheel_transmission prefix="${prefix}" />
   </xacro:macro>
 </robot>

Commit message: standarized joint names

File: rbsherpa_hl_description/robots/rbsherpa_hl_std.urdf.xacro (robot description, xacro)
@@ -8,7 +8,7 @@
   <xacro:include filename="$(find rbsherpa_hl_description)/urdf/bases/rbsherpa_hl_base.urdf.xacro" />
 	<!-- Import RBSHERPA steer wheels -->
-	<xacro:include filename="$(find rbsherpa_hl_description)/urdf/wheels/steer_wheel.urdf.xacro" />
+	<xacro:include filename="$(find rbsherpa_hl_description)/urdf/wheels/wheel_steer.urdf.xacro" />
 	<!-- Import RBSHERPA traction wheels -->
-	<xacro:include filename="$(find rbsherpa_hl_description)/urdf/wheels/traction_wheel.urdf.xacro" />
+	<xacro:include filename="$(find rbsherpa_hl_description)/urdf/wheels/wheel_traction.urdf.xacro" />
 	<!-- Import RBSHERPA structure-->
 	<xacro:include filename="$(find rbsherpa_hl_description)/urdf/structures/structure.urdf.xacro" />
@@ -26,11 +26,11 @@
 	<xacro:property name="PI" value="3.1415926535897931"/>
 	<!-- Steer wheel parameters -->
-	<xacro:property name="steer_wheel_offset_x" value="0.6236" />    <!-- x,y,z in translation from base_link to the center of the wheel -->
-	<xacro:property name="steer_wheel_offset_y" value="0.36063" />
-	<xacro:property name="steer_wheel_offset_z" value="0.28762" />
+	<xacro:property name="wheel_steer_offset_x" value="0.6236" />    <!-- x,y,z in translation from base_link to the center of the wheel -->
+	<xacro:property name="wheel_steer_offset_y" value="0.36063" />
+	<xacro:property name="wheel_steer_offset_z" value="0.28762" />
 	<!-- Traction wheel parameters -->
-	<xacro:property name="traction_wheel_offset_x" value="0.0" />    <!-- x,y,z in translation from base_link to the center of the wheel -->
-	<xacro:property name="traction_wheel_offset_y" value="0.029" />
-	<xacro:property name="traction_wheel_offset_z" value="-0.28762" />
+	<xacro:property name="wheel_traction_offset_x" value="0.0" />    <!-- x,y,z in translation from base_link to the center of the wheel -->
+	<xacro:property name="wheel_traction_offset_y" value="0.029" />
+	<xacro:property name="wheel_traction_offset_z" value="-0.28762" />
 	<!-- *************** -->
 	<!-- Robots Elements -->
@@ -46,29 +46,29 @@
   <xacro:macro name="rbsherpa_hl" params="prefix hq">
 		<!-- STEER WHEELS -->
-		<xacro:steer_wheel prefix="$(arg prefix)front_right_steer" parent="$(arg prefix)base_link" hq="$(arg hq)">
-			<origin xyz="${steer_wheel_offset_x} -${steer_wheel_offset_y} ${steer_wheel_offset_z}" rpy="0 0 0"/>
-		</xacro:steer_wheel>
-		<xacro:steer_wheel prefix="$(arg prefix)front_left_steer" parent="$(arg prefix)base_link" hq="$(arg hq)">
-			<origin xyz="${steer_wheel_offset_x} ${steer_wheel_offset_y} ${steer_wheel_offset_z}" rpy="0 0 0"/>
-		</xacro:steer_wheel>
-		<xacro:steer_wheel prefix="$(arg prefix)back_right_steer" parent="$(arg prefix)base_link" hq="$(arg hq)">
-			<origin xyz="-${steer_wheel_offset_x} -${steer_wheel_offset_y} ${steer_wheel_offset_z}" rpy="0 0 0"/>
-		</xacro:steer_wheel>
-		<xacro:steer_wheel prefix="$(arg prefix)back_left_steer" parent="$(arg prefix)base_link" hq="$(arg hq)">
-			<origin xyz="-${steer_wheel_offset_x} ${steer_wheel_offset_y} ${steer_wheel_offset_z}" rpy="0 0 0"/>
-		</xacro:steer_wheel>
+		<xacro:wheel_steer prefix="$(arg prefix)front_right_wheel_steer" parent="$(arg prefix)base_link" hq="$(arg hq)">
+			<origin xyz="${wheel_steer_offset_x} -${wheel_steer_offset_y} ${wheel_steer_offset_z}" rpy="0 0 0"/>
+		</xacro:wheel_steer>
+		<xacro:wheel_steer prefix="$(arg prefix)front_left_wheel_steer" parent="$(arg prefix)base_link" hq="$(arg hq)">
+			<origin xyz="${wheel_steer_offset_x} ${wheel_steer_offset_y} ${wheel_steer_offset_z}" rpy="0 0 0"/>
+		</xacro:wheel_steer>
+		<xacro:wheel_steer prefix="$(arg prefix)back_right_wheel_steer" parent="$(arg prefix)base_link" hq="$(arg hq)">
+			<origin xyz="-${wheel_steer_offset_x} -${wheel_steer_offset_y} ${wheel_steer_offset_z}" rpy="0 0 0"/>
+		</xacro:wheel_steer>
+		<xacro:wheel_steer prefix="$(arg prefix)back_left_wheel_steer" parent="$(arg prefix)base_link" hq="$(arg hq)">
+			<origin xyz="-${wheel_steer_offset_x} ${wheel_steer_offset_y} ${wheel_steer_offset_z}" rpy="0 0 0"/>
+		</xacro:wheel_steer>
 		<!-- traction WHEELS -->
-		<xacro:traction_wheel prefix="$(arg prefix)front_right_traction" parent="$(arg prefix)front_right_steer_wheel_link" hq="$(arg hq)">
-			<origin xyz="${traction_wheel_offset_x} -${traction_wheel_offset_y} ${traction_wheel_offset_z}" rpy="0 0 ${PI}"/>
-		</xacro:traction_wheel>
-		<xacro:traction_wheel prefix="$(arg prefix)front_left_traction" parent="$(arg prefix)front_left_steer_wheel_link" hq="$(arg hq)">
-			<origin xyz="${traction_wheel_offset_x} ${traction_wheel_offset_y} ${traction_wheel_offset_z}" rpy="0 0 0"/>
-		</xacro:traction_wheel>
-		<xacro:traction_wheel prefix="$(arg prefix)back_right_traction" parent="$(arg prefix)back_right_steer_wheel_link" hq="$(arg hq)">
-			<origin xyz="-${traction_wheel_offset_x} -${traction_wheel_offset_y} ${traction_wheel_offset_z}" rpy="0 0 ${PI}"/>
-		</xacro:traction_wheel>
-		<xacro:traction_wheel prefix="$(arg prefix)back_left_traction" parent="$(arg prefix)back_left_steer_wheel_link" hq="$(arg hq)">
-			<origin xyz="-${traction_wheel_offset_x} ${traction_wheel_offset_y} ${traction_wheel_offset_z}" rpy="0 0 0"/>
-		</xacro:traction_wheel>
+		<xacro:wheel_traction prefix="$(arg prefix)front_right_wheel_traction" parent="$(arg prefix)front_right_wheel_steer_link" hq="$(arg hq)">
+			<origin xyz="${wheel_traction_offset_x} -${wheel_traction_offset_y} ${wheel_traction_offset_z}" rpy="0 0 ${PI}"/>
+		</xacro:wheel_traction>
+		<xacro:wheel_traction prefix="$(arg prefix)front_left_wheel_traction" parent="$(arg prefix)front_left_wheel_steer_link" hq="$(arg hq)">
+			<origin xyz="${wheel_traction_offset_x} ${wheel_traction_offset_y} ${wheel_traction_offset_z}" rpy="0 0 0"/>
+		</xacro:wheel_traction>
+		<xacro:wheel_traction prefix="$(arg prefix)back_right_wheel_traction" parent="$(arg prefix)back_right_wheel_steer_link" hq="$(arg hq)">
+			<origin xyz="-${wheel_traction_offset_x} -${wheel_traction_offset_y} ${wheel_traction_offset_z}" rpy="0 0 ${PI}"/>
+		</xacro:wheel_traction>
+		<xacro:wheel_traction prefix="$(arg prefix)back_left_wheel_traction" parent="$(arg prefix)back_left_wheel_steer_link" hq="$(arg hq)">
+			<origin xyz="-${wheel_traction_offset_x} ${wheel_traction_offset_y} ${wheel_traction_offset_z}" rpy="0 0 0"/>
+		</xacro:wheel_traction>
 		<!-- SENSORS -->
 	    <!--xacro:sensor_imu prefix="imu" parent="${prefix}base_link">

File: rbsherpa_hl_description/urdf/wheels/wheel_steer.transmission.xacro (robot description, xacro)
@@ -2,8 +2,8 @@
 <robot xmlns:xacro="http://www.ros.org/wiki/xacro">
 <xacro:property name="wheel_mechanical_reduction" value="1.0" />
-<xacro:macro name="steer_wheel_transmission" params="prefix">
+<xacro:macro name="wheel_steer_transmission" params="prefix">
 	<transmission name="${prefix}_wheel_joint_trans">
 	  <type>transmission_interface/SimpleTransmission</type>
-	  <joint name="${prefix}_wheel_joint">
+	  <joint name="${prefix}_joint">
 		<hardwareInterface>hardware_interface/PositionJointInterface</hardwareInterface>
 	  </joint>

File: rbsherpa_hl_description/urdf/wheels/wheel_steer.urdf.xacro (robot description, xacro)
@@ -1,5 +1,5 @@
 <?xml version="1.0"?>
-<robot name="steer_wheel" xmlns:xacro="http://www.ros.org/wiki/xacro">
-  <xacro:include filename="$(find rbsherpa_hl_description)/urdf/wheels/steer_wheel.transmission.xacro"/>
+<robot name="wheel_steer" xmlns:xacro="http://www.ros.org/wiki/xacro">
+  <xacro:include filename="$(find rbsherpa_hl_description)/urdf/wheels/wheel_steer.transmission.xacro"/>
   <xacro:property name="M_PI" value="3.1415926535897931" />
   <xacro:property name="steer_joint_damping" value="0.01" />
@@ -11,8 +11,8 @@
               izz="${m*(3*r*r+h*h)/12}" />
   </xacro:macro>
-  <xacro:macro name="steer_wheel" params="prefix parent *origin hq">
-    <joint name="${prefix}_wheel_joint" type="revolute">
+  <xacro:macro name="wheel_steer" params="prefix parent *origin hq">
+    <joint name="${prefix}_joint" type="revolute">
       <parent link="${parent}"/>
-      <child link="${prefix}_wheel_link"/>
+      <child link="${prefix}_link"/>
       <xacro:insert_block name="origin" />
       <axis xyz="0 0 1" rpy="0 0 0" />
@@ -20,10 +20,10 @@
       <joint_properties damping="${steer_joint_damping}" friction="${steer_joint_friction}"/>
     </joint>
-    <link name="${prefix}_wheel_link">
+    <link name="${prefix}_link">
       <visual>
         <xacro:if value="${hq}">
           <origin xyz="0 0 0" rpy="0 0 0" />
           <geometry>
-    			  <mesh filename="package://rbsherpa_hl_description/meshes/wheels/rbsherpa_hl_steer_wheel.dae" />
+    			  <mesh filename="package://rbsherpa_hl_description/meshes/wheels/rbsherpa_hl_wheel_steer.dae" />
           </geometry>
         </xacro:if>
@@ -55,5 +55,5 @@
       </inertial>
     </link>
-    <xacro:steer_wheel_transmission prefix="${prefix}" />
+    <xacro:wheel_steer_transmission prefix="${prefix}" />
   </xacro:macro>
 </robot>

File: rbsherpa_hl_description/urdf/wheels/wheel_traction.urdf.xacro (robot description, xacro)
@@ -1,5 +1,5 @@
 <?xml version="1.0"?>
-<robot name="traction_wheel" xmlns:xacro="http://www.ros.org/wiki/xacro">
-  <xacro:include filename="$(find rbsherpa_hl_description)/urdf/wheels/traction_wheel.transmission.xacro"/>
+<robot name="wheel_traction" xmlns:xacro="http://www.ros.org/wiki/xacro">
+  <xacro:include filename="$(find rbsherpa_hl_description)/urdf/wheels/wheel_traction.transmission.xacro"/>
   <xacro:property name="M_PI" value="3.1415926535897931" />
   <xacro:property name="wheel_joint_damping" value="2.0" />
@@ -12,8 +12,8 @@
 							izz="${m*(3*r*r+h*h)/12}" />
 	</xacro:macro>
-  <xacro:macro name="traction_wheel" params="prefix parent *origin hq">
-	  <joint name="${prefix}_wheel_joint" type="continuous">
+  <xacro:macro name="wheel_traction" params="prefix parent *origin hq">
+	  <joint name="${prefix}_joint" type="continuous">
 	    <parent link="${parent}"/>
-	    <child link="${prefix}_wheel_link"/>
+	    <child link="${prefix}_link"/>
 	    <xacro:insert_block name="origin" />
 	    <axis xyz="0 1 0" rpy="0 0 0" />
@@ -21,10 +21,10 @@
 	    <joint_properties damping="${wheel_joint_damping}" friction="${wheel_joint_friction}"/>
 	  </joint>
-	  <link name="${prefix}_wheel_link">
+	  <link name="${prefix}_link">
 	    <visual>
 				<xacro:if value="${hq}">
 		      <origin xyz="0 0 0" rpy="0 0 0" />
 		      <geometry>
-						<mesh filename="package://rbsherpa_hl_description/meshes/wheels/rbsherpa_hl_traction_wheel.dae" />
+						<mesh filename="package://rbsherpa_hl_description/meshes/wheels/rbsherpa_hl_wheel_traction.dae" />
 		      </geometry>
 				</xacro:if>
@@ -56,5 +56,5 @@
 	    </inertial>
 	  </link>
-	  <xacro:traction_wheel_transmission prefix="${prefix}" />
+	  <xacro:wheel_traction_transmission prefix="${prefix}" />
   </xacro:macro>
 </robot>
