Commit message: added structure to description

File: rbsherpa_hl_description/robots/rbsherpa_hl_std.urdf.xacro (robot description, xacro)
@@ -40,7 +40,7 @@
 	<xacro:rbsherpa_hl_base prefix="$(arg prefix)" publish_bf="true" hq="$(arg hq)" />
 	<!-- Structure -->
-	<!--xacro:structure prefix="$(arg prefix)" parent="$(arg prefix)base_link">
+	<xacro:structure prefix="$(arg prefix)" parent="$(arg prefix)base_link">
 		<origin xyz="0.4785 0.01 2.05265" rpy="0 0 0"/>
-	</xacro:structure-->
+	</xacro:structure>
 	<!--xacro:gazebo_colors prefix="$(arg prefix)"/-->
   <xacro:macro name="rbsherpa_hl" params="prefix hq">

File: rbsherpa_hl_description/urdf/structures/structure.urdf.xacro (robot description, xacro)
@@ -2,4 +2,5 @@
 <robot name="rbsherpa_structure" xmlns:xacro="http://www.ros.org/wiki/xacro">
   <xacro:property name="M_PI" value="3.1415926535897931" />
+  <xacro:property name="deg2rad" value="0.01745329251"/>
   <xacro:macro name="structure" params="prefix parent *origin">
 	<!--fixed joint -->
@@ -58,4 +59,207 @@
       </inertial>
     </link>
+        <!-- PAN TILT BASE -->
+    <joint name="${prefix}torso_pantilt_base_joint" type="fixed">
+      <origin xyz="0.0 0.0 0.0" rpy="0 0 0"/>
+      <parent link="${prefix}structure_link"/>
+      <!--<parent link="${prefix}torso_base_link"/>-->
+      <child link="${prefix}torso_pantilt_base_link"/>
+      <axis xyz="0 0 1"/>
+    </joint>
+    <link name="${prefix}torso_pantilt_base_link">
+      <visual>
+        <origin xyz="0 0 0" rpy="0 0 0"/>
+        <geometry>
+          <mesh filename="package://vulcano_torso_description/meshes/pantilt/base.stl"/>
+        </geometry>
+       <material name="lightgrey">
+         <color rgba="0.3 0.3 0.3 1"/>
+       </material>
+      </visual>
+      <collision>
+        <origin xyz="0 0 0" rpy="0 0 0"/>
+        <geometry>
+          <mesh filename="package://vulcano_torso_description/meshes/pantilt/base.stl"/>
+        </geometry>
+      </collision>
+      <inertial>
+        <origin xyz="0 0 0" rpy="0 0 0"/>
+        <mass value="5"/>
+        <inertia ixx="1.0" ixy="0.0" ixz="0.0" iyy="1.0" iyz="0.0" izz="1.0"/>
+      </inertial>
+    </link>
+    <!-- PAN JOINT/LINK -->
+    <joint name="${prefix}torso_pantilt_pan_base_joint" type="fixed">
+      <origin xyz="0.0 0.0 0.0" rpy="0 0 0"/>
+      <parent link="${prefix}torso_pantilt_base_link"/>
+      <child link="${prefix}torso_pantilt_pan_base_link"/>
+      <axis xyz="0 0 1"/>
+    </joint>
+    <link name="${prefix}torso_pantilt_pan_base_link">
+      <visual>
+        <origin xyz="0 0 0" rpy="0 0 0"/>
+        <geometry>
+          <mesh filename="package://vulcano_torso_description/meshes/pantilt/dynamixel_l42.stl"/>
+        </geometry>
+       <material name="lightgrey">
+         <color rgba="0.3 0.3 0.3 1"/>
+       </material>
+      </visual>
+      <collision>
+        <origin xyz="0 0 0" rpy="0 0 0"/>
+        <geometry>
+          <mesh filename="package://vulcano_torso_description/meshes/pantilt/dynamixel_l42.stl"/>
+        </geometry>
+      </collision>
+      <inertial>
+        <origin xyz="0 0 0" rpy="0 0 0"/>
+        <mass value="5"/>
+        <inertia ixx="1.0" ixy="0.0" ixz="0.0" iyy="1.0" iyz="0.0" izz="1.0"/>
+      </inertial>
+    </link>
+    <joint name="${prefix}torso_pantilt_pan_joint" type="revolute">
+      <origin xyz="0.0 0.0 0.111" rpy="0 0 0"/>
+      <parent link="${prefix}torso_pantilt_pan_base_link"/>
+      <child link="${prefix}torso_pantilt_pan_link"/>
+      <axis xyz="0 0 1"/>
+      <limit lower="${-360*deg2rad}" upper="${360*deg2rad}" effort="100" velocity="100"/>
+      <dynamics friction="1000" damping="1000"/>
+    </joint>
+    <link name="${prefix}torso_pantilt_pan_link">
+      <visual>
+        <origin xyz="0 0 0" rpy="0 0 0"/>
+        <geometry>
+          <mesh filename="package://vulcano_torso_description/meshes/pantilt/pan.stl"/>
+        </geometry>
+       <material name="lightgrey">
+         <color rgba="0.3 0.3 0.3 1"/>
+       </material>
+      </visual>
+      <collision>
+        <origin xyz="0 0 0" rpy="0 0 0"/>
+        <geometry>
+          <mesh filename="package://vulcano_torso_description/meshes/pantilt/pan.stl"/>
+        </geometry>
+      </collision>
+      <inertial>
+        <origin xyz="0 0 0" rpy="0 0 0"/>
+        <mass value="5"/>
+        <inertia ixx="1.0" ixy="0.0" ixz="0.0" iyy="1.0" iyz="0.0" izz="1.0"/>
+      </inertial>
+    </link>
+    <!-- TILT JOINT/LINK -->
+    <joint name="${prefix}torso_pantilt_tilt_joint" type="revolute">
+      <origin xyz="0.0 -0.027 0.0" rpy="${-90*deg2rad} 0 0"/>
+      <parent link="${prefix}torso_pantilt_pan_link"/>
+      <child link="${prefix}torso_pantilt_tilt_base_link"/>
+      <axis xyz="0 0 1"/>
+      <limit lower="${-360*deg2rad}" upper="${360*deg2rad}" effort="100" velocity="100"/>
+      <dynamics friction="1000" damping="1000"/>
+    </joint>
+    <link name="${prefix}torso_pantilt_tilt_base_link">
+      <visual>
+        <origin xyz="0 0 0" rpy="0 0 0"/>
+        <geometry>
+          <mesh filename="package://vulcano_torso_description/meshes/pantilt/dynamixel_l42.stl"/>
+        </geometry>
+       <material name="lightgrey">
+         <color rgba="0.3 0.3 0.3 1"/>
+       </material>
+      </visual>
+      <collision>
+        <origin xyz="0 0 0" rpy="0 0 0"/>
+        <geometry>
+          <mesh filename="package://vulcano_torso_description/meshes/pantilt/dynamixel_l42.stl"/>
+        </geometry>
+      </collision>
+      <inertial>
+        <origin xyz="0 0 0" rpy="0 0 0"/>
+        <mass value="5"/>
+        <inertia ixx="1.0" ixy="0.0" ixz="0.0" iyy="1.0" iyz="0.0" izz="1.0"/>
+      </inertial>
+    </link>
+    <joint name="${prefix}torso_pantilt_tilt_support_joint" type="fixed">
+      <origin xyz="0.0 0.0 0.0" rpy="${90*deg2rad} 0 0"/>
+      <parent link="${prefix}torso_pantilt_tilt_base_link"/>
+      <child link="${prefix}torso_pantilt_tilt_support_link"/>
+      <axis xyz="0 0 1"/>
+    </joint>
+    <link name="${prefix}torso_pantilt_tilt_support_link">
+      <visual>
+        <origin xyz="0 0 0" rpy="0 0 0"/>
+        <geometry>
+          <mesh filename="package://vulcano_torso_description/meshes/pantilt/tilt_support.stl"/>
+        </geometry>
+       <material name="lightgrey">
+         <color rgba="0.3 0.3 0.3 1"/>
+       </material>
+      </visual>
+      <collision>
+        <origin xyz="0 0 0" rpy="0 0 0"/>
+        <geometry>
+          <mesh filename="package://vulcano_torso_description/meshes/pantilt/tilt_support.stl"/>
+        </geometry>
+      </collision>
+      <inertial>
+        <origin xyz="0 0 0" rpy="0 0 0"/>
+        <mass value="5"/>
+        <inertia ixx="1.0" ixy="0.0" ixz="0.0" iyy="1.0" iyz="0.0" izz="1.0"/>
+      </inertial>
+    </link>
+    <joint name="${prefix}torso_pantilt_tilt_fixed_joint" type="fixed">
+      <!--<origin xyz="0.0 0.027 0.027" rpy="0 0 0"/>-->
+      <origin xyz="0.0 -0.027 0.027" rpy="${90*deg2rad} 0 0"/>
+      <parent link="${prefix}torso_pantilt_tilt_base_link"/>
+      <child link="${prefix}torso_pantilt_tilt_link"/>
+    </joint>
+    <link name="${prefix}torso_pantilt_tilt_link">
+      <visual>
+        <origin xyz="0 0 0" rpy="0 0 0"/>
+        <geometry>
+          <mesh filename="package://vulcano_torso_description/meshes/pantilt/tilt.stl"/>
+        </geometry>
+       <material name="lightgrey">
+         <color rgba="0.3 0.3 0.3 1"/>
+       </material>
+      </visual>
+      <collision>
+        <origin xyz="0 0 0" rpy="0 0 0"/>
+        <geometry>
+          <mesh filename="package://vulcano_torso_description/meshes/pantilt/tilt.stl"/>
+        </geometry>
+      </collision>
+      <inertial>
+        <origin xyz="0 0 0" rpy="0 0 0"/>
+        <mass value="5"/>
+        <inertia ixx="1.0" ixy="0.0" ixz="0.0" iyy="1.0" iyz="0.0" izz="1.0"/>
+      </inertial>
+    </link>
+    <joint name="${prefix}torso_pantilt_joint" type="fixed">
+      <origin xyz="0.0 0.0 0.003" rpy="0 0 0"/>
+      <parent link="${prefix}torso_pantilt_tilt_link"/>
+      <child link="${prefix}torso_pantilt_link"/>
+    </joint>
+    <link name="${prefix}torso_pantilt_link">
+      <visual>
+        <origin xyz="0 0 0" rpy="0 0 0"/>
+        <geometry>
+          <mesh filename="package://vulcano_torso_description/meshes/pantilt/pantilt.stl"/>
+        </geometry>
+       <material name="lightgrey">
+         <color rgba="0.3 0.3 0.3 1"/>
+       </material>
+      </visual>
+      <collision>
+        <origin xyz="0 0 0" rpy="0 0 0"/>
+        <geometry>
+          <mesh filename="package://vulcano_torso_description/meshes/pantilt/pantilt.stl"/>
+        </geometry>
+      </collision>
+      <inertial>
+        <origin xyz="0 0 0" rpy="0 0 0"/>
+        <mass value="5"/>
+        <inertia ixx="1.0" ixy="0.0" ixz="0.0" iyy="1.0" iyz="0.0" izz="1.0"/>
+      </inertial>
+    </link>
   </xacro:macro>
 </robot>

Commit message: Added gimbal and elevator structure. Included both structures in rbsherpa_hl_std

File: rbsherpa_hl_description/robots/rbsherpa_hl_std.urdf.xacro (robot description, xacro)
@@ -6,5 +6,5 @@
 	<!-- First we import all posible elements defined in the urdf.xacro files. All these elements are defined as macro:xacros -->
 	<!-- Import RBSHERPA base elements -->
-  <xacro:include filename="$(find rbsherpa_hl_description)/urdf/bases/rbsherpa_hl_base.urdf.xacro" />
+	<xacro:include filename="$(find rbsherpa_hl_description)/urdf/bases/rbsherpa_hl_base.urdf.xacro" />
 	<!-- Import RBSHERPA steer wheels -->
 	<xacro:include filename="$(find rbsherpa_hl_description)/urdf/wheels/wheel_steer.urdf.xacro" />
@@ -12,13 +12,14 @@
 	<xacro:include filename="$(find rbsherpa_hl_description)/urdf/wheels/wheel_traction.urdf.xacro" />
 	<!-- Import RBSHERPA structure-->
-	<xacro:include filename="$(find rbsherpa_hl_description)/urdf/structures/structure.urdf.xacro" />
-  <!-- Import all available sensors -->
-  <xacro:include filename="$(find robotnik_sensors)/urdf/all_sensors.urdf.xacro" />
-  <xacro:arg name="prefix" default="rbsherpa_hl"/>
-	<xacro:arg name="hq" default="false"/>
-  <xacro:arg name="ros_planar_move_plugin" default="true"/>
-  <!-- Import Gazebo Stuff -->
-  <xacro:include filename="$(find rbsherpa_hl_description)/urdf/common.gazebo.xacro" />
-  <xacro:include filename="$(find rbsherpa_hl_description)/urdf/bases/rbsherpa_hl_base.gazebo.xacro" />
+	<xacro:include filename="$(find rbsherpa_hl_description)/urdf/structures/elevator_structure.urdf.xacro" />
+	<xacro:include filename="$(find rbsherpa_hl_description)/urdf/structures/gimbal.urdf.xacro"/>
+	<!-- Import all available sensors -->
+	<xacro:include filename="$(find robotnik_sensors)/urdf/all_sensors.urdf.xacro" />
+	<xacro:arg name="prefix" default="rbsherpa_hl"/>
+	<xacro:arg name="hq" default="true"/>
+	<xacro:arg name="ros_planar_move_plugin" default="true"/>
+	<!-- Import Gazebo Stuff -->
+	<xacro:include filename="$(find rbsherpa_hl_description)/urdf/common.gazebo.xacro" />
+	<xacro:include filename="$(find rbsherpa_hl_description)/urdf/bases/rbsherpa_hl_base.gazebo.xacro" />
 	<!-- ***************** -->
 	<!-- Global parameters -->
@@ -26,11 +27,11 @@
 	<xacro:property name="PI" value="3.1415926535897931"/>
 	<!-- Steer wheel parameters -->
-	<xacro:property name="wheel_steer_offset_x" value="0.6236" />    <!-- x,y,z in translation from base_link to the center of the wheel -->
-	<xacro:property name="wheel_steer_offset_y" value="0.36063" />
-	<xacro:property name="wheel_steer_offset_z" value="0.28762" />
+	<xacro:property name="wheel_steer_offset_x" value="0.622" />    <!-- x,y,z in translation from base_link to the center of the wheel -->
+	<xacro:property name="wheel_steer_offset_y" value="0.367" />
+	<xacro:property name="wheel_steer_offset_z" value="0.285" />
 	<!-- Traction wheel parameters -->
 	<xacro:property name="wheel_traction_offset_x" value="0.0" />    <!-- x,y,z in translation from base_link to the center of the wheel -->
-	<xacro:property name="wheel_traction_offset_y" value="0.029" />
-	<xacro:property name="wheel_traction_offset_z" value="-0.28762" />
+	<xacro:property name="wheel_traction_offset_y" value="0.03" />
+	<xacro:property name="wheel_traction_offset_z" value="-0.285" />
 	<!-- *************** -->
 	<!-- Robots Elements -->
@@ -40,20 +41,24 @@
 	<xacro:rbsherpa_hl_base prefix="$(arg prefix)" publish_bf="true" hq="$(arg hq)" />
 	<!-- Structure -->
-	<xacro:structure prefix="$(arg prefix)" parent="$(arg prefix)base_link">
-		<origin xyz="0.4785 0.01 2.05265" rpy="0 0 0"/>
-	</xacro:structure>
+	<xacro:elevator_structure prefix="$(arg prefix)" parent="$(arg prefix)base_link">
+		<origin xyz="-0.430 0.0 0.302" rpy="0 0 0"/>
+	</xacro:elevator_structure>
+	<!-- Gimbal -->
+	<xacro:gimbal prefix="$(arg prefix)" parent="$(arg prefix)torso_pantilt_pan_link">
+		<origin xyz="-0.44 0.0 0.08" rpy="0 0 ${M_PI}"/>
+	</xacro:gimbal>
 	<!--xacro:gazebo_colors prefix="$(arg prefix)"/-->
-  <xacro:macro name="rbsherpa_hl" params="prefix hq">
+	<xacro:macro name="rbsherpa_hl" params="prefix hq">
 		<!-- STEER WHEELS -->
-		<xacro:wheel_steer prefix="$(arg prefix)front_right_wheel_steer" parent="$(arg prefix)base_link" hq="$(arg hq)">
+		<xacro:wheel_steer prefix="$(arg prefix)front_right_wheel_steer" parent="$(arg prefix)base_link" hq="$(arg hq)" type="revolute">
 			<origin xyz="${wheel_steer_offset_x} -${wheel_steer_offset_y} ${wheel_steer_offset_z}" rpy="0 0 0"/>
 		</xacro:wheel_steer>
-		<xacro:wheel_steer prefix="$(arg prefix)front_left_wheel_steer" parent="$(arg prefix)base_link" hq="$(arg hq)">
+		<xacro:wheel_steer prefix="$(arg prefix)front_left_wheel_steer" parent="$(arg prefix)base_link" hq="$(arg hq)" type="revolute">
 			<origin xyz="${wheel_steer_offset_x} ${wheel_steer_offset_y} ${wheel_steer_offset_z}" rpy="0 0 0"/>
 		</xacro:wheel_steer>
-		<xacro:wheel_steer prefix="$(arg prefix)back_right_wheel_steer" parent="$(arg prefix)base_link" hq="$(arg hq)">
+		<xacro:wheel_steer prefix="$(arg prefix)back_right_wheel_steer" parent="$(arg prefix)base_link" hq="$(arg hq)" type="revolute">
 			<origin xyz="-${wheel_steer_offset_x} -${wheel_steer_offset_y} ${wheel_steer_offset_z}" rpy="0 0 0"/>
 		</xacro:wheel_steer>
-		<xacro:wheel_steer prefix="$(arg prefix)back_left_wheel_steer" parent="$(arg prefix)base_link" hq="$(arg hq)">
+		<xacro:wheel_steer prefix="$(arg prefix)back_left_wheel_steer" parent="$(arg prefix)base_link" hq="$(arg hq)" type="revolute">
 			<origin xyz="-${wheel_steer_offset_x} ${wheel_steer_offset_y} ${wheel_steer_offset_z}" rpy="0 0 0"/>
 		</xacro:wheel_steer>
@@ -72,13 +77,16 @@
 		</xacro:wheel_traction>
 		<!-- SENSORS -->
-	    <!--xacro:sensor_imu prefix="imu" parent="${prefix}base_link">
-	          <origin xyz="-0.40 0.06 0.75" rpy="0 0 0"/>
+		<!--xacro:sensor_imu prefix="imu" parent="${prefix}base_link">
+			<origin xyz="-0.40 0.06 0.75" rpy="0 0 0"/>
 		</xacro:sensor_imu-->
 		<xacro:sensor_sick_s300 prefix="$(arg prefix)front_laser" parent="$(arg prefix)base_link" prefix_topic="front_laser">
-			<origin xyz="0.81495 -0.53572 0.28772" rpy="0 0 ${-PI/4.0}"/>
+			<origin xyz="0.835 -0.55472 0.221" rpy="${PI} 0 ${-PI/4.0}"/>
 		</xacro:sensor_sick_s300>
 		<xacro:sensor_sick_s300 prefix="$(arg prefix)rear_laser" parent="$(arg prefix)base_link" prefix_topic="rear_laser">
-			<origin xyz="-0.81495 0.53572 0.28772" rpy="0 0 ${3.0*PI/4.0}"/>
+			<origin xyz="-0.831 0.518 0.221" rpy="${PI} 0 ${3.0*PI/4.0}"/>
 		</xacro:sensor_sick_s300>
+		<xacro:sensor_velodyne_vlp16 prefix="$(arg prefix)velodyne" parent="$(arg prefix)base_link" prefix_topic="velodyne">
+			<origin xyz="0.869 0 0.248" rpy="0 0 0"/>
+		</xacro:sensor_velodyne_vlp16>
 	</xacro:macro>
 	<!-- Gazebo ros control plugins -->
