Commit message: description: updated pantilt model

File: rbsherpa_hl_description/robots/rbsherpa_hl_ackermann_std.urdf.xacro (robot description, xacro)
@@ -41,4 +41,5 @@
 	<!-- Structure -->
 	<xacro:pantilt prefix="$(arg prefix)" parent="$(arg prefix)base_link" hq="$(arg hq)">
+	   <origin xyz="1.089 0 0.398" rpy="0 0 0"/>
 	</xacro:pantilt>
 	<!--xacro:gazebo_colors prefix="$(arg prefix)"/-->
@@ -83,4 +84,7 @@
 			<origin xyz="0.869 0 0.248" rpy="0 0 0"/>
 		</xacro:sensor_velodyne_vlp16>
+		<xacro:sensor_gps prefix="$(arg prefix)gps" parent="$(arg prefix)base_link" > <!-- prefix_topic="gps" -->
+			<origin xyz="0.809 0 1.02" rpy="0 0 0"/>
+		</xacro:sensor_gps>
 	</xacro:macro>
 	<!-- Gazebo ros control plugins -->

File: rbsherpa_hl_description/urdf/pantilt/pan_tilt.urdf.xacro (robot description, xacro)
@@ -2,8 +2,13 @@
 <robot name="pantilt" xmlns:xacro="http://ros.org/wiki/xacro">
   <xacro:property name="PI" value="3.1415926535897931"/>
-  <xacro:macro name="pantilt" params="prefix parent hq">
+  <xacro:macro name="pantilt" params="prefix parent hq *origin">
+    <joint name="${prefix}torso_pantilt_base_joint" type="fixed">
+      <xacro:insert_block name="origin" />
+      <parent link="${parent}"/>
+      <child link="${prefix}torso_pantilt_base_link"/>
+    </joint>
+    <link name="${prefix}torso_pantilt_base_link"/>
     <joint name="${prefix}torso_pantilt_pan_joint" type="revolute">
-      <origin xyz="-0.547 0.0 1.32" rpy="0 0 0"/>
-      <parent link="${parent}"/>
+      <parent link="${prefix}torso_pantilt_base_link"/>
       <child link="${prefix}torso_pantilt_pan_link"/>
       <axis xyz="0 0 1"/>

Commit message: Added transmission parameter

File: rbsherpa_hl_description/robots/rbsherpa_hl_ackermann_std.urdf.xacro (robot description, xacro)
@@ -46,14 +46,14 @@
   <xacro:macro name="rbsherpa_hl" params="prefix hq">
 		<!-- STEER WHEELS -->
-		<xacro:wheel_steer prefix="$(arg prefix)front_right_wheel_steer" parent="$(arg prefix)base_link" hq="$(arg hq)" type="revolute">
+		<xacro:wheel_steer prefix="$(arg prefix)front_right_wheel_steer" parent="$(arg prefix)base_link" hq="$(arg hq)" type="revolute" transmission="true">
 			<origin xyz="${wheel_steer_offset_x} -${wheel_steer_offset_y} ${wheel_steer_offset_z}" rpy="0 0 0"/>
 		</xacro:wheel_steer>
-		<xacro:wheel_steer prefix="$(arg prefix)front_left_wheel_steer" parent="$(arg prefix)base_link" hq="$(arg hq)" type="revolute">
+		<xacro:wheel_steer prefix="$(arg prefix)front_left_wheel_steer" parent="$(arg prefix)base_link" hq="$(arg hq)" type="revolute" transmission="true">
 			<origin xyz="${wheel_steer_offset_x} ${wheel_steer_offset_y} ${wheel_steer_offset_z}" rpy="0 0 0"/>
 		</xacro:wheel_steer>
-		<xacro:wheel_steer prefix="$(arg prefix)back_right_wheel_steer" parent="$(arg prefix)base_link" hq="$(arg hq)" type="fixed">
+		<xacro:wheel_steer prefix="$(arg prefix)back_right_wheel_steer" parent="$(arg prefix)base_link" hq="$(arg hq)" type="fixed" transmission="false">
 			<origin xyz="-${wheel_steer_offset_x} -${wheel_steer_offset_y} ${wheel_steer_offset_z}" rpy="0 0 0"/>
 		</xacro:wheel_steer>
-		<xacro:wheel_steer prefix="$(arg prefix)back_left_wheel_steer" parent="$(arg prefix)base_link" hq="$(arg hq)" type="fixed">
+		<xacro:wheel_steer prefix="$(arg prefix)back_left_wheel_steer" parent="$(arg prefix)base_link" hq="$(arg hq)" type="fixed" transmission="false">
 			<origin xyz="-${wheel_steer_offset_x} ${wheel_steer_offset_y} ${wheel_steer_offset_z}" rpy="0 0 0"/>
 		</xacro:wheel_steer>

File: rbsherpa_hl_description/robots/rbsherpa_hl_omni_std.urdf.xacro (robot description, xacro)
@@ -51,14 +51,14 @@
 	<xacro:macro name="rbsherpa_hl" params="prefix hq">
 		<!-- STEER WHEELS -->
-		<xacro:wheel_steer prefix="$(arg prefix)front_right_wheel_steer" parent="$(arg prefix)base_link" hq="$(arg hq)" type="revolute">
+		<xacro:wheel_steer prefix="$(arg prefix)front_right_wheel_steer" parent="$(arg prefix)base_link" hq="$(arg hq)" type="revolute" transmission="true">
 			<origin xyz="${wheel_steer_offset_x} -${wheel_steer_offset_y} ${wheel_steer_offset_z}" rpy="0 0 0"/>
 		</xacro:wheel_steer>
-		<xacro:wheel_steer prefix="$(arg prefix)front_left_wheel_steer" parent="$(arg prefix)base_link" hq="$(arg hq)" type="revolute">
+		<xacro:wheel_steer prefix="$(arg prefix)front_left_wheel_steer" parent="$(arg prefix)base_link" hq="$(arg hq)" type="revolute" transmission="true">
 			<origin xyz="${wheel_steer_offset_x} ${wheel_steer_offset_y} ${wheel_steer_offset_z}" rpy="0 0 0"/>
 		</xacro:wheel_steer>
-		<xacro:wheel_steer prefix="$(arg prefix)back_right_wheel_steer" parent="$(arg prefix)base_link" hq="$(arg hq)" type="revolute">
+		<xacro:wheel_steer prefix="$(arg prefix)back_right_wheel_steer" parent="$(arg prefix)base_link" hq="$(arg hq)" type="revolute" transmission="true">
 			<origin xyz="-${wheel_steer_offset_x} -${wheel_steer_offset_y} ${wheel_steer_offset_z}" rpy="0 0 0"/>
 		</xacro:wheel_steer>
-		<xacro:wheel_steer prefix="$(arg prefix)back_left_wheel_steer" parent="$(arg prefix)base_link" hq="$(arg hq)" type="revolute">
+		<xacro:wheel_steer prefix="$(arg prefix)back_left_wheel_steer" parent="$(arg prefix)base_link" hq="$(arg hq)" type="revolute" transmission="true">
 			<origin xyz="-${wheel_steer_offset_x} ${wheel_steer_offset_y} ${wheel_steer_offset_z}" rpy="0 0 0"/>
 		</xacro:wheel_steer>

File: rbsherpa_hl_description/urdf/wheels/wheel_steer.urdf.xacro (robot description, xacro)
@@ -11,5 +11,5 @@
               izz="${m*(3*r*r+h*h)/12}" />
   </xacro:macro>
-  <xacro:macro name="wheel_steer" params="prefix parent *origin type hq">
+  <xacro:macro name="wheel_steer" params="prefix parent *origin type hq transmission">
     <joint name="${prefix}_joint" type="${type}">
       <parent link="${parent}"/>
@@ -55,5 +55,7 @@
       </inertial>
     </link>
-    <xacro:wheel_steer_transmission prefix="${prefix}" />
+    <xacro:if value="${transmission}">
+      <xacro:wheel_steer_transmission prefix="${prefix}" />
+    </xacro:if>
   </xacro:macro>
 </robot>

Commit message: rbsherpa_hl_description:: Added sim argument to URDF

File: rbsherpa_hl_description/robots/rbsherpa_hl_ackermann_std.urdf.xacro (robot description, xacro)
@@ -18,6 +18,7 @@
   <xacro:arg name="hq" default="true"/>
   <xacro:arg name="ros_planar_move_plugin" default="true"/>
+  <xacro:arg name="sim" default="false"/>
   <!-- Import Gazebo Stuff -->
-  <xacro:include filename="$(find rbsherpa_hl_description)/urdf/common.gazebo.xacro" />
+  <!--xacro:include filename="$(find rbsherpa_hl_description)/urdf/common.gazebo.xacro" /-->
   <xacro:include filename="$(find rbsherpa_hl_description)/urdf/bases/rbsherpa_hl_base.gazebo.xacro" />
 	<!-- ***************** -->
@@ -46,10 +47,20 @@
   <xacro:macro name="rbsherpa_hl" params="prefix hq">
 		<!-- STEER WHEELS -->
-		<xacro:wheel_steer prefix="$(arg prefix)front_right_wheel_steer" parent="$(arg prefix)base_link" hq="$(arg hq)" type="revolute" transmission="true">
-			<origin xyz="${wheel_steer_offset_x} -${wheel_steer_offset_y} ${wheel_steer_offset_z}" rpy="0 0 0"/>
-		</xacro:wheel_steer>
-		<xacro:wheel_steer prefix="$(arg prefix)front_left_wheel_steer" parent="$(arg prefix)base_link" hq="$(arg hq)" type="revolute" transmission="true">
-			<origin xyz="${wheel_steer_offset_x} ${wheel_steer_offset_y} ${wheel_steer_offset_z}" rpy="0 0 0"/>
-		</xacro:wheel_steer>
+		<xacro:if value="$(arg sim)">
+			<xacro:wheel_steer prefix="$(arg prefix)front_right_wheel_steer" parent="$(arg prefix)base_link" hq="$(arg hq)" type="fixed" transmission="false">
+				<origin xyz="${wheel_steer_offset_x} -${wheel_steer_offset_y} ${wheel_steer_offset_z}" rpy="0 0 0"/>
+			</xacro:wheel_steer>
+			<xacro:wheel_steer prefix="$(arg prefix)front_left_wheel_steer" parent="$(arg prefix)base_link" hq="$(arg hq)" type="fixed" transmission="false">
+				<origin xyz="${wheel_steer_offset_x} ${wheel_steer_offset_y} ${wheel_steer_offset_z}" rpy="0 0 0"/>
+			</xacro:wheel_steer>
+		</xacro:if>
+		<xacro:unless value="$(arg sim)">
+			<xacro:wheel_steer prefix="$(arg prefix)front_right_wheel_steer" parent="$(arg prefix)base_link" hq="$(arg hq)" type="revolute" transmission="true">
+				<origin xyz="${wheel_steer_offset_x} -${wheel_steer_offset_y} ${wheel_steer_offset_z}" rpy="0 0 0"/>
+			</xacro:wheel_steer>
+			<xacro:wheel_steer prefix="$(arg prefix)front_left_wheel_steer" parent="$(arg prefix)base_link" hq="$(arg hq)" type="revolute" transmission="true">
+				<origin xyz="${wheel_steer_offset_x} ${wheel_steer_offset_y} ${wheel_steer_offset_z}" rpy="0 0 0"/>
+			</xacro:wheel_steer>
+		</xacro:unless>
 		<xacro:wheel_steer prefix="$(arg prefix)back_right_wheel_steer" parent="$(arg prefix)base_link" hq="$(arg hq)" type="fixed" transmission="false">
 			<origin xyz="-${wheel_steer_offset_x} -${wheel_steer_offset_y} ${wheel_steer_offset_z}" rpy="0 0 0"/>

Commit message: rbsherpa_hl_description:: reverted changes to ackermann_std.urdf

File: rbsherpa_hl_description/robots/rbsherpa_hl_ackermann_std.urdf.xacro (robot description, xacro)
@@ -47,20 +47,10 @@
   <xacro:macro name="rbsherpa_hl" params="prefix hq">
 		<!-- STEER WHEELS -->
-		<xacro:if value="$(arg sim)">
-			<xacro:wheel_steer prefix="$(arg prefix)front_right_wheel_steer" parent="$(arg prefix)base_link" hq="$(arg hq)" type="fixed" transmission="false">
-				<origin xyz="${wheel_steer_offset_x} -${wheel_steer_offset_y} ${wheel_steer_offset_z}" rpy="0 0 0"/>
-			</xacro:wheel_steer>
-			<xacro:wheel_steer prefix="$(arg prefix)front_left_wheel_steer" parent="$(arg prefix)base_link" hq="$(arg hq)" type="fixed" transmission="false">
-				<origin xyz="${wheel_steer_offset_x} ${wheel_steer_offset_y} ${wheel_steer_offset_z}" rpy="0 0 0"/>
-			</xacro:wheel_steer>
-		</xacro:if>
-		<xacro:unless value="$(arg sim)">
-			<xacro:wheel_steer prefix="$(arg prefix)front_right_wheel_steer" parent="$(arg prefix)base_link" hq="$(arg hq)" type="revolute" transmission="true">
-				<origin xyz="${wheel_steer_offset_x} -${wheel_steer_offset_y} ${wheel_steer_offset_z}" rpy="0 0 0"/>
-			</xacro:wheel_steer>
-			<xacro:wheel_steer prefix="$(arg prefix)front_left_wheel_steer" parent="$(arg prefix)base_link" hq="$(arg hq)" type="revolute" transmission="true">
-				<origin xyz="${wheel_steer_offset_x} ${wheel_steer_offset_y} ${wheel_steer_offset_z}" rpy="0 0 0"/>
-			</xacro:wheel_steer>
-		</xacro:unless>
+		<xacro:wheel_steer prefix="$(arg prefix)front_right_wheel_steer" parent="$(arg prefix)base_link" hq="$(arg hq)" type="revolute" transmission="true">
+			<origin xyz="${wheel_steer_offset_x} -${wheel_steer_offset_y} ${wheel_steer_offset_z}" rpy="0 0 0"/>
+		</xacro:wheel_steer>
+		<xacro:wheel_steer prefix="$(arg prefix)front_left_wheel_steer" parent="$(arg prefix)base_link" hq="$(arg hq)" type="revolute" transmission="true">
+			<origin xyz="${wheel_steer_offset_x} ${wheel_steer_offset_y} ${wheel_steer_offset_z}" rpy="0 0 0"/>
+		</xacro:wheel_steer>
 		<xacro:wheel_steer prefix="$(arg prefix)back_right_wheel_steer" parent="$(arg prefix)base_link" hq="$(arg hq)" type="fixed" transmission="false">
 			<origin xyz="-${wheel_steer_offset_x} -${wheel_steer_offset_y} ${wheel_steer_offset_z}" rpy="0 0 0"/>
