Commit message: Added physical properties to base_pantilt and inertia xacro

File: rbsherpa_hl_description/urdf/pantilt/pan_tilt.urdf.xacro (robot description, xacro)
@@ -2,4 +2,10 @@
 <robot name="pantilt" xmlns:xacro="http://ros.org/wiki/xacro">
   <xacro:property name="PI" value="3.1415926535897931"/>
+    <xacro:macro name="solid_cuboid_inertia" params="m h d w">
+      <inertia  ixx="${(m*(h*h+d*d))/12}" ixy = "0" ixz = "0"
+                iyy="${(m*(w*w+d*d))/12}" iyz = "0"
+                izz="${(m*(w*w+h*h))/12}"
+      />
+    </xacro:macro>
   <xacro:macro name="pantilt" params="prefix parent hq *origin">
     <joint name="${prefix}torso_pantilt_base_joint" type="fixed">
@@ -8,5 +14,23 @@
       <child link="${prefix}torso_pantilt_base_link"/>
     </joint>
-    <link name="${prefix}torso_pantilt_base_link"/>
+    <link name="${prefix}torso_pantilt_base_link">
+      <visual>
+        <origin xyz="0 0 0" rpy="0 0 0" />
+        <geometry>
+          <box size="0.01 0.01 0.01" />
+        </geometry>
+      </visual>
+      <collision>
+        <origin xyz="0 0 0" rpy="0 0 0"/>
+        <geometry>
+          <cylinder radius="0.01" length="0.01"/>
+        </geometry>
+      </collision>
+      <inertial>
+        <mass value="0.005" />
+        <origin xyz="0 0 0" />
+        <solid_cuboid_inertia m="0.005" h="0.05" d="0.05" w="0.05"/>
+      </inertial>
+    </link>
     <joint name="${prefix}torso_pantilt_pan_joint" type="revolute">
       <parent link="${prefix}torso_pantilt_base_link"/>
@@ -19,9 +43,9 @@
         <type>transmission_interface/SimpleTransmission</type>
         <joint name="${prefix}torso_pantilt_pan_joint">
-          <hardwareInterface>PositionJointInterface</hardwareInterface>
+          <hardwareInterface>hardware_interface/PositionJointInterface</hardwareInterface>
         </joint>
         <actuator name="${prefix}torso_pantilt_pan_motor">
           <mechanicalReduction>1</mechanicalReduction>
-          <hardwareInterface>PositionJointInterface</hardwareInterface>
+          <hardwareInterface>hardware_interface/PositionJointInterface</hardwareInterface>
         </actuator>
     </transmission>
@@ -39,16 +63,16 @@
         <origin xyz="0 0 0" rpy="0 0 0"/>
         <geometry>
-          <mesh filename="package://rbsherpa_hl_description/meshes/pantilt/pan_dynamixel.stl"/>
+          <box size="0.01 0.01 0.01" />
         </geometry>
       </collision>
       <inertial>
-        <origin xyz="0 0 0" rpy="0 0 0"/>
-        <mass value="5"/>
-        <inertia ixx="1.0" ixy="0.0" ixz="0.0" iyy="1.0" iyz="0.0" izz="1.0"/>
+        <mass value="0.005" />
+        <origin xyz="0 0 0" />
+        <solid_cuboid_inertia m="0.005" h="0.05" d="0.05" w="0.05"/>
       </inertial>
     </link>
     <!-- TILT JOINT/LINK -->
     <joint name="${prefix}torso_pantilt_tilt_joint" type="revolute">
-      <origin xyz="0.0 0.0 0.126" rpy="0 0 0"/>
+      <origin xyz="0.0 0.0 0.13" rpy="0 0 0"/>
       <parent link="${prefix}torso_pantilt_pan_link"/>
       <child link="${prefix}torso_pantilt_tilt_link"/>
@@ -60,5 +84,5 @@
       <type>transmission_interface/SimpleTransmission</type>
       <joint name="${prefix}torso_pantilt_tilt_joint">
-        <hardwareInterface>PositionJointInterface</hardwareInterface>
+        <hardwareInterface>hardware_interface/PositionJointInterface</hardwareInterface>
       </joint>
       <actuator name="${prefix}torso_pantilt_tilt_motor">
@@ -80,11 +104,11 @@
         <origin xyz="0 0 0" rpy="0 0 0"/>
         <geometry>
-          <mesh filename="package://rbsherpa_hl_description/meshes/pantilt/tilt_dynamixel.stl"/>
+          <box size="0.01 0.01 0.01" />
         </geometry>
       </collision>
       <inertial>
-        <origin xyz="0 0 0" rpy="0 0 0"/>
-        <mass value="5"/>
-        <inertia ixx="1.0" ixy="0.0" ixz="0.0" iyy="1.0" iyz="0.0" izz="1.0"/>
+        <mass value="0.005" />
+        <origin xyz="0 0 0" />
+        <solid_cuboid_inertia m="0.005" h="0.05" d="0.05" w="0.05"/>
       </inertial>
     </link>
@@ -107,11 +131,11 @@
         <origin xyz="0 0 0" rpy="0 0 0"/>
         <geometry>
-          <mesh filename="package://rbsherpa_hl_description/meshes/pantilt/sprayer.stl"/>
+          <box size="0.01 0.01 0.01" />
         </geometry>
       </collision>
       <inertial>
-        <origin xyz="0 0 0" rpy="0 0 0"/>
-        <mass value="5"/>
-        <inertia ixx="1.0" ixy="0.0" ixz="0.0" iyy="1.0" iyz="0.0" izz="1.0"/>
+        <mass value="0.005" />
+        <origin xyz="0 0 0" />
+        <solid_cuboid_inertia m="0.005" h="0.05" d="0.05" w="0.05"/>
       </inertial>
     </link>

Commit message: rbsherpa_hl_description:: updated interta and friction values

File: rbsherpa_hl_description/urdf/pantilt/pan_tilt.urdf.xacro (robot description, xacro)
@@ -37,6 +37,6 @@
       <child link="${prefix}torso_pantilt_pan_link"/>
       <axis xyz="0 0 1"/>
-      <limit lower="-0.95" upper="0.95" effort="100" velocity="100"/>
-      <dynamics friction="1000" damping="1000"/>
+      <limit lower="-0.95" upper="0.95" effort="100" velocity="50"/>
+      <joint_properties friction="0.01" damping="0.01"/>
     </joint>
     <transmission name="${prefix}torso_pantilt_pan_trans">
@@ -63,11 +63,11 @@
         <origin xyz="0 0 0" rpy="0 0 0"/>
         <geometry>
-          <box size="0.01 0.01 0.01" />
+          <box size="0.1 0.1 0.1" />
         </geometry>
       </collision>
       <inertial>
-        <mass value="0.5" />
+        <mass value="1" />
         <origin xyz="0 0 0" />
-        <solid_cuboid_inertia m="0.5" h="0.05" d="0.05" w="0.05"/>
+        <solid_cuboid_inertia m="1" h="0.1" d="0.1" w="0.1"/>
       </inertial>
     </link>
@@ -78,6 +78,6 @@
       <child link="${prefix}torso_pantilt_tilt_link"/>
       <axis xyz="0 1 0"/>
-      <limit lower="-0.26" upper="0.26" effort="100" velocity="100"/>
-      <dynamics friction="1000" damping="1000"/>
+      <limit lower="-0.26" upper="0.26" effort="100" velocity="5"/>
+      <joint_properties friction="0.01" damping="0.01"/>
     </joint>
 	<transmission name="${prefix}torso_pantilt_tilt_trans">
@@ -104,11 +104,11 @@
         <origin xyz="0 0 0" rpy="0 0 0"/>
         <geometry>
-          <box size="0.01 0.01 0.01" />
+          <box size="0.1 0.1 0.1" />
         </geometry>
       </collision>
       <inertial>
-        <mass value="0.5" />
+        <mass value="1" />
         <origin xyz="0 0 0" />
-        <solid_cuboid_inertia m="0.5" h="0.05" d="0.05" w="0.05"/>
+        <solid_cuboid_inertia m="1" h="0.1" d="0.1" w="0.1"/>
       </inertial>
     </link>

File: rbsherpa_hl_description/urdf/wheels/wheel_steer.transmission.xacro (robot description, xacro)
@@ -9,5 +9,5 @@
 	  </joint>
 	  <actuator name="${prefix}_wheel_joint_motor">
-		<hardwareInterface>hardware_interface/PositionActuatorInterface</hardwareInterface>
+		<hardwareInterface>hardware_interface/PositionJointInterface</hardwareInterface>
 		<mechanicalReduction>${wheel_mechanical_reduction}</mechanicalReduction>
 	  </actuator>

File: rbsherpa_hl_description/urdf/wheels/wheel_steer.urdf.xacro (robot description, xacro)
@@ -38,9 +38,9 @@
 		    <origin xyz="0 0 0" rpy="0 0 0" />
         <geometry>
-			    <cylinder length="0.2" radius="0.1" />
+			    <cylinder length="0.1" radius="0.1" />
         </geometry>
       </collision>
       <inertial>
-        <mass value="5" />
+        <mass value="30.0" />
         <!--xacro:if value="${hq}">
           <origin xyz="0.00002 -0.06358 -0.18084" />

File: rbsherpa_hl_description/urdf/wheels/wheel_traction.transmission.xacro (robot description, xacro)
@@ -9,5 +9,5 @@
 	  </joint>
 	  <actuator name="${prefix}_wheel_traction_joint_motor">
-		<hardwareInterface>hardware_interface/VelocityActuatorInterface</hardwareInterface>
+		<hardwareInterface>hardware_interface/VelocityJointInterface</hardwareInterface>
 		<mechanicalReduction>${wheel_traction_mechanical_reduction}</mechanicalReduction>
 	  </actuator>

File: rbsherpa_hl_description/urdf/wheels/wheel_traction.urdf.xacro (robot description, xacro)
@@ -43,5 +43,5 @@
 	    </collision>
 	    <inertial>
-	      <mass value="6.91837" />
+	      <mass value="5.0" />
 				<!--xacro:if value="${hq}">
 		      <origin xyz="0 0.00036 0" />
@@ -51,6 +51,6 @@
 				</xacro:if>
 				<xacro:unless value="${hq}"-->
-					<origin xyz="0 0 0" />
-	        <cylinder_inertia  m="6.91837" r="${wheel_radius}" h="${wheel_height}" />
+					<origin xyz="0 0 0.0" />
+	        <cylinder_inertia  m="5.0" r="${wheel_radius}" h="${wheel_height}" />
 				<!--/xacro:unless-->
 	    </inertial>
