Commit message: rbsherpa_hl_description:: Changed collision radius value to inner radius value

File: rbsherpa_hl_description/urdf/wheels/wheel_traction.urdf.xacro (robot description, xacro)
@@ -6,4 +6,5 @@
   <xacro:property name="wheel_joint_friction" value="1.0" />
 	<xacro:property name="wheel_radius" value="0.18415" />
+	<xacro:property name="wheel_inner_radius" value="0.155" />
 	<xacro:property name="wheel_height" value="0.14" />
 	<xacro:macro name="cylinder_inertia" params="m r h">
@@ -39,5 +40,5 @@
 				<origin xyz="0 0 0" rpy="${M_PI/2} 0 0" />
 	      <geometry>
-	        <cylinder length="${wheel_height}" radius="${wheel_radius}" />
+	        <cylinder length="${wheel_height}" radius="${wheel_inner_radius}" />
 	      </geometry>
 	    </collision>
