Commit message: Added transmission for simulation and physical properties to link

File: rbsherpa_hl_description/urdf/structures/elevator_structure.urdf.xacro (robot description, xacro)
@@ -4,4 +4,10 @@
   <xacro:property name="deg2rad" value="0.01745329251"/>
   <xacro:macro name="elevator_structure" params="prefix parent *origin">
+   <xacro:macro name="solid_cuboid_inertia" params="m h d w">
+    <inertia  ixx="${(m*(h*h+d*d))/12}" ixy = "0" ixz = "0"
+              iyy="${(m*(w*w+d*d))/12}" iyz = "0"
+              izz="${(m*(w*w+h*h))/12}"
+    />
+   </xacro:macro>
 	<!--fixed joint -->
     <joint name="${prefix}structure_joint" type="fixed">
@@ -24,9 +30,7 @@
       </collision>
       <inertial>
-        <mass value="14.92765" />
-        <origin xyz="-0.0195 -0.01 -0.750" />
-        <inertia  ixx="2.80754349924" ixy = "0" ixz = "0"
-                  iyy="2.80407121984" iyz = "0"
-                  izz="0.01374410335" />
+        <mass value="0.005" />
+        <origin xyz="0 0 -0.27" />
+        <solid_cuboid_inertia m="0.005" h="0.05" d="0.05" w="0.05"/>
       </inertial>
     </link>
@@ -37,5 +41,5 @@
       <child link="${prefix}torso_elevator_link"/>
       <axis xyz="0 0 1"/>
-      <limit lower="0.0" upper="0.5" effort="1.0" velocity="0.5"/>
+      <limit lower="0.0" upper="0.5" effort="1.0" velocity="0.07"/>
       <xacro:insert_block name="origin" />
     </joint>
@@ -54,16 +58,25 @@
       </collision>
       <inertial>
-        <mass value="14.92765" />
-        <origin xyz="-0.0195 -0.01 -0.750" />
-        <inertia  ixx="2.80754349924" ixy = "0" ixz = "0"
-                  iyy="2.80407121984" iyz = "0"
-                  izz="0.01374410335" />
+        <mass value="0.005" />
+        <origin xyz="0 0 -0.27" />
+        <solid_cuboid_inertia m="0.005" h="0.05" d="0.05" w="0.05"/>
       </inertial>
     </link>
-    <joint name="${prefix}torso_pantilt_pan_joint" type="continuous">
+    <transmission name="${prefix}torso_elevator_trans">
+        <type>transmission_interface/SimpleTransmission</type>
+        <joint name="${prefix}torso_elevator_joint">
+          <hardwareInterface>hardware_interface/PositionJointInterface</hardwareInterface>
+        </joint>
+        <actuator name="${prefix}torso_elevator_motor">
+          <mechanicalReduction>1</mechanicalReduction>
+          <hardwareInterface>hardware_interface/PositionJointInterface</hardwareInterface>
+        </actuator>
+    </transmission>
+    <joint name="${prefix}torso_pantilt_pan_joint" type="revolute">
       <parent link="${prefix}torso_elevator_link"/>
       <origin xyz="0.0 0.0 1.37" rpy="0 0 0" />
       <child link="${prefix}torso_pantilt_pan_link"/>
       <axis xyz="0 0 1"/>
+      <limit lower="-3.14" upper="3.14" effort="1.0" velocity="0.1"/>
       <xacro:insert_block name="origin" />
     </joint>
@@ -82,11 +95,19 @@
       </collision>
       <inertial>
-        <mass value="14.92765" />
-        <origin xyz="-0.0195 -0.01 -0.750" />
-        <inertia  ixx="2.80754349924" ixy = "0" ixz = "0"
-                  iyy="2.80407121984" iyz = "0"
-                  izz="0.01374410335" />
+        <mass value="0.005" />
+        <origin xyz="0 0 -0.27" />
+        <solid_cuboid_inertia m="0.005" h="0.05" d="0.05" w="0.05"/>
       </inertial>
     </link>
+    <transmission name="${prefix}torso_pantilt_pan_trans">
+        <type>transmission_interface/SimpleTransmission</type>
+        <joint name="${prefix}torso_pantilt_pan_joint">
+          <hardwareInterface>hardware_interface/PositionJointInterface</hardwareInterface>
+        </joint>
+        <actuator name="${prefix}torso_pantilt_pan_motor">
+          <mechanicalReduction>1</mechanicalReduction>
+          <hardwareInterface>hardware_interface/PositionJointInterface</hardwareInterface>
+        </actuator>
+    </transmission>
     <joint name="${prefix}torso_beacon_joint" type="fixed">
       <parent link="${prefix}torso_pantilt_pan_link"/>
@@ -102,5 +123,5 @@
       <child link="${prefix}gun_tilt_link"/>
       <axis xyz="0 1 0"/>
-      <limit lower="0.0" upper="-0.57" effort="1.0" velocity="0.5"/>
+      <limit lower="-0.57" upper="0.1" effort="1.0" velocity="0.5"/>
       <xacro:insert_block name="origin" />
     </joint>
@@ -122,9 +143,19 @@
       </collision>
       <inertial>
-        <origin xyz="0 0 0" rpy="0 0 0"/>
-        <mass value="5"/>
-        <inertia ixx="1.0" ixy="0.0" ixz="0.0" iyy="1.0" iyz="0.0" izz="1.0"/>
+        <mass value="0.005" />
+        <origin xyz="0 0 -0.27" />
+        <solid_cuboid_inertia m="0.005" h="0.05" d="0.05" w="0.05"/>
       </inertial>
     </link>
+    <transmission name="${prefix}gun_tilt_trans">
+        <type>transmission_interface/SimpleTransmission</type>
+        <joint name="${prefix}gun_tilt_joint">
+          <hardwareInterface>hardware_interface/PositionJointInterface</hardwareInterface>
+        </joint>
+        <actuator name="${prefix}gun_tilt_motor">
+          <mechanicalReduction>1</mechanicalReduction>
+          <hardwareInterface>hardware_interface/PositionJointInterface</hardwareInterface>
+        </actuator>
+    </transmission>
     <joint name="${prefix}gun_joint" type="fixed">
       <parent link="${prefix}gun_tilt_link"/>

File: rbsherpa_hl_description/urdf/structures/gimbal.urdf.xacro (robot description, xacro)
@@ -3,4 +3,10 @@
   <xacro:property name="M_PI" value="3.1415926535897931" />
   <xacro:macro name="gimbal" params="prefix parent *origin">
+    <xacro:macro name="solid_cuboid_inertia" params="m h d w">
+    <inertia  ixx="${(m*(h*h+d*d))/12}" ixy = "0" ixz = "0"
+              iyy="${(m*(w*w+d*d))/12}" iyz = "0"
+              izz="${(m*(w*w+h*h))/12}"
+    />
+    </xacro:macro>
     <!-- gimbal base -->
     <joint name="${prefix}gimbal_base_joint" type="fixed">
@@ -11,4 +17,21 @@
     </joint>
     <link name="${prefix}gimbal_base_link">
+    <visual>
+        <origin xyz="0 0 0" rpy="0 0 0" />
+        <geometry>
+          <box size="0.01 0.01 0.01" />
+        </geometry>
+      </visual>
+      <collision>
+        <origin xyz="0 0 0" rpy="0 0 0"/>
+        <geometry>
+          <cylinder radius="0.05" length="0.05"/>
+        </geometry>
+      </collision>
+      <inertial>
+        <mass value="0.005" />
+        <origin xyz="0 0 -0.27" />
+        <solid_cuboid_inertia m="0.005" h="0.05" d="0.05" w="0.05"/>
+      </inertial>
     </link>
     <joint name="${prefix}gimbal_yaw_joint" type="revolute">
@@ -17,15 +40,35 @@
       <child link="${prefix}gimbal_yaw_link"/>
       <axis xyz="0 0 1"/>
-      <limit lower="-1.57" upper="1.57" effort="1.0" velocity="0.5"/>
+      <limit lower="-1.57" upper="1.57" effort="1.0" velocity="0.2"/>
     </joint>
     <link name="${prefix}gimbal_yaw_link">
+      <visual>
+        <origin xyz="0 0 0" rpy="0 0 0" />
+        <geometry>
+          <box size="0.01 0.01 0.01" />
+        </geometry>
+      </visual>
+      <collision>
+        <origin xyz="0 0 0" rpy="0 0 0"/>
+        <geometry>
+          <cylinder radius="0.05" length="0.05"/>
+        </geometry>
+      </collision>
+      <inertial>
+        <mass value="0.005" />
+        <origin xyz="0 0 -0.27" />
+        <solid_cuboid_inertia m="0.005" h="0.05" d="0.05" w="0.05"/>
+      </inertial>
     </link>
-    <!--joint name="${prefix}gimbal_first_axis_joint" type="fixed">
-      <parent link="${prefix}gimbal_yaw_link"/>
-      <origin xyz="-0.072 0.0 -0.026" rpy="0 0 0" />
-      <child link="${prefix}gimbal_first_axis_link"/>
-    </joint>
-    <link name="${prefix}gimbal_first_axis_link">
-    </link-->
+    <transmission name="${prefix}gimbal_yaw_trans">
+        <type>transmission_interface/SimpleTransmission</type>
+        <joint name="${prefix}gimbal_yaw_joint">
+          <hardwareInterface>hardware_interface/PositionJointInterface</hardwareInterface>
+        </joint>
+        <actuator name="${prefix}gimbal_yaw_motor">
+          <mechanicalReduction>1</mechanicalReduction>
+          <hardwareInterface>hardware_interface/PositionJointInterface</hardwareInterface>
+        </actuator>
+    </transmission>
     <joint name="${prefix}gimbal_roll_joint" type="revolute">
       <parent link="${prefix}gimbal_yaw_link"/>
@@ -33,8 +76,23 @@
       <child link="${prefix}gimbal_roll_link"/>
       <axis xyz="1 0 0"/>
-      <limit lower="-1.57" upper="1.57" effort="1.0" velocity="0.5"/>
+      <limit lower="-1.57" upper="1.57" effort="1.0" velocity="0.2"/>
     </joint>
     <link name="${prefix}gimbal_roll_link">
+      <inertial>
+        <mass value="0.005" />
+        <origin xyz="0 0 -0.27" />
+        <solid_cuboid_inertia m="0.005" h="0.05" d="0.05" w="0.05"/>
+      </inertial>
     </link>
+    <transmission name="${prefix}gimbal_roll_trans">
+        <type>transmission_interface/SimpleTransmission</type>
+        <joint name="${prefix}gimbal_roll_joint">
+          <hardwareInterface>hardware_interface/PositionJointInterface</hardwareInterface>
+        </joint>
+        <actuator name="${prefix}gimbal_roll_motor">
+          <mechanicalReduction>1</mechanicalReduction>
+          <hardwareInterface>hardware_interface/PositionJointInterface</hardwareInterface>
+        </actuator>
+    </transmission>
     <joint name="${prefix}gimbal_pitch_joint" type="revolute">
       <parent link="${prefix}gimbal_roll_link"/>
@@ -42,8 +100,23 @@
       <child link="${prefix}gimbal_pitch_link"/>
       <axis xyz="0 1 0"/>
-      <limit lower="-1.57" upper="1.57" effort="1.0" velocity="0.5"/>
+      <limit lower="-1.57" upper="1.57" effort="1.0" velocity="0.2"/>
     </joint>
     <link name="${prefix}gimbal_pitch_link">
+      <inertial>
+        <mass value="0.005" />
+        <origin xyz="0 0 -0.27" />
+        <solid_cuboid_inertia m="0.005" h="0.05" d="0.05" w="0.05"/>
+      </inertial>
     </link>
+    <transmission name="${prefix}gimbal_pitch_trans">
+        <type>transmission_interface/SimpleTransmission</type>
+        <joint name="${prefix}gimbal_pitch_joint">
+          <hardwareInterface>hardware_interface/PositionJointInterface</hardwareInterface>
+        </joint>
+        <actuator name="${prefix}gimbal_pitch_motor">
+          <mechanicalReduction>1</mechanicalReduction>
+          <hardwareInterface>hardware_interface/PositionJointInterface</hardwareInterface>
+        </actuator>
+    </transmission>
     <joint name="${prefix}gimbal_camera_joint" type="fixed">
       <parent link="${prefix}gimbal_pitch_link"/>

Commit message: Merge rbsherpa_hl_description from robot

File: rbsherpa_hl_description/urdf/structures/elevator_structure.urdf.xacro (robot description, xacro)
@@ -1,14 +1,12 @@
 <?xml version="1.0"?>
-<robot name="rbsherpa_structure" xmlns:xacro="http://www.ros.org/wiki/xacro">
+<robot name="rbsherpa_structure"
+  xmlns:xacro="http://www.ros.org/wiki/xacro">
   <xacro:property name="M_PI" value="3.1415926535897931" />
   <xacro:property name="deg2rad" value="0.01745329251"/>
   <xacro:macro name="elevator_structure" params="prefix parent *origin">
-   <xacro:macro name="solid_cuboid_inertia" params="m h d w">
-    <inertia  ixx="${(m*(h*h+d*d))/12}" ixy = "0" ixz = "0"
-              iyy="${(m*(w*w+d*d))/12}" iyz = "0"
-              izz="${(m*(w*w+h*h))/12}"
-    />
-   </xacro:macro>
-	<!--fixed joint -->
+    <xacro:macro name="solid_cuboid_inertia" params="m h d w">
+      <inertia ixx="${(m*(h*h+d*d))/12}" ixy = "0" ixz = "0" iyy="${(m*(w*w+d*d))/12}" iyz = "0" izz="${(m*(w*w+h*h))/12}" />
+    </xacro:macro>
+    <!--fixed joint -->
     <joint name="${prefix}structure_joint" type="fixed">
       <parent link="${parent}"/>
@@ -20,11 +18,11 @@
         <origin xyz="0 0 0" rpy="0 0 0" />
         <geometry>
-		      <mesh filename="package://rbsherpa_hl_description/meshes/structure/rbsherpa_hl_structure.dae" />
+          <mesh filename="package://rbsherpa_hl_description/meshes/structure/rbsherpa_hl_structure.dae" />
         </geometry>
       </visual>
       <collision>
-		    <origin xyz="0 0 0" rpy="0 0 0" />
+        <origin xyz="0 0 0" rpy="0 0 0" />
         <geometry>
-			    <mesh filename="package://rbsherpa_hl_description/meshes/structure/rbsherpa_hl_structure.stl" />
+          <mesh filename="package://rbsherpa_hl_description/meshes/structure/rbsherpa_hl_structure.stl" />
         </geometry>
       </collision>
@@ -41,5 +39,5 @@
       <child link="${prefix}torso_elevator_link"/>
       <axis xyz="0 0 1"/>
-      <limit lower="0.0" upper="0.5" effort="100.0" velocity="0.07"/>
+      <limit lower="0.0" upper="1.2" effort="100.0" velocity="0.07"/>
       <xacro:insert_block name="origin" />
     </joint>
@@ -48,11 +46,11 @@
         <origin xyz="0 0 0" rpy="0 0 0" />
         <geometry>
-		      <mesh filename="package://rbsherpa_hl_description/meshes/structure/rbsherpa_hl_elevator.dae" />
+          <mesh filename="package://rbsherpa_hl_description/meshes/structure/rbsherpa_hl_elevator.dae" />
         </geometry>
       </visual>
       <collision>
-		    <origin xyz="0 0 0" rpy="0 0 0" />
+        <origin xyz="0 0 0" rpy="0 0 0" />
         <geometry>
-			    <mesh filename="package://rbsherpa_hl_description/meshes/structure/rbsherpa_hl_elevator.stl" />
+          <mesh filename="package://rbsherpa_hl_description/meshes/structure/rbsherpa_hl_elevator.stl" />
         </geometry>
       </collision>
@@ -64,19 +62,19 @@
     </link>
     <transmission name="${prefix}torso_elevator_trans">
-        <type>transmission_interface/SimpleTransmission</type>
-        <joint name="${prefix}torso_elevator_joint">
-          <hardwareInterface>hardware_interface/PositionJointInterface</hardwareInterface>
-        </joint>
-        <actuator name="${prefix}torso_elevator_motor">
-          <mechanicalReduction>1</mechanicalReduction>
-          <hardwareInterface>hardware_interface/PositionJointInterface</hardwareInterface>
-        </actuator>
+      <type>transmission_interface/SimpleTransmission</type>
+      <joint name="${prefix}torso_elevator_joint">
+        <hardwareInterface>hardware_interface/PositionJointInterface</hardwareInterface>
+      </joint>
+      <actuator name="${prefix}torso_elevator_motor">
+        <mechanicalReduction>1</mechanicalReduction>
+        <hardwareInterface>hardware_interface/PositionJointInterface</hardwareInterface>
+      </actuator>
     </transmission>
     <joint name="${prefix}torso_pantilt_pan_joint" type="revolute">
       <parent link="${prefix}torso_elevator_link"/>
-      <origin xyz="0.0 0.0 1.37" rpy="0 0 0" />
+      <origin xyz="0.0 0.0 1.37" rpy="0 0 3.14" />
       <child link="${prefix}torso_pantilt_pan_link"/>
-      <axis xyz="0 0 1"/>
-      <limit lower="-3.14" upper="3.14" effort="10.0" velocity="0.5"/>
+      <limit lower="-3.0" upper="3.1415" effort="1" velocity="0.5"/>
+      <axis xyz="0 0 -1"/>
       <xacro:insert_block name="origin" />
     </joint>
@@ -85,11 +83,11 @@
         <origin xyz="0 0 0" rpy="0 0 0" />
         <geometry>
-		      <mesh filename="package://rbsherpa_hl_description/meshes/structure/rbsherpa_hl_pan_structure.dae" />
+          <mesh filename="package://rbsherpa_hl_description/meshes/structure/rbsherpa_hl_pan_structure.dae" />
         </geometry>
       </visual>
       <collision>
-		    <origin xyz="0 0 0" rpy="0 0 0" />
+        <origin xyz="0 0 0" rpy="0 0 0" />
         <geometry>
-			    <mesh filename="package://rbsherpa_hl_description/meshes/structure/rbsherpa_hl_pan_structure.stl" />
+          <mesh filename="package://rbsherpa_hl_description/meshes/structure/rbsherpa_hl_pan_structure.stl" />
         </geometry>
       </collision>
@@ -101,12 +99,12 @@
     </link>
     <transmission name="${prefix}torso_pantilt_pan_trans">
-        <type>transmission_interface/SimpleTransmission</type>
-        <joint name="${prefix}torso_pantilt_pan_joint">
-          <hardwareInterface>hardware_interface/PositionJointInterface</hardwareInterface>
-        </joint>
-        <actuator name="${prefix}torso_pantilt_pan_motor">
-          <mechanicalReduction>1</mechanicalReduction>
-          <hardwareInterface>hardware_interface/PositionJointInterface</hardwareInterface>
-        </actuator>
+      <type>transmission_interface/SimpleTransmission</type>
+      <joint name="${prefix}torso_pantilt_pan_joint">
+        <hardwareInterface>hardware_interface/PositionJointInterface</hardwareInterface>
+      </joint>
+      <actuator name="${prefix}torso_pantilt_pan_motor">
+        <mechanicalReduction>1</mechanicalReduction>
+        <hardwareInterface>hardware_interface/PositionJointInterface</hardwareInterface>
+      </actuator>
     </transmission>
     <joint name="${prefix}torso_beacon_joint" type="fixed">
@@ -118,21 +116,21 @@
     <link name="${prefix}torso_beacon_link">
     </link>
-    <joint name="${prefix}gun_tilt_joint" type="revolute">
+    <joint name="${prefix}torso_pantilt_tilt_joint" type="revolute">
       <parent link="${prefix}torso_pantilt_pan_link"/>
       <origin xyz="-0.42 -0.015 0.23" rpy="0 0 ${M_PI}" />
-      <child link="${prefix}gun_tilt_link"/>
+      <child link="${prefix}torso_pantilt_tilt_link"/>
       <axis xyz="0 1 0"/>
-      <limit lower="-0.57" upper="0.1" effort="10.0" velocity="0.5"/>
+      <limit lower="-0.21" upper="0.25" effort="10.0" velocity="0.5"/>
       <xacro:insert_block name="origin" />
     </joint>
-    <link name="${prefix}gun_tilt_link">
-       <visual>
+    <link name="${prefix}torso_pantilt_tilt_link">
+      <visual>
         <origin xyz="0 0.045 0" rpy="0 0 ${M_PI}"/>
         <geometry>
           <mesh filename="package://rbsherpa_hl_description/meshes/pantilt/tilt_dynamixel.stl"/>
         </geometry>
-       <material name="lightgrey">
-         <color rgba="0.3 0.3 0.3 1"/>
-       </material>
+        <material name="lightgrey">
+          <color rgba="0.3 0.3 0.3 1"/>
+        </material>
       </visual>
       <collision>
@@ -149,15 +147,15 @@
     </link>
     <transmission name="${prefix}gun_tilt_trans">
-        <type>transmission_interface/SimpleTransmission</type>
-        <joint name="${prefix}gun_tilt_joint">
-          <hardwareInterface>hardware_interface/PositionJointInterface</hardwareInterface>
-        </joint>
-        <actuator name="${prefix}gun_tilt_motor">
-          <mechanicalReduction>1</mechanicalReduction>
-          <hardwareInterface>hardware_interface/PositionJointInterface</hardwareInterface>
-        </actuator>
+      <type>transmission_interface/SimpleTransmission</type>
+      <joint name="${prefix}torso_pantilt_tilt_joint">
+        <hardwareInterface>hardware_interface/PositionJointInterface</hardwareInterface>
+      </joint>
+      <actuator name="${prefix}gun_tilt_motor">
+        <mechanicalReduction>1</mechanicalReduction>
+        <hardwareInterface>hardware_interface/PositionJointInterface</hardwareInterface>
+      </actuator>
     </transmission>
     <joint name="${prefix}gun_joint" type="fixed">
-      <parent link="${prefix}gun_tilt_link"/>
+      <parent link="${prefix}torso_pantilt_tilt_link"/>
       <origin xyz="0.0 -0.03 0.0" rpy="0 0 0" />
       <child link="${prefix}gun_link"/>

File: rbsherpa_hl_description/urdf/structures/gimbal.urdf.xacro (robot description, xacro)
@@ -39,6 +39,6 @@
       <origin xyz="0.0 0.0 -0.097" rpy="0 0 0" />
       <child link="${prefix}gimbal_yaw_link"/>
-      <axis xyz="0 0 1"/>
-      <limit lower="-1.57" upper="1.57" effort="1.0" velocity="0.2"/>
+      <axis xyz="0 0 -1"/>
+      <limit lower="-1.57" upper="1.57" effort="1.0" velocity="0.5"/>
     </joint>
     <link name="${prefix}gimbal_yaw_link">
@@ -99,6 +99,6 @@
       <origin xyz="0.134 0.110 0.0" rpy="0 0 0" />
       <child link="${prefix}gimbal_pitch_link"/>
-      <axis xyz="0 1 0"/>
-      <limit lower="-1.57" upper="1.57" effort="1.0" velocity="0.2"/>
+      <axis xyz="0 -1 0"/>
+      <limit lower="-1.57" upper="1.57" effort="1.0" velocity="0.5"/>
     </joint>
     <link name="${prefix}gimbal_pitch_link">
